File: Kicad/ps2.sch (KiCad schematic (older format))
At the start: 1 part, among them J701 Double-mini-DIN-6

Commit message: Completed PSU design.
Also changed footprint for stacked USB connector to change
shield pins from SHx to Pin 9.
Parts:
- removed J701: Double-mini-DIN-6, Neotron-Common-Hardware:Double_mini-DIN_6, symbol Neotron-Common-Hardware:Double-mini-DIN-6
Connections:
- no-connect marks 12 -> 0
Other:
- note removed: "Dual mini-DIN 6 connectors for PS/2 Keyboard and PS/2 Mouse.\nSignalling is 5V open-collector, with pull-up required."
Changed lines of the file:
@@
 Comment4 ""
 $EndDescr
-$Comp
-L Neotron-Common-Hardware:Double-mini-DIN-6 J?
-U 1 1 5FDEE757
-P 3550 3100
-AR Path="/5FDEE757" Ref="J?"  Part="1"
-AR Path="/5FDEDE75/5FDEE757" Ref="J701"  Part="1"
-F 0 "J701" H 3550 3798 50  0000 C CNN
-F 1 "Double-mini-DIN-6" H 3550 3707 50  0000 C CNN
-F 2 "Neotron-Common-Hardware:Double_mini-DIN_6" H 3550 3350 50  0001 C CNN
-F 3 "http://www.kycon.com/Pub_Eng_Draw/KMDGX-6S-6S-S4N.pdf" H 3550 3350 50  0001 C CNN
-F 4 "2092-KMDGX-6S/6S-S4N-ND" H 3550 3100 50  0001 C CNN "Digikey"
-F 5 "0" H 3550 3100 50  0001 C CNN "DNP"
-	1    3550 3100
-	1    0    0    -1
-$EndComp
-Text Notes 4250 2800 0    50   ~ 0
-Dual mini-DIN 6 connectors for PS/2 Keyboard and PS/2 Mouse.\nSignalling is 5V open-collector, with pull-up required.
-NoConn ~ 3250 2750
-NoConn ~ 3250 2850
-NoConn ~ 3250 2950
-NoConn ~ 3250 3300
-NoConn ~ 3250 3400
-NoConn ~ 3250 3500
-NoConn ~ 3850 3500
-NoConn ~ 3850 3400
-NoConn ~ 3850 3300
-NoConn ~ 3850 2950
-NoConn ~ 3850 2850
-NoConn ~ 3850 2750
 $EndSCHEMATC
