File: Kicad/audio.sch (KiCad schematic (older format))
At the start: 71 parts, among them J401 CD Audio In, J402 AC'97 Audio Header, J403 Line Out, U401 TLV320AIC23BPW, U402 STX-4335-5BGP-S1, Y401 12M

Commit message: Replaced NUC029 (TSSOP) with KE04 (SOIC).
Also updated the BOM with some part nos.
Parts:
- C402, C403, C404, C407, C409, C410, C412, C414, C415, C417: Digikey 493-10359-1-ND -> 493-10359-1-ND; MPN (none) -> UMW1E100MDD1TP; mpn UMW1E100MDD1TP -> (none)
- C406, C408, C411, C413, C416: Digikey BC1150CT-ND -> BC1150CT-ND; MPN (none) -> K104K15X7RF5TL2; mpn K104K15X7RF5TL2 -> (none)
- C418, C419, C422, C423: MPN (none) -> FG18X7R1H474KRT06; mpn FG18X7R1H474KRT06 -> (none)
- C420, C421: Digikey 493-15424-ND -> 493-15424-ND; MPN (none) -> UKT1C221MED; mpn UKT1C221MED -> (none)
- C425: Digikey 493-10944-1-ND -> 493-10944-1-ND; MPN (none) -> UFG1H010MDM1TD; mpn UFG1H010MDM1TD -> (none)
- FB401, FB402, FB403, FB404, FB405, FB406, FB408, FB409, FB410, FB411: MPN (none) -> BLM21PG221SN1D; mpn BLM21PG221SN1D -> (none)
- FB407: MPN (none) -> HZ0805E601R-10; mpn HZ0805E601R-10 -> (none)
- U401: Digikey (none) -> 296-26817-1-ND; MPN (none) -> TLV320AIC23BPW; Manufacturer (none) -> Texas Instruments
- U402: Digikey (none) -> 2092-STX-4335-5BGP-S1-ND; MPN (none) -> STX-4335-5BGP-S1; Manufacturer (none) -> Kycon
- Y401: Digikey 535-9037-ND -> 535-9037-ND; MPN (none) -> ABL-12.000MHZ-B2; mpn ABL-12.000MHZ-B2 -> (none)

Commit message: Bring in R2R DAC from Neotron-9X schematic.
Parts:
- renumbered C412 to C601, C413 to C602, C407 to C603, C411 to C604, C418 to C605, C419 to C606, C424 to C607, C427 to C608, C431 to C609, C435 to C610, C402 to C611, C406 to C612, C408 to C613, C420 to C614, C421 to C615, C426 to C616, C428 to C617, C432 to C618, C437 to C619, C422 to C620, C423 to C621, C430 to C622, C433 to C623, C436 to C624, C438 to C625, C415 to C626, C416 to C627, C401 to C628, C405 to C629, C425 to C630, C429 to C631, C434 to C632, C403 to C633, C409 to C634, C414 to C635, C417 to C636, C404 to C637, C410 to C638, FB405 to FB601, FB409 to FB602, FB406 to FB603, FB410 to FB604, FB408 to FB605, FB411 to FB606, FB407 to FB607, FB401 to FB608, FB403 to FB609, FB402 to FB610, FB404 to FB611, J403 to J601, J402 to J602, J401 to J603, R404 to R601, R405 to R602, R406 to R603, R409 to R604, R407 to R605, R410 to R606, R414 to R607, R415 to R608, R408 to R609, R413 to R610, R411 to R611, R412 to R612, R416 to R613, R401 to R614, R403 to R615, R402 to R616, U401 to U601, U402 to U602, Y401 to Y601
