File: Kicad/video.sch (KiCad schematic (older format))
At the start: 18 parts, among them J201 DE15HD, U201 TPF133A, U202 TPD7S019

Commit message: Fix up ERC errors.
~FAULT on the MIC2005 is an active-low common collector output.
Well done ERC for spotting that I can't join three output pins together!
Other:
- note added: "Place near U201"
- note added: "RGB Buffer\n0.7V p-p inputs\n1.4V p-p outputs, into 75 ohm co-ax"
- note removed: "Place near U102"
- note removed: "RGB Buffer"
- moved on the sheet: C201
Changed lines of the file:
@@
 L Device:C C201
 U 1 1 5FEDB6AA
-P 6900 4200
-F 0 "C201" V 6648 4200 50  0000 C CNN
-F 1 "220n" V 6739 4200 50  0000 C CNN
-F 2 "Capacitor_SMD:C_0805_2012Metric_Pad1.15x1.40mm_HandSolder" H 6938 4050 50  0001 C CNN
-F 3 "~" H 6900 4200 50  0001 C CNN
-	1    6900 4200
+P 6750 4200
+F 0 "C201" V 6498 4200 50  0000 C CNN
+F 1 "220n" V 6589 4200 50  0000 C CNN
+F 2 "Capacitor_SMD:C_0805_2012Metric_Pad1.15x1.40mm_HandSolder" H 6788 4050 50  0001 C CNN
+F 3 "~" H 6750 4200 50  0001 C CNN
+	1    6750 4200
 	0    1    1    0
 $EndComp
@@
 L power:GND #PWR0212
 U 1 1 5FEDBFC5
-P 7100 4250
-F 0 "#PWR0212" H 7100 4000 50  0001 C CNN
-F 1 "GND" H 7250 4200 50  0000 C CNN
-F 2 "" H 7100 4250 50  0001 C CNN
-F 3 "" H 7100 4250 50  0001 C CNN
-	1    7100 4250
+P 6950 4250
+F 0 "#PWR0212" H 6950 4000 50  0001 C CNN
+F 1 "GND" H 7100 4200 50  0000 C CNN
+F 2 "" H 6950 4250 50  0001 C CNN
+F 3 "" H 6950 4250 50  0001 C CNN
+	1    6950 4250
 	1    0    0    -1
 $EndComp
@@
 Text Notes 5300 5000 2    50   Italic 0
 ESD Protection
-Text Notes 3700 3400 0    50   Italic 0
-RGB Buffer
+Text Notes 1900 2550 0    50   Italic 0
+RGB Buffer\n0.7V p-p inputs\n1.4V p-p outputs, into 75 ohm co-ax
 $Comp
 L power:+3V3 #PWR0201
@@
 Place near U202
 Text Notes 2250 6600 0    50   Italic 0
-Place near U102
+Place near U201
 $Comp
 L power:+3V3 #PWR0220
@@
 	8150 3950 8300 3950
 Wire Wire Line
-	6600 4200 6750 4200
-Wire Wire Line
-	7050 4200 7100 4200
-Wire Wire Line
-	7100 4200 7100 4250
+	6900 4200 6950 4200
+Wire Wire Line
+	6950 4200 6950 4250
+Text Notes 4050 3350 0    50   Italic 0
+Place near U201
+Text Notes 1300 3600 0    50   Italic 0
+Place near U201
 $EndSCHEMATC

Commit message: Replaced NUC029 (TSSOP) with KE04 (SOIC).
Also updated the BOM with some part nos.
Parts:
- C201, R201, R202, R203, R204, R205, R206, R207, R208: DNP (none) -> 0
- C202, C203, C204, C205: DNP (none) -> 0; Digikey (none) -> BC1150CT-ND; MPN (none) -> K104K15X7RF5TL2; Manufacturer (none) -> Vishay
- C206: DNP (none) -> 0; Digikey (none) -> 493-10359-1-ND; MPN (none) -> UMW1E100MDD1TP; Manufacturer (none) -> Nichicon
- R209: value DNP -> DNF; DNP (none) -> 1
- U201: value TPF133A -> THS7316; DNP (none) -> 0; Digikey (none) -> 296-26684-1-ND; MPN (none) -> THS7316; Manufacturer 3Peak -> Texas Instruments
- U202: DNP (none) -> 0; Digikey (none) -> 296-27595-1-ND
Changed lines of the file:
@@
 F 2 "Resistor_SMD:R_0805_2012Metric_Pad1.15x1.40mm_HandSolder" V 4380 2800 50  0001 C CNN
 F 3 "~" H 4450 2800 50  0001 C CNN
+F 4 "0" H 4450 2800 50  0001 C CNN "DNP"
 	1    4450 2800
 	0    1    1    0
@@
 F 2 "Resistor_SMD:R_0805_2012Metric_Pad1.15x1.40mm_HandSolder" V 4380 3000 50  0001 C CNN
 F 3 "~" H 4450 3000 50  0001 C CNN
+F 4 "0" H 4450 3000 50  0001 C CNN "DNP"
 	1    4450 3000
 	0    1    1    0
@@
 F 2 "Resistor_SMD:R_0805_2012Metric_Pad1.15x1.40mm_HandSolder" V 4380 3200 50  0001 C CNN
 F 3 "~" H 4450 3200 50  0001 C CNN
+F 4 "0" H 4450 3200 50  0001 C CNN "DNP"
 	1    4450 3200
 	0    1    1    0
@@
 F 2 "Resistor_SMD:R_0805_2012Metric_Pad1.15x1.40mm_HandSolder" V 2130 3350 50  0001 C CNN
 F 3 "~" H 2200 3350 50  0001 C CNN
+F 4 "0" H 2200 3350 50  0001 C CNN "DNP"
 	1    2200 3350
 	-1   0    0    1
@@
 F 2 "Resistor_SMD:R_0805_2012Metric_Pad1.15x1.40mm_HandSolder" V 2480 3350 50  0001 C CNN
 F 3 "~" H 2550 3350 50  0001 C CNN
+F 4 "0" H 2550 3350 50  0001 C CNN "DNP"
 	1    2550 3350
 	-1   0    0    1
@@
 F 2 "Resistor_SMD:R_0805_2012Metric_Pad1.15x1.40mm_HandSolder" V 2830 3350 50  0001 C CNN
 F 3 "~" H 2900 3350 50  0001 C CNN
+F 4 "0" H 2900 3350 50  0001 C CNN "DNP"
 	1    2900 3350
 	-1   0    0    1
@@
 F 4 "Texas Instruments" H 5950 2950 50  0001 C CNN "Manufacturer"
 F 5 "TPD7S019" H 5950 2850 50  0001 C CNN "MPN"
+F 6 "0" H 5950 4300 50  0001 C CNN "DNP"
+F 7 "296-27595-1-ND" H 5950 4300 50  0001 C CNN "Digikey"
 	1    5950 4300
 	1    0    0    -1
@@
 P 3700 3000
 F 0 "U201" H 4000 3300 50  0000 R CNN
-F 1 "TPF133A" H 3250 3300 50  0000 C CNN
+F 1 "THS7316" H 3250 3300 50  0000 C CNN
 F 2 "Package_SO:SOIC-8_3.9x4.9mm_P1.27mm" H 3700 2450 100 0001 C CNN
 F 3 "https://datasheet.lcsc.com/szlcsc/1810181731_3PEAK-TPF133A-SR_C155446.pdf" H 3000 2950 100 0001 C CNN
-F 4 "3Peak" H 3800 3300 50  0001 C CNN "Manufacturer"
+F 4 "Texas Instruments" H 3800 3300 50  0001 C CNN "Manufacturer"
+F 5 "0" H 3700 3000 50  0001 C CNN "DNP"
+F 6 "296-26684-1-ND" H 3700 3000 50  0001 C CNN "Digikey"
+F 7 "THS7316" H 3700 3000 50  0001 C CNN "MPN"
 	1    3700 3000
 	1    0    0    -1
@@
 F 2 "Resistor_SMD:R_0805_2012Metric_Pad1.15x1.40mm_HandSolder" V 8580 4250 50  0001 C CNN
 F 3 "~" H 8650 4250 50  0001 C CNN
+F 4 "0" H 8650 4250 50  0001 C CNN "DNP"
 	1    8650 4250
 	1    0    0    -1
@@
 F 2 "Resistor_SMD:R_0805_2012Metric_Pad1.15x1.40mm_HandSolder" V 8930 4250 50  0001 C CNN
 F 3 "~" H 9000 4250 50  0001 C CNN
+F 4 "0" H 9000 4250 50  0001 C CNN "DNP"
 	1    9000 4250
 	1    0    0    -1
@@
 F 2 "Capacitor_SMD:C_0805_2012Metric_Pad1.15x1.40mm_HandSolder" H 6788 4050 50  0001 C CNN
 F 3 "~" H 6750 4200 50  0001 C CNN
+F 4 "0" H 6750 4200 50  0001 C CNN "DNP"
 	1    6750 4200
 	0    1    1    0
@@
 F 2 "Capacitor_SMD:C_0805_2012Metric_Pad1.15x1.40mm_HandSolder" H 838 7000 50  0001 C CNN
 F 3 "~" H 800 7150 50  0001 C CNN
+F 4 "0" H 800 7150 50  0001 C CNN "DNP"
+F 5 "BC1150CT-ND" H 800 7150 50  0001 C CNN "Digikey"
+F 6 "K104K15X7RF5TL2" H 800 7150 50  0001 C CNN "MPN"
+F 7 "Vishay" H 800 7150 50  0001 C CNN "Manufacturer"
 	1    800  7150
 	-1   0    0    1
@@
 F 2 "Capacitor_SMD:C_0805_2012Metric_Pad1.15x1.40mm_HandSolder" H 1288 7000 50  0001 C CNN
 F 3 "~" H 1250 7150 50  0001 C CNN
+F 4 "0" H 1250 7150 50  0001 C CNN "DNP"
+F 5 "BC1150CT-ND" H 1250 7150 50  0001 C CNN "Digikey"
+F 6 "K104K15X7RF5TL2" H 1250 7150 50  0001 C CNN "MPN"
+F 7 "Vishay" H 1250 7150 50  0001 C CNN "Manufacturer"
 	1    1250 7150
 	-1   0    0    1
@@
 F 2 "Capacitor_SMD:C_0805_2012Metric_Pad1.15x1.40mm_HandSolder" H 1738 7000 50  0001 C CNN
 F 3 "~" H 1700 7150 50  0001 C CNN
+F 4 "0" H 1700 7150 50  0001 C CNN "DNP"
+F 5 "BC1150CT-ND" H 1700 7150 50  0001 C CNN "Digikey"
+F 6 "K104K15X7RF5TL2" H 1700 7150 50  0001 C CNN "MPN"
+F 7 "Vishay" H 1700 7150 50  0001 C CNN "Manufacturer"
 	1    1700 7150
 	-1   0    0    1
@@
 F 2 "Capacitor_SMD:C_0805_2012Metric_Pad1.15x1.40mm_HandSolder" H 2338 7000 50  0001 C CNN
 F 3 "~" H 2300 7150 50  0001 C CNN
+F 4 "0" H 2300 7150 50  0001 C CNN "DNP"
+F 5 "BC1150CT-ND" H 2300 7150 50  0001 C CNN "Digikey"
+F 6 "K104K15X7RF5TL2" H 2300 7150 50  0001 C CNN "MPN"
+F 7 "Vishay" H 2300 7150 50  0001 C CNN "Manufacturer"
 	1    2300 7150
 	-1   0    0    1
@@
 F 2 "Capacitor_THT:CP_Radial_D6.3mm_P2.50mm" H 2788 7000 50  0001 C CNN
 F 3 "~" H 2750 7150 50  0001 C CNN
+F 4 "0" H 2750 7150 50  0001 C CNN "DNP"
+F 5 "493-10359-1-ND" H 2750 7150 50  0001 C CNN "Digikey"
+F 6 "UMW1E100MDD1TP" H 2750 7150 50  0001 C CNN "MPN"
+F 7 "Nichicon" H 2750 7150 50  0001 C CNN "Manufacturer"
 	1    2750 7150
 	-1   0    0    1
@@
 P 8000 3950
 F 0 "R209" V 8100 3950 50  0000 C CNN
-F 1 "DNP" V 7900 3950 50  0000 C CNN
+F 1 "DNF" V 7900 3950 50  0000 C CNN
 F 2 "Resistor_SMD:R_0805_2012Metric_Pad1.15x1.40mm_HandSolder" V 7930 3950 50  0001 C CNN
 F 3 "~" H 8000 3950 50  0001 C CNN
+F 4 "1" H 8000 3950 50  0001 C CNN "DNP"
 	1    8000 3950
 	0    -1   -1   0

Commit message: Video sheet takes digital video, not analog video.
DAC is TBD.
Connections:
- net labels added: BLUE[7..0], BLUE_ANA, GREEN[7..0], GREEN_ANA, RED[7..0], RED_ANA
- net labels removed: BLUE, GREEN, RED
- no-connect marks 2 -> 5
Other:
- note added: "TODO: 24-bit R2R DAC here"
Changed lines of the file:
@@
 $Descr A4 11693 8268
 encoding utf-8
-Sheet 2 9
+Sheet 2 8
 Title "Neotron Common Hardware - Video Output"
 Date "2020-12-26"
@@
 Wire Wire Line
 	3550 2550 3550 2650
-Text HLabel 2000 2850 0    50   Input ~ 0
-RED
-Text HLabel 2000 3000 0    50   Input ~ 0
-GREEN
-Text HLabel 2000 3150 0    50   Input ~ 0
-BLUE
-Wire Wire Line
-	2000 3150 2900 3150
-Wire Wire Line
-	2000 3000 2550 3000
-Wire Wire Line
-	2000 2850 2200 2850
 $Comp
 L Device:R R204
@@
 Text Notes 1300 3600 0    50   Italic 0
 Place near U201
+Text Label 2000 2850 2    50   ~ 0
+RED_ANA
+Text Label 2000 3000 2    50   ~ 0
+GREEN_ANA
+Text Label 2000 3150 2    50   ~ 0
+BLUE_ANA
+Wire Wire Line
+	1750 2850 2200 2850
+Wire Wire Line
+	1750 3000 2550 3000
+Wire Wire Line
+	1750 3150 2900 3150
+Text HLabel 2000 1125 0    50   Input ~ 0
+RED[7..0]
+Text HLabel 2000 1250 0    50   Input ~ 0
+GREEN[7..0]
+Text HLabel 2000 1375 0    50   Input ~ 0
+BLUE[7..0]
+NoConn ~ 2000 1125
+NoConn ~ 2000 1250
+NoConn ~ 2000 1375
+Text Notes 2075 1275 0    50   ~ 0
+TODO: 24-bit R2R DAC here
 $EndSCHEMATC

Commit message: Revised CPU connector to be two 2x20.
This gives more room for larger TQFP-176+ CPUs to be fitted that
didn't fit on the PGA-80 design.
Connections:
- net labels added: BLUE[5..0], GREEN[5..0], RED[5..0]
- net labels removed: BLUE[7..0], GREEN[7..0], RED[7..0]
Other:
- note added: "TODO: 18-bit R2R DAC here"
- note removed: "TODO: 24-bit R2R DAC here"
Changed lines of the file:
@@
 	1750 3150 2900 3150
 Text HLabel 2000 1125 0    50   Input ~ 0
-RED[7..0]
+RED[5..0]
 Text HLabel 2000 1250 0    50   Input ~ 0
-GREEN[7..0]
+GREEN[5..0]
 Text HLabel 2000 1375 0    50   Input ~ 0
-BLUE[7..0]
+BLUE[5..0]
 NoConn ~ 2000 1125
 NoConn ~ 2000 1250
 NoConn ~ 2000 1375
 Text Notes 2075 1275 0    50   ~ 0
-TODO: 24-bit R2R DAC here
+TODO: 18-bit R2R DAC here
 $EndSCHEMATC

Commit message: Bring in R2R DAC from Neotron-9X schematic.
Parts:
- renumbered R209 to R207, R207 to R208, R208 to R209
Connections:
- net labels added: BLUE[0..5], GREEN[0..5], RED[0..5]
- net labels removed: BLUE[5..0], GREEN[5..0], RED[5..0]
- wire segments 99 -> 105
- no-connect marks 5 -> 2
Other:
- note removed: "TODO: 18-bit R2R DAC here"
- moved on the sheet: C201, J201, R201, R202, R203, R204, R205, R206, R207, R208, R209, U201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
