File: Kicad/video.sch (KiCad schematic (older format))
At the start: 18 parts, among them J201 DE15HD, U201 THS7316, U202 TPD7S019

Commit message: Added some part numbers.
Parts:
- C201: Digikey (none) -> 1276-1093-1-ND; MPN (none) -> CL21B224KBFNNNE; Manufacturer (none) -> Samsung
- J201: Digikey (none) -> 609-5180-ND‎; MPN (none) -> ICD15S13E4GV00LF; Manufacturer (none) -> Amphenol
- R201, R202, R203: Digikey (none) -> RMCF0805FT75R0-ND; MPN (none) -> RMCF0805FT75R0
- R204, R205, R206: Digikey (none) -> RMCF0805FT10K0-ND; MPN (none) -> RMCF0805FT10K0
- R208, R209: Digikey (none) -> RMCF0805FT1K50-ND; MPN (none) -> RMCF0805FT1K50
Changed lines of the file:
@@
 F 3 " ~" H 8400 4400 50  0001 C CNN
 F 4 "0" H 9350 4000 50  0001 C CNN "DNP"
+F 5 "609-5180-ND‎" H 9350 4000 50  0001 C CNN "Digikey"
+F 6 "ICD15S13E4GV00LF" H 9350 4000 50  0001 C CNN "MPN"
+F 7 "Amphenol" H 9350 4000 50  0001 C CNN "Manufacturer"
 	1    9350 4000
 	1    0    0    -1
@@
 F 3 "~" H 5500 3600 50  0001 C CNN
 F 4 "0" H 5500 3600 50  0001 C CNN "DNP"
+F 5 "RMCF0805FT75R0-ND" H 5500 3600 50  0001 C CNN "Digikey"
+F 6 "RMCF0805FT75R0" H 5500 3600 50  0001 C CNN "MPN"
 	1    5500 3600
 	0    1    1    0
@@
 F 3 "~" H 5500 3800 50  0001 C CNN
 F 4 "0" H 5500 3800 50  0001 C CNN "DNP"
+F 5 "RMCF0805FT75R0-ND" H 5500 3800 50  0001 C CNN "Digikey"
+F 6 "RMCF0805FT75R0" H 5500 3800 50  0001 C CNN "MPN"
 	1    5500 3800
 	0    1    1    0
@@
 F 3 "~" H 5500 4000 50  0001 C CNN
 F 4 "0" H 5500 4000 50  0001 C CNN "DNP"
+F 5 "RMCF0805FT75R0-ND" H 5500 4000 50  0001 C CNN "Digikey"
+F 6 "RMCF0805FT75R0" H 5500 4000 50  0001 C CNN "MPN"
 	1    5500 4000
 	0    1    1    0
@@
 F 3 "~" H 3250 4150 50  0001 C CNN
 F 4 "0" H 3250 4150 50  0001 C CNN "DNP"
+F 5 "RMCF0805FT10K0-ND" H 3250 4150 50  0001 C CNN "Digikey"
+F 6 "RMCF0805FT10K0" H 3250 4150 50  0001 C CNN "MPN"
 	1    3250 4150
 	-1   0    0    1
@@
 F 3 "~" H 3600 4150 50  0001 C CNN
 F 4 "0" H 3600 4150 50  0001 C CNN "DNP"
+F 5 "RMCF0805FT10K0-ND" H 3600 4150 50  0001 C CNN "Digikey"
+F 6 "RMCF0805FT10K0" H 3600 4150 50  0001 C CNN "MPN"
 	1    3600 4150
 	-1   0    0    1
@@
 F 3 "~" H 3950 4150 50  0001 C CNN
 F 4 "0" H 3950 4150 50  0001 C CNN "DNP"
+F 5 "RMCF0805FT10K0-ND" H 3950 4150 50  0001 C CNN "Digikey"
+F 6 "RMCF0805FT10K0" H 3950 4150 50  0001 C CNN "MPN"
 	1    3950 4150
 	-1   0    0    1
@@
 F 3 "~" H 9700 5050 50  0001 C CNN
 F 4 "0" H 9700 5050 50  0001 C CNN "DNP"
+F 5 "RMCF0805FT1K50-ND" H 9700 5050 50  0001 C CNN "Digikey"
+F 6 "RMCF0805FT1K50" H 9700 5050 50  0001 C CNN "MPN"
 	1    9700 5050
 	1    0    0    -1
@@
 F 3 "~" H 10050 5050 50  0001 C CNN
 F 4 "0" H 10050 5050 50  0001 C CNN "DNP"
+F 5 "RMCF0805FT1K50-ND" H 10050 5050 50  0001 C CNN "Digikey"
+F 6 "RMCF0805FT1K50" H 10050 5050 50  0001 C CNN "MPN"
 	1    10050 5050
 	1    0    0    -1
@@
 F 3 "~" H 7800 5000 50  0001 C CNN
 F 4 "0" H 7800 5000 50  0001 C CNN "DNP"
+F 5 "1276-1093-1-ND" H 7800 5000 50  0001 C CNN "Digikey"
+F 6 "CL21B224KBFNNNE" H 7800 5000 50  0001 C CNN "MPN"
+F 7 "Samsung" H 7800 5000 50  0001 C CNN "Manufacturer"
 	1    7800 5000
 	0    1    1    0
@@
 F 3 "~" H 9050 4750 50  0001 C CNN
 F 4 "1" H 9050 4750 50  0001 C CNN "DNP"
+F 5 "~" H 9050 4750 50  0001 C CNN "Digikey"
+F 6 "~" H 9050 4750 50  0001 C CNN "MPN"
+F 7 "~" H 9050 4750 50  0001 C CNN "Manufacturer"
 	1    9050 4750
 	0    -1   -1   0

Commit message: Marked no-fit parts
Parts:
- R201, R202, R203, R204, R205, R206, R208, R209: Manufacturer (none) -> Stackpole
Changed lines of the file:
@@
 F 5 "RMCF0805FT75R0-ND" H 5500 3600 50  0001 C CNN "Digikey"
 F 6 "RMCF0805FT75R0" H 5500 3600 50  0001 C CNN "MPN"
+F 7 "Stackpole" H 5500 3600 50  0001 C CNN "Manufacturer"
 	1    5500 3600
 	0    1    1    0
@@
 F 5 "RMCF0805FT75R0-ND" H 5500 3800 50  0001 C CNN "Digikey"
 F 6 "RMCF0805FT75R0" H 5500 3800 50  0001 C CNN "MPN"
+F 7 "Stackpole" H 5500 3800 50  0001 C CNN "Manufacturer"
 	1    5500 3800
 	0    1    1    0
@@
 F 5 "RMCF0805FT75R0-ND" H 5500 4000 50  0001 C CNN "Digikey"
 F 6 "RMCF0805FT75R0" H 5500 4000 50  0001 C CNN "MPN"
+F 7 "Stackpole" H 5500 4000 50  0001 C CNN "Manufacturer"
 	1    5500 4000
 	0    1    1    0
@@
 F 5 "RMCF0805FT10K0-ND" H 3250 4150 50  0001 C CNN "Digikey"
 F 6 "RMCF0805FT10K0" H 3250 4150 50  0001 C CNN "MPN"
+F 7 "Stackpole" H 3250 4150 50  0001 C CNN "Manufacturer"
 	1    3250 4150
 	-1   0    0    1
@@
 F 5 "RMCF0805FT10K0-ND" H 3600 4150 50  0001 C CNN "Digikey"
 F 6 "RMCF0805FT10K0" H 3600 4150 50  0001 C CNN "MPN"
+F 7 "Stackpole" H 3600 4150 50  0001 C CNN "Manufacturer"
 	1    3600 4150
 	-1   0    0    1
@@
 F 5 "RMCF0805FT10K0-ND" H 3950 4150 50  0001 C CNN "Digikey"
 F 6 "RMCF0805FT10K0" H 3950 4150 50  0001 C CNN "MPN"
+F 7 "Stackpole" H 3950 4150 50  0001 C CNN "Manufacturer"
 	1    3950 4150
 	-1   0    0    1
@@
 F 5 "RMCF0805FT1K50-ND" H 9700 5050 50  0001 C CNN "Digikey"
 F 6 "RMCF0805FT1K50" H 9700 5050 50  0001 C CNN "MPN"
+F 7 "Stackpole" H 9700 5050 50  0001 C CNN "Manufacturer"
 	1    9700 5050
 	1    0    0    -1
@@
 F 5 "RMCF0805FT1K50-ND" H 10050 5050 50  0001 C CNN "Digikey"
 F 6 "RMCF0805FT1K50" H 10050 5050 50  0001 C CNN "MPN"
+F 7 "Stackpole" H 10050 5050 50  0001 C CNN "Manufacturer"
 	1    10050 5050
 	1    0    0    -1
