File: Kicad/rtc.sch (KiCad schematic (older format))
At the start: 6 parts, among them U1201 MCP7940, Y1201 32,768 Hz

Commit message: Switch some of the radial THT Electrolytic caps for SMD MLCCs.
Also changed the STM32 for an LQFP-32 as it has a bigger pitch on the
pins.

The LQFP is easier to solder than the TSSOP, and the MLCC takes are
cheaper and take up less space.
Parts:
- BT1201: value Coin Cell -> CR2032
Changed lines of the file:
@@
 $Descr A4 11693 8268
 encoding utf-8
-Sheet 9 12
+Sheet 12 12
 Title "Neotron Common Hardware - Real Time Clock"
 Date "2021-01-01"
@@
 P 6300 3400
 F 0 "BT1201" H 6418 3496 50  0000 L CNN
-F 1 "Coin Cell" H 6418 3405 50  0000 L CNN
+F 1 "CR2032" H 6418 3405 50  0000 L CNN
 F 2 "Neotron-Common-Hardware:BatteryHolder_Keystone_103_1x20mm" V 6300 3460 50  0001 C CNN
 F 3 "http://keyelco.com/userAssets/file/M65p3.pdf" V 6300 3460 50  0001 C CNN

Commit message: Added 12-bit video DAC.
Also had to change footprints to suit Kicad 5.1.9
Parts:
- C87: renamed from C1202; footprint Capacitor_SMD:C_0805_2012Metric_Pad1.15x1.40mm_HandSolder -> Capacitor_SMD:C_0805_2012Metric_Pad1.18x1.45mm_HandSolder
- C88: renamed from C1203; footprint Capacitor_SMD:C_0805_2012Metric_Pad1.15x1.40mm_HandSolder -> Capacitor_SMD:C_0805_2012Metric_Pad1.18x1.45mm_HandSolder
- C89: renamed from C1201; footprint Capacitor_SMD:C_0805_2012Metric_Pad1.15x1.40mm_HandSolder -> Capacitor_SMD:C_0805_2012Metric_Pad1.18x1.45mm_HandSolder
- renumbered BT1201 to BT1, U1201 to U18, Y1201 to Y4
Changed lines of the file:
@@
 $Descr A4 11693 8268
 encoding utf-8
-Sheet 12 12
+Sheet 12 16
 Title "Neotron Common Hardware - Real Time Clock"
 Date "2021-01-01"
@@
 I2C_SCL
 $Comp
-L Timer:MCP7940N-xP U1201
+L Timer:MCP7940N-xP U18
 U 1 1 5E0F47D7
 P 4075 2675
-F 0 "U1201" H 4375 3025 50  0000 C CNN
+F 0 "U18" H 4375 3025 50  0000 C CNN
 F 1 "MCP7940" H 3675 3025 50  0000 C CNN
 F 2 "Package_SO:SOIC-8_3.9x4.9mm_P1.27mm" H 4075 2675 50  0001 C CNN
@@
 $EndComp
 $Comp
-L Device:Battery_Cell BT1201
+L Device:Battery_Cell BT1
 U 1 1 5E0F507E
 P 6300 3400
-F 0 "BT1201" H 6418 3496 50  0000 L CNN
+F 0 "BT1" H 6418 3496 50  0000 L CNN
 F 1 "CR2032" H 6418 3405 50  0000 L CNN
 F 2 "Neotron-Common-Hardware:BatteryHolder_Keystone_103_1x20mm" V 6300 3460 50  0001 C CNN
@@
 AR Path="/5DF1D0B0/5E0203C5" Ref="#PWR?"  Part="1"
 AR Path="/5DF66898/5E0203C5" Ref="#PWR?"  Part="1"
-AR Path="/5FEF404D/5E0203C5" Ref="#PWR01204"  Part="1"
-F 0 "#PWR01204" H 7050 2950 50  0001 C CNN
+AR Path="/5FEF404D/5E0203C5" Ref="#PWR0202"  Part="1"
+F 0 "#PWR0202" H 7050 2950 50  0001 C CNN
 F 1 "+3V3" H 7050 3250 50  0000 C CNN
 F 2 "" H 7050 3100 50  0001 C CNN
@@
 AR Path="/5DF1D0B0/5E0203CB" Ref="C?"  Part="1"
 AR Path="/5DF66898/5E0203CB" Ref="C?"  Part="1"
-AR Path="/5FEF404D/5E0203CB" Ref="C1201"  Part="1"
-F 0 "C1201" H 7165 3396 50  0000 L CNN
+AR Path="/5FEF404D/5E0203CB" Ref="C89"  Part="1"
+F 0 "C89" H 7165 3396 50  0000 L CNN
 F 1 "100n" H 7165 3305 50  0000 L CNN
-F 2 "Capacitor_SMD:C_0805_2012Metric_Pad1.15x1.40mm_HandSolder" H 7088 3200 50  0001 C CNN
+F 2 "Capacitor_SMD:C_0805_2012Metric_Pad1.18x1.45mm_HandSolder" H 7088 3200 50  0001 C CNN
 F 3 "~" H 7050 3350 50  0001 C CNN
 F 4 "Vishay" H 0   0   50  0001 C CNN "Manufacturer"
@@
 AR Path="/5DF1D0B0/5E0203D1" Ref="#PWR?"  Part="1"
 AR Path="/5DF66898/5E0203D1" Ref="#PWR?"  Part="1"
-AR Path="/5FEF404D/5E0203D1" Ref="#PWR01207"  Part="1"
-F 0 "#PWR01207" H 7050 3350 50  0001 C CNN
+AR Path="/5FEF404D/5E0203D1" Ref="#PWR0203"  Part="1"
+F 0 "#PWR0203" H 7050 3350 50  0001 C CNN
 F 1 "GND" H 7050 3450 50  0000 C CNN
 F 2 "" H 7050 3600 50  0001 C CNN
@@
 NoConn ~ 3675 2775
 $Comp
-L power:+3V3 #PWR01201
+L power:+3V3 #PWR0195
 U 1 1 5E027CB5
 P 3975 2225
-F 0 "#PWR01201" H 3975 2075 50  0001 C CNN
+F 0 "#PWR0195" H 3975 2075 50  0001 C CNN
 F 1 "+3V3" H 3975 2375 50  0000 C CNN
 F 2 "" H 3975 2225 50  0001 C CNN
@@
 AR Path="/5DF1D0B0/5E02823D" Ref="#PWR?"  Part="1"
 AR Path="/5DF66898/5E02823D" Ref="#PWR?"  Part="1"
-AR Path="/5FEF404D/5E02823D" Ref="#PWR01205"  Part="1"
-F 0 "#PWR01205" H 4075 2925 50  0001 C CNN
+AR Path="/5FEF404D/5E02823D" Ref="#PWR0196"  Part="1"
+F 0 "#PWR0196" H 4075 2925 50  0001 C CNN
 F 1 "GND" H 4075 3025 50  0000 C CNN
 F 2 "" H 4075 3175 50  0001 C CNN
@@
 $EndComp
 $Comp
-L Device:Crystal Y1201
+L Device:Crystal Y4
 U 1 1 5E028A76
 P 5025 3000
-F 0 "Y1201" H 4925 2850 50  0000 L CNN
+F 0 "Y4" H 4925 2850 50  0000 L CNN
 F 1 "32,768 Hz" H 4825 3150 50  0000 L CNN
 F 2 "Crystal:Crystal_DS26_D2.0mm_L6.0mm_Horizontal" H 5025 3000 50  0001 C CNN
@@
 	4075 3075 4075 3175
 $Comp
-L power:+BATT #PWR01202
+L power:+BATT #PWR0197
 U 1 1 5E0292FA
 P 4275 2225
-F 0 "#PWR01202" H 4275 2075 50  0001 C CNN
+F 0 "#PWR0197" H 4275 2075 50  0001 C CNN
 F 1 "+BATT" H 4275 2375 50  0000 C CNN
 F 2 "" H 4275 2225 50  0001 C CNN
@@
 	4175 2225 4275 2225
 $Comp
-L power:+BATT #PWR01203
+L power:+BATT #PWR0200
 U 1 1 5E029FFB
 P 6300 3100
-F 0 "#PWR01203" H 6300 2950 50  0001 C CNN
+F 0 "#PWR0200" H 6300 2950 50  0001 C CNN
 F 1 "+BATT" H 6300 3250 50  0000 C CNN
 F 2 "" H 6300 3100 50  0001 C CNN
@@
 AR Path="/5DF1D0B0/5E02A51C" Ref="#PWR?"  Part="1"
 AR Path="/5DF66898/5E02A51C" Ref="#PWR?"  Part="1"
-AR Path="/5FEF404D/5E02A51C" Ref="#PWR01206"  Part="1"
-F 0 "#PWR01206" H 6300 3350 50  0001 C CNN
+AR Path="/5FEF404D/5E02A51C" Ref="#PWR0201"  Part="1"
+F 0 "#PWR0201" H 6300 3350 50  0001 C CNN
 F 1 "GND" H 6300 3450 50  0000 C CNN
 F 2 "" H 6300 3600 50  0001 C CNN
@@
 	6300 3500 6300 3600
 $Comp
-L Device:C C1203
+L Device:C C88
 U 1 1 5E02C5CE
 P 5350 3500
-F 0 "C1203" H 5465 3546 50  0000 L CNN
+F 0 "C88" H 5465 3546 50  0000 L CNN
 F 1 "6p" H 5465 3455 50  0000 L CNN
-F 2 "Capacitor_SMD:C_0805_2012Metric_Pad1.15x1.40mm_HandSolder" H 5388 3350 50  0001 C CNN
+F 2 "Capacitor_SMD:C_0805_2012Metric_Pad1.18x1.45mm_HandSolder" H 5388 3350 50  0001 C CNN
 F 3 "~" H 5350 3500 50  0001 C CNN
 F 4 "Yageo" H -200 550 50  0001 C CNN "Manufacturer"
@@
 $EndComp
 $Comp
-L Device:C C1202
+L Device:C C87
 U 1 1 5E02CC31
 P 4700 3500
-F 0 "C1202" H 4815 3546 50  0000 L CNN
+F 0 "C87" H 4815 3546 50  0000 L CNN
 F 1 "6p" H 4815 3455 50  0000 L CNN
-F 2 "Capacitor_SMD:C_0805_2012Metric_Pad1.15x1.40mm_HandSolder" H 4738 3350 50  0001 C CNN
+F 2 "Capacitor_SMD:C_0805_2012Metric_Pad1.18x1.45mm_HandSolder" H 4738 3350 50  0001 C CNN
 F 3 "~" H 4700 3500 50  0001 C CNN
 F 4 "Yageo" H -850 -250 50  0001 C CNN "Manufacturer"
@@
 AR Path="/5DF1D0B0/5E02D069" Ref="#PWR?"  Part="1"
 AR Path="/5DF66898/5E02D069" Ref="#PWR?"  Part="1"
-AR Path="/5FEF404D/5E02D069" Ref="#PWR01208"  Part="1"
-F 0 "#PWR01208" H 4700 3450 50  0001 C CNN
+AR Path="/5FEF404D/5E02D069" Ref="#PWR0198"  Part="1"
+F 0 "#PWR0198" H 4700 3450 50  0001 C CNN
 F 1 "GND" H 4700 3550 50  0000 C CNN
 F 2 "" H 4700 3700 50  0001 C CNN
@@
 	4700 3650 4700 3700
 $Comp
-L power:PWR_FLAG #FLG01201
+L power:PWR_FLAG #FLG08
 U 1 1 5E3BA2C7
 P 6300 3150
-F 0 "#FLG01201" H 6300 3225 50  0001 C CNN
+F 0 "#FLG08" H 6300 3225 50  0001 C CNN
 F 1 "PWR_FLAG" V 6300 3278 50  0000 L CNN
 F 2 "" H 6300 3150 50  0001 C CNN
@@
 AR Path="/5DF1D0B0/5FF0B56D" Ref="#PWR?"  Part="1"
 AR Path="/5DF66898/5FF0B56D" Ref="#PWR?"  Part="1"
-AR Path="/5FEF404D/5FF0B56D" Ref="#PWR01209"  Part="1"
-F 0 "#PWR01209" H 5350 3450 50  0001 C CNN
+AR Path="/5FEF404D/5FF0B56D" Ref="#PWR0199"  Part="1"
+F 0 "#PWR0199" H 5350 3450 50  0001 C CNN
 F 1 "GND" H 5350 3550 50  0000 C CNN
 F 2 "" H 5350 3700 50  0001 C CNN

Commit message: Add 4-bit Video DAC, and re-wire BMC.
Now the BMC is an SPI device, and has a four-wire UART.
Parts:
- renumbered BT1 to BT1201, C87 to C1201, C88 to C1202, C89 to C1203, U18 to U1201, Y4 to Y1201
Changed lines of the file:
@@
 Sheet 12 16
 Title "Neotron Common Hardware - Real Time Clock"
-Date "2021-01-01"
+Date "2021-04-02"
 Rev "[Uncontrolled]"
 Comp "https://neotron-compute.github.io/"
@@
 I2C_SCL
 $Comp
-L Timer:MCP7940N-xP U18
+L Timer:MCP7940N-xP U1201
 U 1 1 5E0F47D7
 P 4075 2675
-F 0 "U18" H 4375 3025 50  0000 C CNN
+F 0 "U1201" H 4375 3025 50  0000 C CNN
 F 1 "MCP7940" H 3675 3025 50  0000 C CNN
 F 2 "Package_SO:SOIC-8_3.9x4.9mm_P1.27mm" H 4075 2675 50  0001 C CNN
@@
 $EndComp
 $Comp
-L Device:Battery_Cell BT1
+L Device:Battery_Cell BT1201
 U 1 1 5E0F507E
 P 6300 3400
-F 0 "BT1" H 6418 3496 50  0000 L CNN
+F 0 "BT1201" H 6418 3496 50  0000 L CNN
 F 1 "CR2032" H 6418 3405 50  0000 L CNN
 F 2 "Neotron-Common-Hardware:BatteryHolder_Keystone_103_1x20mm" V 6300 3460 50  0001 C CNN
@@
 AR Path="/5DF1D0B0/5E0203C5" Ref="#PWR?"  Part="1"
 AR Path="/5DF66898/5E0203C5" Ref="#PWR?"  Part="1"
-AR Path="/5FEF404D/5E0203C5" Ref="#PWR0202"  Part="1"
-F 0 "#PWR0202" H 7050 2950 50  0001 C CNN
+AR Path="/5FEF404D/5E0203C5" Ref="#PWR01208"  Part="1"
+F 0 "#PWR01208" H 7050 2950 50  0001 C CNN
 F 1 "+3V3" H 7050 3250 50  0000 C CNN
 F 2 "" H 7050 3100 50  0001 C CNN
@@
 AR Path="/5DF1D0B0/5E0203CB" Ref="C?"  Part="1"
 AR Path="/5DF66898/5E0203CB" Ref="C?"  Part="1"
-AR Path="/5FEF404D/5E0203CB" Ref="C89"  Part="1"
-F 0 "C89" H 7165 3396 50  0000 L CNN
+AR Path="/5FEF404D/5E0203CB" Ref="C1203"  Part="1"
+F 0 "C1203" H 7165 3396 50  0000 L CNN
 F 1 "100n" H 7165 3305 50  0000 L CNN
 F 2 "Capacitor_SMD:C_0805_2012Metric_Pad1.18x1.45mm_HandSolder" H 7088 3200 50  0001 C CNN
@@
 AR Path="/5DF1D0B0/5E0203D1" Ref="#PWR?"  Part="1"
 AR Path="/5DF66898/5E0203D1" Ref="#PWR?"  Part="1"
-AR Path="/5FEF404D/5E0203D1" Ref="#PWR0203"  Part="1"
-F 0 "#PWR0203" H 7050 3350 50  0001 C CNN
+AR Path="/5FEF404D/5E0203D1" Ref="#PWR01209"  Part="1"
+F 0 "#PWR01209" H 7050 3350 50  0001 C CNN
 F 1 "GND" H 7050 3450 50  0000 C CNN
 F 2 "" H 7050 3600 50  0001 C CNN
@@
 NoConn ~ 3675 2775
 $Comp
-L power:+3V3 #PWR0195
+L power:+3V3 #PWR01201
 U 1 1 5E027CB5
 P 3975 2225
-F 0 "#PWR0195" H 3975 2075 50  0001 C CNN
+F 0 "#PWR01201" H 3975 2075 50  0001 C CNN
 F 1 "+3V3" H 3975 2375 50  0000 C CNN
 F 2 "" H 3975 2225 50  0001 C CNN
@@
 AR Path="/5DF1D0B0/5E02823D" Ref="#PWR?"  Part="1"
 AR Path="/5DF66898/5E02823D" Ref="#PWR?"  Part="1"
-AR Path="/5FEF404D/5E02823D" Ref="#PWR0196"  Part="1"
-F 0 "#PWR0196" H 4075 2925 50  0001 C CNN
+AR Path="/5FEF404D/5E02823D" Ref="#PWR01202"  Part="1"
+F 0 "#PWR01202" H 4075 2925 50  0001 C CNN
 F 1 "GND" H 4075 3025 50  0000 C CNN
 F 2 "" H 4075 3175 50  0001 C CNN
@@
 $EndComp
 $Comp
-L Device:Crystal Y4
+L Device:Crystal Y1201
 U 1 1 5E028A76
 P 5025 3000
-F 0 "Y4" H 4925 2850 50  0000 L CNN
+F 0 "Y1201" H 4925 2850 50  0000 L CNN
 F 1 "32,768 Hz" H 4825 3150 50  0000 L CNN
 F 2 "Crystal:Crystal_DS26_D2.0mm_L6.0mm_Horizontal" H 5025 3000 50  0001 C CNN
@@
 	4075 3075 4075 3175
 $Comp
-L power:+BATT #PWR0197
+L power:+BATT #PWR01203
 U 1 1 5E0292FA
 P 4275 2225
-F 0 "#PWR0197" H 4275 2075 50  0001 C CNN
+F 0 "#PWR01203" H 4275 2075 50  0001 C CNN
 F 1 "+BATT" H 4275 2375 50  0000 C CNN
 F 2 "" H 4275 2225 50  0001 C CNN
@@
 	4175 2225 4275 2225
 $Comp
-L power:+BATT #PWR0200
+L power:+BATT #PWR01206
 U 1 1 5E029FFB
 P 6300 3100
-F 0 "#PWR0200" H 6300 2950 50  0001 C CNN
+F 0 "#PWR01206" H 6300 2950 50  0001 C CNN
 F 1 "+BATT" H 6300 3250 50  0000 C CNN
 F 2 "" H 6300 3100 50  0001 C CNN
@@
 AR Path="/5DF1D0B0/5E02A51C" Ref="#PWR?"  Part="1"
 AR Path="/5DF66898/5E02A51C" Ref="#PWR?"  Part="1"
-AR Path="/5FEF404D/5E02A51C" Ref="#PWR0201"  Part="1"
-F 0 "#PWR0201" H 6300 3350 50  0001 C CNN
+AR Path="/5FEF404D/5E02A51C" Ref="#PWR01207"  Part="1"
+F 0 "#PWR01207" H 6300 3350 50  0001 C CNN
 F 1 "GND" H 6300 3450 50  0000 C CNN
 F 2 "" H 6300 3600 50  0001 C CNN
@@
 	6300 3500 6300 3600
 $Comp
-L Device:C C88
+L Device:C C1202
 U 1 1 5E02C5CE
 P 5350 3500
-F 0 "C88" H 5465 3546 50  0000 L CNN
+F 0 "C1202" H 5465 3546 50  0000 L CNN
 F 1 "6p" H 5465 3455 50  0000 L CNN
 F 2 "Capacitor_SMD:C_0805_2012Metric_Pad1.18x1.45mm_HandSolder" H 5388 3350 50  0001 C CNN
@@
 $EndComp
 $Comp
-L Device:C C87
+L Device:C C1201
 U 1 1 5E02CC31
 P 4700 3500
-F 0 "C87" H 4815 3546 50  0000 L CNN
+F 0 "C1201" H 4815 3546 50  0000 L CNN
 F 1 "6p" H 4815 3455 50  0000 L CNN
 F 2 "Capacitor_SMD:C_0805_2012Metric_Pad1.18x1.45mm_HandSolder" H 4738 3350 50  0001 C CNN
@@
 AR Path="/5DF1D0B0/5E02D069" Ref="#PWR?"  Part="1"
 AR Path="/5DF66898/5E02D069" Ref="#PWR?"  Part="1"
-AR Path="/5FEF404D/5E02D069" Ref="#PWR0198"  Part="1"
-F 0 "#PWR0198" H 4700 3450 50  0001 C CNN
+AR Path="/5FEF404D/5E02D069" Ref="#PWR01204"  Part="1"
+F 0 "#PWR01204" H 4700 3450 50  0001 C CNN
 F 1 "GND" H 4700 3550 50  0000 C CNN
 F 2 "" H 4700 3700 50  0001 C CNN
@@
 	4700 3650 4700 3700
 $Comp
-L power:PWR_FLAG #FLG08
+L power:PWR_FLAG #FLG01201
 U 1 1 5E3BA2C7
 P 6300 3150
-F 0 "#FLG08" H 6300 3225 50  0001 C CNN
+F 0 "#FLG01201" H 6300 3225 50  0001 C CNN
 F 1 "PWR_FLAG" V 6300 3278 50  0000 L CNN
 F 2 "" H 6300 3150 50  0001 C CNN
@@
 AR Path="/5DF1D0B0/5FF0B56D" Ref="#PWR?"  Part="1"
 AR Path="/5DF66898/5FF0B56D" Ref="#PWR?"  Part="1"
-AR Path="/5FEF404D/5FF0B56D" Ref="#PWR0199"  Part="1"
-F 0 "#PWR0199" H 5350 3450 50  0001 C CNN
+AR Path="/5FEF404D/5FF0B56D" Ref="#PWR01205"  Part="1"
+F 0 "#PWR01205" H 5350 3450 50  0001 C CNN
 F 1 "GND" H 5350 3550 50  0000 C CNN
 F 2 "" H 5350 3700 50  0001 C CNN

Commit message: Tidy up part nos and swapped I2C/UART on BMC.
Mark all resistors as 1% if not specified.
Added some Mouser part numbers.
BMC can now be programmed over UART.
Parts:
- C1201, C1202: Mouser (none) -> 603-CC805DRNPO9BN6R0
- C1203: Mouser (none) -> 594-K104K15X7RF5TL2
- U1201: Mouser (none) -> 579-MCP7940NT-I/SN
- Y1201: Mouser (none) -> CFS-20632768DZBB
Changed lines of the file:
@@
 F 6 "MCP7940NT-I/SN" H 4075 2675 50  0001 C CNN "MPN"
 F 7 "MCP7940NT-I/SNCT-ND" H 4075 2675 50  0001 C CNN "Digikey"
+F 8 "579-MCP7940NT-I/SN" H 4075 2675 50  0001 C CNN "Mouser"
 	1    4075 2675
 	1    0    0    -1
@@
 F 6 "BC1150CT-ND" H 7050 3350 50  0001 C CNN "Digikey"
 F 7 "K104K15X7RF5TL2" H 7050 3350 50  0001 C CNN "MPN"
+F 8 "594-K104K15X7RF5TL2" H 7050 3350 50  0001 C CNN "Mouser"
 	1    7050 3350
 	1    0    0    -1
@@
 F 6 "CFS-20632768DZBB " H 5025 3000 50  0001 C CNN "MPN"
 F 7 "300-8301-ND" H 5025 3000 50  0001 C CNN "Digikey"
+F 8 "CFS-20632768DZBB" H 5025 3000 50  0001 C CNN "Mouser"
 	1    5025 3000
 	-1   0    0    1
@@
 F 6 "CC0805DRNPO9BN6R0" H 5350 3500 50  0001 C CNN "MPN"
 F 7 "311-1095-1-ND" H 5350 3500 50  0001 C CNN "Digikey"
+F 8 "603-CC805DRNPO9BN6R0" H 5350 3500 50  0001 C CNN "Mouser"
 	1    5350 3500
 	1    0    0    -1
@@
 F 6 "CC0805DRNPO9BN6R0" H 4700 3500 50  0001 C CNN "MPN"
 F 7 "311-1095-1-ND" H 4700 3500 50  0001 C CNN "Digikey"
+F 8 "603-CC805DRNPO9BN6R0" H 4700 3500 50  0001 C CNN "Mouser"
 	1    4700 3500
 	1    0    0    -1

Commit message: Changes to BMC
* Swapped BUTTON_PWR and SYS_RESET to avoid DRC issue
* Split PSU and BMC into two separate sheets
* Swapped some pins on the STM32 to make it compatible with more
alternatives
Parts:
- renumbered BT1201 to BT1101, C1201 to C1101, C1202 to C1102, C1203 to C1103, U1201 to U1101, Y1201 to Y1101
Changed lines of the file:
@@
 $Descr A4 11693 8268
 encoding utf-8
-Sheet 12 16
+Sheet 12 17
 Title "Neotron Common Hardware - Real Time Clock"
 Date "2021-04-02"
@@
 I2C_SCL
 $Comp
-L Timer:MCP7940N-xP U1201
+L Timer:MCP7940N-xP U1101
 U 1 1 5E0F47D7
 P 4075 2675
-F 0 "U1201" H 4375 3025 50  0000 C CNN
+F 0 "U1101" H 4375 3025 50  0000 C CNN
 F 1 "MCP7940" H 3675 3025 50  0000 C CNN
 F 2 "Package_SO:SOIC-8_3.9x4.9mm_P1.27mm" H 4075 2675 50  0001 C CNN
@@
 $EndComp
 $Comp
-L Device:Battery_Cell BT1201
+L Device:Battery_Cell BT1101
 U 1 1 5E0F507E
 P 6300 3400
-F 0 "BT1201" H 6418 3496 50  0000 L CNN
+F 0 "BT1101" H 6418 3496 50  0000 L CNN
 F 1 "CR2032" H 6418 3405 50  0000 L CNN
 F 2 "Neotron-Common-Hardware:BatteryHolder_Keystone_103_1x20mm" V 6300 3460 50  0001 C CNN
@@
 AR Path="/5DF1D0B0/5E0203C5" Ref="#PWR?"  Part="1"
 AR Path="/5DF66898/5E0203C5" Ref="#PWR?"  Part="1"
-AR Path="/5FEF404D/5E0203C5" Ref="#PWR01208"  Part="1"
-F 0 "#PWR01208" H 7050 2950 50  0001 C CNN
+AR Path="/5FEF404D/5E0203C5" Ref="#PWR01108"  Part="1"
+F 0 "#PWR01108" H 7050 2950 50  0001 C CNN
 F 1 "+3V3" H 7050 3250 50  0000 C CNN
 F 2 "" H 7050 3100 50  0001 C CNN
@@
 AR Path="/5DF1D0B0/5E0203CB" Ref="C?"  Part="1"
 AR Path="/5DF66898/5E0203CB" Ref="C?"  Part="1"
-AR Path="/5FEF404D/5E0203CB" Ref="C1203"  Part="1"
-F 0 "C1203" H 7165 3396 50  0000 L CNN
+AR Path="/5FEF404D/5E0203CB" Ref="C1103"  Part="1"
+F 0 "C1103" H 7165 3396 50  0000 L CNN
 F 1 "100n" H 7165 3305 50  0000 L CNN
 F 2 "Capacitor_SMD:C_0805_2012Metric_Pad1.18x1.45mm_HandSolder" H 7088 3200 50  0001 C CNN
@@
 AR Path="/5DF1D0B0/5E0203D1" Ref="#PWR?"  Part="1"
 AR Path="/5DF66898/5E0203D1" Ref="#PWR?"  Part="1"
-AR Path="/5FEF404D/5E0203D1" Ref="#PWR01209"  Part="1"
-F 0 "#PWR01209" H 7050 3350 50  0001 C CNN
+AR Path="/5FEF404D/5E0203D1" Ref="#PWR01109"  Part="1"
+F 0 "#PWR01109" H 7050 3350 50  0001 C CNN
 F 1 "GND" H 7050 3450 50  0000 C CNN
 F 2 "" H 7050 3600 50  0001 C CNN
@@
 NoConn ~ 3675 2775
 $Comp
-L power:+3V3 #PWR01201
+L power:+3V3 #PWR01101
 U 1 1 5E027CB5
 P 3975 2225
-F 0 "#PWR01201" H 3975 2075 50  0001 C CNN
+F 0 "#PWR01101" H 3975 2075 50  0001 C CNN
 F 1 "+3V3" H 3975 2375 50  0000 C CNN
 F 2 "" H 3975 2225 50  0001 C CNN
@@
 AR Path="/5DF1D0B0/5E02823D" Ref="#PWR?"  Part="1"
 AR Path="/5DF66898/5E02823D" Ref="#PWR?"  Part="1"
-AR Path="/5FEF404D/5E02823D" Ref="#PWR01202"  Part="1"
-F 0 "#PWR01202" H 4075 2925 50  0001 C CNN
+AR Path="/5FEF404D/5E02823D" Ref="#PWR01102"  Part="1"
+F 0 "#PWR01102" H 4075 2925 50  0001 C CNN
 F 1 "GND" H 4075 3025 50  0000 C CNN
 F 2 "" H 4075 3175 50  0001 C CNN
@@
 $EndComp
 $Comp
-L Device:Crystal Y1201
+L Device:Crystal Y1101
 U 1 1 5E028A76
 P 5025 3000
-F 0 "Y1201" H 4925 2850 50  0000 L CNN
+F 0 "Y1101" H 4925 2850 50  0000 L CNN
 F 1 "32,768 Hz" H 4825 3150 50  0000 L CNN
 F 2 "Crystal:Crystal_DS26_D2.0mm_L6.0mm_Horizontal" H 5025 3000 50  0001 C CNN
@@
 	4075 3075 4075 3175
 $Comp
-L power:+BATT #PWR01203
+L power:+BATT #PWR01103
 U 1 1 5E0292FA
 P 4275 2225
-F 0 "#PWR01203" H 4275 2075 50  0001 C CNN
+F 0 "#PWR01103" H 4275 2075 50  0001 C CNN
 F 1 "+BATT" H 4275 2375 50  0000 C CNN
 F 2 "" H 4275 2225 50  0001 C CNN
@@
 	4175 2225 4275 2225
 $Comp
-L power:+BATT #PWR01206
+L power:+BATT #PWR01106
 U 1 1 5E029FFB
 P 6300 3100
-F 0 "#PWR01206" H 6300 2950 50  0001 C CNN
+F 0 "#PWR01106" H 6300 2950 50  0001 C CNN
 F 1 "+BATT" H 6300 3250 50  0000 C CNN
 F 2 "" H 6300 3100 50  0001 C CNN
@@
 AR Path="/5DF1D0B0/5E02A51C" Ref="#PWR?"  Part="1"
 AR Path="/5DF66898/5E02A51C" Ref="#PWR?"  Part="1"
-AR Path="/5FEF404D/5E02A51C" Ref="#PWR01207"  Part="1"
-F 0 "#PWR01207" H 6300 3350 50  0001 C CNN
+AR Path="/5FEF404D/5E02A51C" Ref="#PWR01107"  Part="1"
+F 0 "#PWR01107" H 6300 3350 50  0001 C CNN
 F 1 "GND" H 6300 3450 50  0000 C CNN
 F 2 "" H 6300 3600 50  0001 C CNN
@@
 	6300 3500 6300 3600
 $Comp
-L Device:C C1202
+L Device:C C1102
 U 1 1 5E02C5CE
 P 5350 3500
-F 0 "C1202" H 5465 3546 50  0000 L CNN
+F 0 "C1102" H 5465 3546 50  0000 L CNN
 F 1 "6p" H 5465 3455 50  0000 L CNN
 F 2 "Capacitor_SMD:C_0805_2012Metric_Pad1.18x1.45mm_HandSolder" H 5388 3350 50  0001 C CNN
@@
 $EndComp
 $Comp
-L Device:C C1201
+L Device:C C1101
 U 1 1 5E02CC31
 P 4700 3500
-F 0 "C1201" H 4815 3546 50  0000 L CNN
+F 0 "C1101" H 4815 3546 50  0000 L CNN
 F 1 "6p" H 4815 3455 50  0000 L CNN
 F 2 "Capacitor_SMD:C_0805_2012Metric_Pad1.18x1.45mm_HandSolder" H 4738 3350 50  0001 C CNN
@@
 AR Path="/5DF1D0B0/5E02D069" Ref="#PWR?"  Part="1"
 AR Path="/5DF66898/5E02D069" Ref="#PWR?"  Part="1"
-AR Path="/5FEF404D/5E02D069" Ref="#PWR01204"  Part="1"
-F 0 "#PWR01204" H 4700 3450 50  0001 C CNN
+AR Path="/5FEF404D/5E02D069" Ref="#PWR01104"  Part="1"
+F 0 "#PWR01104" H 4700 3450 50  0001 C CNN
 F 1 "GND" H 4700 3550 50  0000 C CNN
 F 2 "" H 4700 3700 50  0001 C CNN
@@
 	4700 3650 4700 3700
 $Comp
-L power:PWR_FLAG #FLG01201
+L power:PWR_FLAG #FLG01101
 U 1 1 5E3BA2C7
 P 6300 3150
-F 0 "#FLG01201" H 6300 3225 50  0001 C CNN
+F 0 "#FLG01101" H 6300 3225 50  0001 C CNN
 F 1 "PWR_FLAG" V 6300 3278 50  0000 L CNN
 F 2 "" H 6300 3150 50  0001 C CNN
@@
 AR Path="/5DF1D0B0/5FF0B56D" Ref="#PWR?"  Part="1"
 AR Path="/5DF66898/5FF0B56D" Ref="#PWR?"  Part="1"
-AR Path="/5FEF404D/5FF0B56D" Ref="#PWR01205"  Part="1"
-F 0 "#PWR01205" H 5350 3450 50  0001 C CNN
+AR Path="/5FEF404D/5FF0B56D" Ref="#PWR01105"  Part="1"
+F 0 "#PWR01105" H 5350 3450 50  0001 C CNN
 F 1 "GND" H 5350 3550 50  0000 C CNN
 F 2 "" H 5350 3700 50  0001 C CNN

Commit message: Remove more errant spaces.
Parts:
- Y1101: MPN CFS-20632768DZBB -> CFS-20632768DZBB
Changed lines of the file:
@@
 F 4 "Citizen" H 5025 3000 50  0001 C CNN "Manufacturer"
 F 5 "0" H 5025 3000 50  0001 C CNN "DNP"
-F 6 "CFS-20632768DZBB " H 5025 3000 50  0001 C CNN "MPN"
+F 6 "CFS-20632768DZBB" H 5025 3000 50  0001 C CNN "MPN"
 F 7 "300-8301-ND" H 5025 3000 50  0001 C CNN "Digikey"
 F 8 "CFS-20632768DZBB" H 5025 3000 50  0001 C CNN "Mouser"
