File: Kicad/rtc.sch (KiCad schematic (older format))
At the start: 6 parts, among them U1101 MCP7940, Y1101 32,768 Hz

Commit message: Brought in sheets from Neotron Pico.
Also includes DB15HD and PSU 3D models.
Parts:
- C1101, C1102: value 6p -> 6pF; LCSC Part# (none) -> C67560; Voltage (none) -> C0G
- C1103: value 100n -> 100nF; Digikey BC1150CT-ND -> (none); LCSC Part# (none) -> C49678; MPN K104K15X7RF5TL2 -> CPL-CAP-X7R-0805-100NF-50V; Manufacturer Vishay -> CPL; Mouser 594-K104K15X7RF5TL2 -> (none)
- U1101: value MCP7940 -> MCP7940N; footprint Package_SO:SOIC-8_3.9x4.9mm_P1.27mm -> Package_DIP:DIP-8_W7.62mm; Digikey MCP7940NT-I/SNCT-ND -> MCP7940N-I/P-ND; LCSC Part# (none) -> C51106; MPN MCP7940NT-I/SN -> MCP7940N-I/P; Mouser 579-MCP7940NT-I/SN -> 579-MCP7940N-I/P
Changed lines of the file:
@@
 $Descr A4 11693 8268
 encoding utf-8
-Sheet 11 17
-Title "Neotron Common Hardware - Real Time Clock"
-Date "2021-04-02"
+Sheet 11 18
+Title "Neotron Common Hardware"
+Date "2021-06-18"
 Rev "[Uncontrolled]"
 Comp "https://neotron-compute.github.io/"
@@
 P 4075 2675
 F 0 "U1101" H 4375 3025 50  0000 C CNN
-F 1 "MCP7940" H 3675 3025 50  0000 C CNN
-F 2 "Package_SO:SOIC-8_3.9x4.9mm_P1.27mm" H 4075 2675 50  0001 C CNN
+F 1 "MCP7940N" H 3675 3025 50  0000 C CNN
+F 2 "Package_DIP:DIP-8_W7.62mm" H 4075 2675 50  0001 C CNN
 F 3 "http://ww1.microchip.com/downloads/en/DeviceDoc/20005010F.pdf" H 4075 2675 50  0001 C CNN
 F 4 "Microchip" H 4075 2675 50  0001 C CNN "Manufacturer"
 F 5 "0" H 4075 2675 50  0001 C CNN "DNP"
-F 6 "MCP7940NT-I/SN" H 4075 2675 50  0001 C CNN "MPN"
-F 7 "MCP7940NT-I/SNCT-ND" H 4075 2675 50  0001 C CNN "Digikey"
-F 8 "579-MCP7940NT-I/SN" H 4075 2675 50  0001 C CNN "Mouser"
+F 6 "MCP7940N-I/P" H 4075 2675 50  0001 C CNN "MPN"
+F 7 "MCP7940N-I/P-ND" H 4075 2675 50  0001 C CNN "Digikey"
+F 8 "579-MCP7940N-I/P" H 4075 2675 50  0001 C CNN "Mouser"
+F 9 "C51106" H 4075 2675 50  0001 C CNN "LCSC Part#"
 	1    4075 2675
 	1    0    0    -1
@@
 F 6 "103" H 6300 3400 50  0001 C CNN "MPN"
 F 7 "36-103-ND" H 6300 3400 50  0001 C CNN "Digikey"
+F 8 "~" H 6300 3400 50  0001 C CNN "LCSC Part#"
 	1    6300 3400
 	1    0    0    -1
@@
 AR Path="/5FEF404D/5E0203CB" Ref="C1103"  Part="1"
 F 0 "C1103" H 7165 3396 50  0000 L CNN
-F 1 "100n" H 7165 3305 50  0000 L CNN
+F 1 "100nF" H 7165 3305 50  0000 L CNN
 F 2 "Capacitor_SMD:C_0805_2012Metric_Pad1.18x1.45mm_HandSolder" H 7088 3200 50  0001 C CNN
 F 3 "~" H 7050 3350 50  0001 C CNN
-F 4 "Vishay" H 0   0   50  0001 C CNN "Manufacturer"
+F 4 "CPL" H 0   0   50  0001 C CNN "Manufacturer"
 F 5 "0" H 7050 3350 50  0001 C CNN "DNP"
-F 6 "BC1150CT-ND" H 7050 3350 50  0001 C CNN "Digikey"
-F 7 "K104K15X7RF5TL2" H 7050 3350 50  0001 C CNN "MPN"
-F 8 "594-K104K15X7RF5TL2" H 7050 3350 50  0001 C CNN "Mouser"
+F 6 "" H 7050 3350 50  0001 C CNN "Digikey"
+F 7 "CPL-CAP-X7R-0805-100NF-50V" H 7050 3350 50  0001 C CNN "MPN"
+F 8 "" H 7050 3350 50  0001 C CNN "Mouser"
+F 9 "C49678" H 7050 3350 50  0001 C CNN "LCSC Part#"
 	1    7050 3350
 	1    0    0    -1
@@
 F 7 "300-8301-ND" H 5025 3000 50  0001 C CNN "Digikey"
 F 8 "CFS-20632768DZBB" H 5025 3000 50  0001 C CNN "Mouser"
+F 9 "~" H 5025 3000 50  0001 C CNN "LCSC Part#"
 	1    5025 3000
 	-1   0    0    1
@@
 P 5350 3500
 F 0 "C1102" H 5465 3546 50  0000 L CNN
-F 1 "6p" H 5465 3455 50  0000 L CNN
+F 1 "6pF" H 5465 3455 50  0000 L CNN
 F 2 "Capacitor_SMD:C_0805_2012Metric_Pad1.18x1.45mm_HandSolder" H 5388 3350 50  0001 C CNN
 F 3 "~" H 5350 3500 50  0001 C CNN
@@
 F 7 "311-1095-1-ND" H 5350 3500 50  0001 C CNN "Digikey"
 F 8 "603-CC805DRNPO9BN6R0" H 5350 3500 50  0001 C CNN "Mouser"
+F 9 "C67560" H 5350 3500 50  0001 C CNN "LCSC Part#"
+F 10 "C0G" H 5350 3500 50  0001 C CNN "Voltage"
 	1    5350 3500
 	1    0    0    -1
@@
 P 4700 3500
 F 0 "C1101" H 4815 3546 50  0000 L CNN
-F 1 "6p" H 4815 3455 50  0000 L CNN
+F 1 "6pF" H 4815 3455 50  0000 L CNN
 F 2 "Capacitor_SMD:C_0805_2012Metric_Pad1.18x1.45mm_HandSolder" H 4738 3350 50  0001 C CNN
 F 3 "~" H 4700 3500 50  0001 C CNN
@@
 F 7 "311-1095-1-ND" H 4700 3500 50  0001 C CNN "Digikey"
 F 8 "603-CC805DRNPO9BN6R0" H 4700 3500 50  0001 C CNN "Mouser"
+F 9 "C67560" H 4700 3500 50  0001 C CNN "LCSC Part#"
+F 10 "C0G" H 4700 3500 50  0001 C CNN "Voltage"
 	1    4700 3500
 	1    0    0    -1
