File: Kicad/serial.sch (KiCad schematic (older format))
At the start: 9 parts, among them J801 Conn_02x05, J802 DB9_Male_MountingHoles, U801 ST3232CDR

Commit message: Change ST to ST Micro for consistency
Parts:
- U801: Manufacturer ST -> ST Micro
Changed lines of the file:
@@
 F 2 "Package_SO:SO-16_5.3x10.2mm_P1.27mm" H 5500 2000 50  0001 L CNN
 F 3 "https://www.st.com/content/ccc/resource/technical/document/datasheet/group1/40/2c/7f/62/3a/3f/47/3c/CD00002253/files/CD00002253.pdf/jcr:content/translations/en.CD00002253.pdf" H 5450 3150 50  0001 C CNN
-F 4 "ST" H 5450 3050 50  0001 C CNN "Manufacturer"
+F 4 "ST Micro" H 5450 3050 50  0001 C CNN "Manufacturer"
 F 5 "0" H 5450 3050 50  0001 C CNN "DNP"
 F 6 "497-3731-1-ND" H 5450 3050 50  0001 C CNN "Digikey"

Commit message: Added 12-bit video DAC.
Also had to change footprints to suit Kicad 5.1.9
Parts:
- C47: renamed from C805; footprint Capacitor_SMD:C_0805_2012Metric_Pad1.15x1.40mm_HandSolder -> Capacitor_SMD:C_0805_2012Metric_Pad1.18x1.45mm_HandSolder
- C48: renamed from C801; footprint Capacitor_SMD:C_0805_2012Metric_Pad1.15x1.40mm_HandSolder -> Capacitor_SMD:C_0805_2012Metric_Pad1.18x1.45mm_HandSolder
- C49: renamed from C802; footprint Capacitor_SMD:C_0805_2012Metric_Pad1.15x1.40mm_HandSolder -> Capacitor_SMD:C_0805_2012Metric_Pad1.18x1.45mm_HandSolder
- C50: renamed from C803; footprint Capacitor_SMD:C_0805_2012Metric_Pad1.15x1.40mm_HandSolder -> Capacitor_SMD:C_0805_2012Metric_Pad1.18x1.45mm_HandSolder
- C51: renamed from C804; footprint Capacitor_SMD:C_0805_2012Metric_Pad1.15x1.40mm_HandSolder -> Capacitor_SMD:C_0805_2012Metric_Pad1.18x1.45mm_HandSolder
- R65: renamed from R801; footprint Resistor_SMD:R_0805_2012Metric_Pad1.15x1.40mm_HandSolder -> Resistor_SMD:R_0805_2012Metric_Pad1.20x1.40mm_HandSolder
- renumbered J801 to J10, J802 to J11, U801 to U6
Changed lines of the file:
@@
 $Descr A4 11693 8268
 encoding utf-8
-Sheet 8 12
+Sheet 8 16
 Title "Neotron Common Hardware - Serial Port"
 Date "2021-01-01"
@@
 AR Path="/5FDF5821" Ref="J?"  Part="1"
 AR Path="/5FDEDE75/5FDF5821" Ref="J?"  Part="1"
-AR Path="/5FDF53DB/5FDF5821" Ref="J802"  Part="1"
-F 0 "J802" H 8350 4700 50  0000 L CNN
+AR Path="/5FDF53DB/5FDF5821" Ref="J11"  Part="1"
+F 0 "J11" H 8350 4700 50  0000 L CNN
 F 1 "DB9_Male_MountingHoles" H 8350 4600 50  0000 L CNN
 F 2 "Connector_Dsub:DSUB-9_Male_Horizontal_P2.77x2.84mm_EdgePinOffset7.70mm_Housed_MountingHolesOffset9.12mm" H 8100 4700 50  0001 C CNN
@@
 RS232_CTS_TO_MCU
 $Comp
-L Interface_UART:MAX232 U801
+L Interface_UART:MAX232 U6
 U 1 1 5E0F5F91
 P 5450 3050
-F 0 "U801" H 5950 4150 50  0000 C CNN
+F 0 "U6" H 5950 4150 50  0000 C CNN
 F 1 "ST3232CDR" H 5000 4150 50  0000 C CNN
 F 2 "Package_SO:SO-16_5.3x10.2mm_P1.27mm" H 5500 2000 50  0001 L CNN
@@
 RS232_RTS_OUT
 $Comp
-L power:GND #PWR0802
+L power:GND #PWR0117
 U 1 1 5E180507
 P 7150 2850
-F 0 "#PWR0802" H 7150 2600 50  0001 C CNN
+F 0 "#PWR0117" H 7150 2600 50  0001 C CNN
 F 1 "GND" H 7155 2677 50  0000 C CNN
 F 2 "" H 7150 2850 50  0001 C CNN
@@
 	7150 2850 7150 2800
 $Comp
-L Device:C C802
+L Device:C C49
 U 1 1 5E181E57
 P 6350 2300
-F 0 "C802" H 6650 2350 50  0000 R CNN
+F 0 "C49" H 6650 2350 50  0000 R CNN
 F 1 "100n" H 6650 2250 50  0000 R CNN
-F 2 "Capacitor_SMD:C_0805_2012Metric_Pad1.15x1.40mm_HandSolder" H 6388 2150 50  0001 C CNN
+F 2 "Capacitor_SMD:C_0805_2012Metric_Pad1.18x1.45mm_HandSolder" H 6388 2150 50  0001 C CNN
 F 3 "~" H 6350 2300 50  0001 C CNN
 F 4 "Vishay" H -150 -600 50  0001 C CNN "Manufacturer"
@@
 $EndComp
 $Comp
-L Device:C C804
+L Device:C C51
 U 1 1 5E182C3F
 P 6550 2950
-F 0 "C804" V 6450 2700 50  0000 L CNN
+F 0 "C51" V 6450 2700 50  0000 L CNN
 F 1 "100n" V 6450 3200 50  0000 R CNN
-F 2 "Capacitor_SMD:C_0805_2012Metric_Pad1.15x1.40mm_HandSolder" H 6588 2800 50  0001 C CNN
+F 2 "Capacitor_SMD:C_0805_2012Metric_Pad1.18x1.45mm_HandSolder" H 6588 2800 50  0001 C CNN
 F 3 "~" H 6550 2950 50  0001 C CNN
 F 4 "Vishay" H -250 -600 50  0001 C CNN "Manufacturer"
@@
 $EndComp
 $Comp
-L Device:C C805
+L Device:C C47
 U 1 1 5E183108
 P 1900 3400
-F 0 "C805" H 1785 3354 50  0000 R CNN
+F 0 "C47" H 1785 3354 50  0000 R CNN
 F 1 "100n" H 1785 3445 50  0000 R CNN
-F 2 "Capacitor_SMD:C_0805_2012Metric_Pad1.15x1.40mm_HandSolder" H 1938 3250 50  0001 C CNN
+F 2 "Capacitor_SMD:C_0805_2012Metric_Pad1.18x1.45mm_HandSolder" H 1938 3250 50  0001 C CNN
 F 3 "~" H 1900 3400 50  0001 C CNN
 F 4 "Vishay" H -1450 300 50  0001 C CNN "Manufacturer"
@@
 $EndComp
 $Comp
-L power:+3V3 #PWR0801
+L power:+3V3 #PWR0115
 U 1 1 5E183A22
 P 5450 1750
-F 0 "#PWR0801" H 5450 1600 50  0001 C CNN
+F 0 "#PWR0115" H 5450 1600 50  0001 C CNN
 F 1 "+3V3" H 5465 1923 50  0000 C CNN
 F 2 "" H 5450 1750 50  0001 C CNN
@@
 $EndComp
 $Comp
-L power:+3V3 #PWR0803
+L power:+3V3 #PWR0113
 U 1 1 5E18439B
 P 1900 3150
-F 0 "#PWR0803" H 1900 3000 50  0001 C CNN
+F 0 "#PWR0113" H 1900 3000 50  0001 C CNN
 F 1 "+3V3" H 1915 3323 50  0000 C CNN
 F 2 "" H 1900 3150 50  0001 C CNN
@@
 $EndComp
 $Comp
-L power:GND #PWR0805
+L power:GND #PWR0114
 U 1 1 5E1846FE
 P 1900 3650
-F 0 "#PWR0805" H 1900 3400 50  0001 C CNN
+F 0 "#PWR0114" H 1900 3400 50  0001 C CNN
 F 1 "GND" H 1905 3477 50  0000 C CNN
 F 2 "" H 1900 3650 50  0001 C CNN
@@
 	4500 2450 4650 2450
 $Comp
-L power:GND #PWR0806
+L power:GND #PWR0116
 U 1 1 5E18A6A9
 P 5450 4300
-F 0 "#PWR0806" H 5450 4050 50  0001 C CNN
+F 0 "#PWR0116" H 5450 4050 50  0001 C CNN
 F 1 "GND" H 5455 4127 50  0000 C CNN
 F 2 "" H 5450 4300 50  0001 C CNN
@@
 NoConn ~ 8250 3350
 $Comp
-L Connector_Generic:Conn_02x05_Top_Bottom J801
+L Connector_Generic:Conn_02x05_Top_Bottom J10
 U 1 1 5E02DBC9
 P 7950 3450
-F 0 "J801" H 8000 3025 50  0000 C CNN
+F 0 "J10" H 8000 3025 50  0000 C CNN
 F 1 "Conn_02x05" H 8000 3116 50  0000 C CNN
 F 2 "Connector_IDC:IDC-Header_2x05_P2.54mm_Vertical" H 7950 3450 50  0001 C CNN
@@
 $EndComp
 $Comp
-L power:GND #PWR0804
+L power:GND #PWR0118
 U 1 1 5E03D39E
 P 7550 3250
-F 0 "#PWR0804" H 7550 3000 50  0001 C CNN
+F 0 "#PWR0118" H 7550 3000 50  0001 C CNN
 F 1 "GND" H 7550 3100 50  0000 C CNN
 F 2 "" H 7550 3250 50  0001 C CNN
@@
 	7800 4700 7250 4700
 $Comp
-L power:GND #PWR0807
+L power:GND #PWR0119
 U 1 1 60A551CD
 P 7600 4300
-F 0 "#PWR0807" H 7600 4050 50  0001 C CNN
+F 0 "#PWR0119" H 7600 4050 50  0001 C CNN
 F 1 "GND" H 7600 4150 50  0000 C CNN
 F 2 "" H 7600 4300 50  0001 C CNN
@@
 	7600 4250 7600 4300
 $Comp
-L power:GND #PWR0808
+L power:GND #PWR0120
 U 1 1 60A56FF6
 P 8100 5700
-F 0 "#PWR0808" H 8100 5450 50  0001 C CNN
+F 0 "#PWR0120" H 8100 5450 50  0001 C CNN
 F 1 "GND" H 8100 5550 50  0000 C CNN
 F 2 "" H 8100 5700 50  0001 C CNN
@@
 $EndComp
 $Comp
-L Device:R R801
+L Device:R R65
 U 1 1 60A5752A
 P 8100 5500
-F 0 "R801" H 8170 5546 50  0000 L CNN
+F 0 "R65" H 8170 5546 50  0000 L CNN
 F 1 "DNF" H 8170 5455 50  0000 L CNN
-F 2 "Resistor_SMD:R_0805_2012Metric_Pad1.15x1.40mm_HandSolder" V 8030 5500 50  0001 C CNN
+F 2 "Resistor_SMD:R_0805_2012Metric_Pad1.20x1.40mm_HandSolder" V 8030 5500 50  0001 C CNN
 F 3 "~" H 8100 5500 50  0001 C CNN
 F 4 "1" H 8100 5500 50  0001 C CNN "DNP"
@@
 	6250 2650 6400 2650
 $Comp
-L Device:C C803
+L Device:C C50
 U 1 1 5E188858
 P 6550 2650
-F 0 "C803" V 6450 2400 50  0000 L CNN
+F 0 "C50" V 6450 2400 50  0000 L CNN
 F 1 "100n" V 6450 2900 50  0000 R CNN
-F 2 "Capacitor_SMD:C_0805_2012Metric_Pad1.15x1.40mm_HandSolder" H 6588 2500 50  0001 C CNN
+F 2 "Capacitor_SMD:C_0805_2012Metric_Pad1.18x1.45mm_HandSolder" H 6588 2500 50  0001 C CNN
 F 3 "~" H 6550 2650 50  0001 C CNN
 F 4 "Vishay" H -500 -150 50  0001 C CNN "Manufacturer"
@@
 $EndComp
 $Comp
-L Device:C C801
+L Device:C C48
 U 1 1 5E182DBA
 P 4500 2300
-F 0 "C801" H 4600 2250 50  0000 L CNN
+F 0 "C48" H 4600 2250 50  0000 L CNN
 F 1 "100n" H 4600 2350 50  0000 L CNN
-F 2 "Capacitor_SMD:C_0805_2012Metric_Pad1.15x1.40mm_HandSolder" H 4538 2150 50  0001 C CNN
+F 2 "Capacitor_SMD:C_0805_2012Metric_Pad1.18x1.45mm_HandSolder" H 4538 2150 50  0001 C CNN
 F 3 "~" H 4500 2300 50  0001 C CNN
 F 4 "Vishay" H -150 -600 50  0001 C CNN "Manufacturer"

Commit message: Add 4-bit Video DAC, and re-wire BMC.
Now the BMC is an SPI device, and has a four-wire UART.
Parts:
- renumbered C47 to C801, C48 to C802, C49 to C803, C50 to C804, C51 to C805, J10 to J801, J11 to J802, R65 to R801, U6 to U801
Changed lines of the file:
@@
 Sheet 8 16
 Title "Neotron Common Hardware - Serial Port"
-Date "2021-01-01"
+Date "2021-04-02"
 Rev "[Uncontrolled]"
 Comp "https://neotron-compute.github.io/"
@@
 AR Path="/5FDF5821" Ref="J?"  Part="1"
 AR Path="/5FDEDE75/5FDF5821" Ref="J?"  Part="1"
-AR Path="/5FDF53DB/5FDF5821" Ref="J11"  Part="1"
-F 0 "J11" H 8350 4700 50  0000 L CNN
+AR Path="/5FDF53DB/5FDF5821" Ref="J802"  Part="1"
+F 0 "J802" H 8350 4700 50  0000 L CNN
 F 1 "DB9_Male_MountingHoles" H 8350 4600 50  0000 L CNN
 F 2 "Connector_Dsub:DSUB-9_Male_Horizontal_P2.77x2.84mm_EdgePinOffset7.70mm_Housed_MountingHolesOffset9.12mm" H 8100 4700 50  0001 C CNN
@@
 RS232_CTS_TO_MCU
 $Comp
-L Interface_UART:MAX232 U6
+L Interface_UART:MAX232 U801
 U 1 1 5E0F5F91
 P 5450 3050
-F 0 "U6" H 5950 4150 50  0000 C CNN
+F 0 "U801" H 5950 4150 50  0000 C CNN
 F 1 "ST3232CDR" H 5000 4150 50  0000 C CNN
 F 2 "Package_SO:SO-16_5.3x10.2mm_P1.27mm" H 5500 2000 50  0001 L CNN
@@
 RS232_RTS_OUT
 $Comp
-L power:GND #PWR0117
+L power:GND #PWR0805
 U 1 1 5E180507
 P 7150 2850
-F 0 "#PWR0117" H 7150 2600 50  0001 C CNN
+F 0 "#PWR0805" H 7150 2600 50  0001 C CNN
 F 1 "GND" H 7155 2677 50  0000 C CNN
 F 2 "" H 7150 2850 50  0001 C CNN
@@
 	7150 2850 7150 2800
 $Comp
-L Device:C C49
+L Device:C C803
 U 1 1 5E181E57
 P 6350 2300
-F 0 "C49" H 6650 2350 50  0000 R CNN
+F 0 "C803" H 6650 2350 50  0000 R CNN
 F 1 "100n" H 6650 2250 50  0000 R CNN
 F 2 "Capacitor_SMD:C_0805_2012Metric_Pad1.18x1.45mm_HandSolder" H 6388 2150 50  0001 C CNN
@@
 $EndComp
 $Comp
-L Device:C C51
+L Device:C C805
 U 1 1 5E182C3F
 P 6550 2950
-F 0 "C51" V 6450 2700 50  0000 L CNN
+F 0 "C805" V 6450 2700 50  0000 L CNN
 F 1 "100n" V 6450 3200 50  0000 R CNN
 F 2 "Capacitor_SMD:C_0805_2012Metric_Pad1.18x1.45mm_HandSolder" H 6588 2800 50  0001 C CNN
@@
 $EndComp
 $Comp
-L Device:C C47
+L Device:C C801
 U 1 1 5E183108
 P 1900 3400
-F 0 "C47" H 1785 3354 50  0000 R CNN
+F 0 "C801" H 1785 3354 50  0000 R CNN
 F 1 "100n" H 1785 3445 50  0000 R CNN
 F 2 "Capacitor_SMD:C_0805_2012Metric_Pad1.18x1.45mm_HandSolder" H 1938 3250 50  0001 C CNN
@@
 $EndComp
 $Comp
-L power:+3V3 #PWR0115
+L power:+3V3 #PWR0803
 U 1 1 5E183A22
 P 5450 1750
-F 0 "#PWR0115" H 5450 1600 50  0001 C CNN
+F 0 "#PWR0803" H 5450 1600 50  0001 C CNN
 F 1 "+3V3" H 5465 1923 50  0000 C CNN
 F 2 "" H 5450 1750 50  0001 C CNN
@@
 $EndComp
 $Comp
-L power:+3V3 #PWR0113
+L power:+3V3 #PWR0801
 U 1 1 5E18439B
 P 1900 3150
-F 0 "#PWR0113" H 1900 3000 50  0001 C CNN
+F 0 "#PWR0801" H 1900 3000 50  0001 C CNN
 F 1 "+3V3" H 1915 3323 50  0000 C CNN
 F 2 "" H 1900 3150 50  0001 C CNN
@@
 $EndComp
 $Comp
-L power:GND #PWR0114
+L power:GND #PWR0802
 U 1 1 5E1846FE
 P 1900 3650
-F 0 "#PWR0114" H 1900 3400 50  0001 C CNN
+F 0 "#PWR0802" H 1900 3400 50  0001 C CNN
 F 1 "GND" H 1905 3477 50  0000 C CNN
 F 2 "" H 1900 3650 50  0001 C CNN
@@
 	4500 2450 4650 2450
 $Comp
-L power:GND #PWR0116
+L power:GND #PWR0804
 U 1 1 5E18A6A9
 P 5450 4300
-F 0 "#PWR0116" H 5450 4050 50  0001 C CNN
+F 0 "#PWR0804" H 5450 4050 50  0001 C CNN
 F 1 "GND" H 5455 4127 50  0000 C CNN
 F 2 "" H 5450 4300 50  0001 C CNN
@@
 NoConn ~ 8250 3350
 $Comp
-L Connector_Generic:Conn_02x05_Top_Bottom J10
+L Connector_Generic:Conn_02x05_Top_Bottom J801
 U 1 1 5E02DBC9
 P 7950 3450
-F 0 "J10" H 8000 3025 50  0000 C CNN
+F 0 "J801" H 8000 3025 50  0000 C CNN
 F 1 "Conn_02x05" H 8000 3116 50  0000 C CNN
 F 2 "Connector_IDC:IDC-Header_2x05_P2.54mm_Vertical" H 7950 3450 50  0001 C CNN
@@
 $EndComp
 $Comp
-L power:GND #PWR0118
+L power:GND #PWR0806
 U 1 1 5E03D39E
 P 7550 3250
-F 0 "#PWR0118" H 7550 3000 50  0001 C CNN
+F 0 "#PWR0806" H 7550 3000 50  0001 C CNN
 F 1 "GND" H 7550 3100 50  0000 C CNN
 F 2 "" H 7550 3250 50  0001 C CNN
@@
 	7800 4700 7250 4700
 $Comp
-L power:GND #PWR0119
+L power:GND #PWR0807
 U 1 1 60A551CD
 P 7600 4300
-F 0 "#PWR0119" H 7600 4050 50  0001 C CNN
+F 0 "#PWR0807" H 7600 4050 50  0001 C CNN
 F 1 "GND" H 7600 4150 50  0000 C CNN
 F 2 "" H 7600 4300 50  0001 C CNN
@@
 	7600 4250 7600 4300
 $Comp
-L power:GND #PWR0120
+L power:GND #PWR0808
 U 1 1 60A56FF6
 P 8100 5700
-F 0 "#PWR0120" H 8100 5450 50  0001 C CNN
+F 0 "#PWR0808" H 8100 5450 50  0001 C CNN
 F 1 "GND" H 8100 5550 50  0000 C CNN
 F 2 "" H 8100 5700 50  0001 C CNN
@@
 $EndComp
 $Comp
-L Device:R R65
+L Device:R R801
 U 1 1 60A5752A
 P 8100 5500
-F 0 "R65" H 8170 5546 50  0000 L CNN
+F 0 "R801" H 8170 5546 50  0000 L CNN
 F 1 "DNF" H 8170 5455 50  0000 L CNN
 F 2 "Resistor_SMD:R_0805_2012Metric_Pad1.20x1.40mm_HandSolder" V 8030 5500 50  0001 C CNN
@@
 	6250 2650 6400 2650
 $Comp
-L Device:C C50
+L Device:C C804
 U 1 1 5E188858
 P 6550 2650
-F 0 "C50" V 6450 2400 50  0000 L CNN
+F 0 "C804" V 6450 2400 50  0000 L CNN
 F 1 "100n" V 6450 2900 50  0000 R CNN
 F 2 "Capacitor_SMD:C_0805_2012Metric_Pad1.18x1.45mm_HandSolder" H 6588 2500 50  0001 C CNN
@@
 $EndComp
 $Comp
-L Device:C C48
+L Device:C C802
 U 1 1 5E182DBA
 P 4500 2300
-F 0 "C48" H 4600 2250 50  0000 L CNN
+F 0 "C802" H 4600 2250 50  0000 L CNN
 F 1 "100n" H 4600 2350 50  0000 L CNN
 F 2 "Capacitor_SMD:C_0805_2012Metric_Pad1.18x1.45mm_HandSolder" H 4538 2150 50  0001 C CNN

Commit message: Tidy up part nos and swapped I2C/UART on BMC.
Mark all resistors as 1% if not specified.
Added some Mouser part numbers.
BMC can now be programmed over UART.
Parts:
- C801, C802, C803, C804, C805: Mouser (none) -> 594-K104K15X7RF5TL2
- U801: Mouser (none) -> 511-ST3232CDR
Changed lines of the file:
@@
 F 6 "497-3731-1-ND" H 5450 3050 50  0001 C CNN "Digikey"
 F 7 "ST3232CDR" H 5450 3050 50  0001 C CNN "MPN"
+F 8 "511-ST3232CDR" H 5450 3050 50  0001 C CNN "Mouser"
 	1    5450 3050
 	1    0    0    -1
@@
 F 6 "BC1150CT-ND" H 6350 2300 50  0001 C CNN "Digikey"
 F 7 "K104K15X7RF5TL2" H 6350 2300 50  0001 C CNN "MPN"
+F 8 "594-K104K15X7RF5TL2" H 6350 2300 50  0001 C CNN "Mouser"
 	1    6350 2300
 	1    0    0    -1
@@
 F 6 "BC1150CT-ND" H 6550 2950 50  0001 C CNN "Digikey"
 F 7 "K104K15X7RF5TL2" H 6550 2950 50  0001 C CNN "MPN"
+F 8 "594-K104K15X7RF5TL2" H 6550 2950 50  0001 C CNN "Mouser"
 	1    6550 2950
 	0    1    1    0
@@
 F 6 "BC1150CT-ND" H 1900 3400 50  0001 C CNN "Digikey"
 F 7 "K104K15X7RF5TL2" H 1900 3400 50  0001 C CNN "MPN"
+F 8 "594-K104K15X7RF5TL2" H 1900 3400 50  0001 C CNN "Mouser"
 	1    1900 3400
 	-1   0    0    1
@@
 F 6 "BC1150CT-ND" H 6550 2650 50  0001 C CNN "Digikey"
 F 7 "K104K15X7RF5TL2" H 6550 2650 50  0001 C CNN "MPN"
+F 8 "594-K104K15X7RF5TL2" H 6550 2650 50  0001 C CNN "Mouser"
 	1    6550 2650
 	0    1    1    0
@@
 F 6 "BC1150CT-ND" H 4500 2300 50  0001 C CNN "Digikey"
 F 7 "K104K15X7RF5TL2" H 4500 2300 50  0001 C CNN "MPN"
+F 8 "594-K104K15X7RF5TL2" H 4500 2300 50  0001 C CNN "Mouser"
 	1    4500 2300
 	-1   0    0    1
