File: Kicad/powersupply.sch (KiCad schematic (older format))
At the start: 35 parts, among them J901 Jack-DC, J902 Conn_02x04_Odd_Even, J903 Double-mini-DIN-6, J904 Header, Q901 BC548, SW901 SW_DIP_x01, SW902 SW_DIP_x01, U901 5V DC-DC Module, U902 TLV1117 3.3V 1A, U903 MAX1615, U904 STM32F030F4Px

Commit message: Replace inductor with horizontal footprint.
Parts:
- L901: footprint Inductor_THT:L_Axial_L26.0mm_D11.0mm_P7.62mm_Vertical_Fastron_77A -> Inductor_THT:L_Axial_L26.7mm_D12.1mm_P35.00mm_Horizontal_Vishay_IHA-103
Changed lines of the file:
@@
 F 0 "L901" V 2090 1400 50  0000 C CNN
 F 1 "22uH 6A" V 1999 1400 50  0000 C CNN
-F 2 "Inductor_THT:L_Axial_L26.0mm_D11.0mm_P7.62mm_Vertical_Fastron_77A" H 1900 1400 50  0001 C CNN
+F 2 "Inductor_THT:L_Axial_L26.7mm_D12.1mm_P35.00mm_Horizontal_Vishay_IHA-103" H 1900 1400 50  0001 C CNN
 F 3 "https://abracon.com/Magnetics/axial/AIAP-03.pdf" H 1900 1400 50  0001 C CNN
 F 4 "0" H 1900 1400 50  0001 C CNN "DNP"

Commit message: Switch some of the radial THT Electrolytic caps for SMD MLCCs.
Also changed the STM32 for an LQFP-32 as it has a bigger pitch on the
pins.

The LQFP is easier to solder than the TSSOP, and the MLCC takes are
cheaper and take up less space.
Parts:
- removed J902: Conn_02x04_Odd_Even, Connector_PinHeader_2.54mm:PinHeader_2x04_P2.54mm_Vertical, symbol Connector_Generic:Conn_02x04_Odd_Even
- removed TP901: TestPoint, Connector_PinHeader_2.54mm:PinHeader_1x01_P2.54mm_Vertical, symbol Connector:TestPoint
- removed U904: STM32F030F4Px, Package_SO:TSSOP-20_4.4x6.5mm_P0.65mm, symbol MCU_ST_STM32F0:STM32F030F4Px
- added C908: 100n, Capacitor_SMD:C_0805_2012Metric_Pad1.15x1.40mm_HandSolder, symbol Device:C
- added C911: 10n, Capacitor_SMD:C_0805_2012Metric_Pad1.15x1.40mm_HandSolder, symbol Device:C
- added C912: 1u 10V, Capacitor_SMD:C_0805_2012Metric_Pad1.15x1.40mm_HandSolder, symbol Device:C
- added J902: Conn_01x06, Connector_PinHeader_2.54mm:PinHeader_1x06_P2.54mm_Vertical, symbol Connector_Generic:Conn_01x06
- added J903: Conn_01x03, Connector_PinHeader_2.54mm:PinHeader_1x03_P2.54mm_Vertical, symbol Connector_Generic:Conn_01x03
- added JP901: Jumper, Connector_PinHeader_2.54mm:PinHeader_1x02_P2.54mm_Vertical, symbol Device:Jumper_NO_Small
- added TP901, TP902, TP903, TP904, TP905, TP906: TestPoint_Small, Connector_PinHeader_2.54mm:PinHeader_1x01_P2.54mm_Vertical, symbol Connector:TestPoint_Small
- added U904: STM32F031K6T6, Package_QFP:LQFP-32_7x7mm_P0.8mm, symbol MCU_ST_STM32F0:STM32F031K6Tx
- C903: value 22u -> 22u 16V; footprint Capacitor_THT:CP_Radial_D6.3mm_P2.50mm -> Capacitor_SMD:C_0805_2012Metric_Pad1.15x1.40mm_HandSolder; symbol Device:CP -> Device:C; Digikey 493-11025-1-ND -> 1276-7092-1-ND; MPN UFW1J220MDD1TD -> CL21A226KOQNNNG; Manufacturer Nichicon -> Samsung
- C905: value 1u -> 1u 10V; Digikey 493-12597-1-ND -> 1276-6471-1-ND; MPN UVK1V470MDD1TD -> CL21B105KOFNNNG; Manufacturer Nichicon -> Samsung
- C906: footprint Capacitor_THT:CP_Radial_D6.3mm_P2.50mm -> Capacitor_SMD:C_0805_2012Metric_Pad1.15x1.40mm_HandSolder; symbol Device:CP -> Device:C; Digikey 493-10944-1-ND -> 1276-6470-1-ND; MPN UFG1H010MDM1TD -> CL21B105KBFNNNG; Manufacturer Nichicon -> Samsung
- C907: value 4u7 -> 4u7 10V; footprint Capacitor_THT:CP_Radial_D6.3mm_P2.50mm -> Capacitor_SMD:C_0805_2012Metric_Pad1.15x1.40mm_HandSolder; symbol Device:CP -> Device:C; Digikey 493-12612-1-ND -> 1276-6464-1-ND; MPN UVK2A4R7MDD1TD -> CL21A475KPFNNNG; Manufacturer Nichicon -> Samsung
- C910: renamed from C909; value 100n -> 4u7 10V; Digikey BC1150CT-ND -> 1276-6464-1-ND; MPN K104K15X7RF5TL2 -> CL21A475KPFNNNG; Manufacturer Vishay -> Samsung
- U901: footprint Connector_PinSocket_2.54mm:PinSocket_1x12_P2.54mm_Vertical -> Neotron-Common-Hardware:K78xx-3AR3
- renumbered C908 to C909, J903 to J905, R907 to R904, R904 to R905, R908 to R907, R910 to R908, R905 to R909, R909 to R910
Connections:
- net labels added: BOOT_RX, SWCLK_BOOT_TX, SWDIO, UART_RX, UART_TX
- net labels removed: BOOT0, SCL_U1TX, SDA_U1RX, USART1_TX
- wire segments 148 -> 177
Other:
- note added: "If JPx01 fitted, UART on Jx02.2 / Jx02.3\nIf JPx01 removed, SWD on Jx02.3 / Jx02.4"
- note added: "Manual reset switch:\nTap to reboot host"
- note added: "Place near Ux04 VDD"
- note added: "Place near Ux04 VDDA"
- note added: "UART Console"
- note removed: "BOOT0 = 0 => Run Program\nBOOT0 = 1 => Bootloader"
- note removed: "Manual reset switch:\nTap for reset"
- note removed: "Normal Operation:\n* Remove all connections from J902\n* Fit jumper to J902 1-2\n* Fit jumper to J902 3-4\n\nUART Programming:\n* Remove all connections from J902\n* Fit jumper to Jx 5-7 to select Bootloader\n* Connect J902 Pin 2 to UART RX\n* Connect J902 Pin 4 to UART TX\n* Connect DC power\n* Short J902 6-8 to reset BMC as required\n"
- note removed: "Place near U604"
- moved on the sheet: C909, C910, D901, J904, R904, R906, R907, R908, R909, R910, SW901, SW902

Commit message: Added 12-bit video DAC.
Also had to change footprints to suit Kicad 5.1.9
Parts:
- C54: renamed from C906; footprint Capacitor_SMD:C_0805_2012Metric_Pad1.15x1.40mm_HandSolder -> Capacitor_SMD:C_0805_2012Metric_Pad1.18x1.45mm_HandSolder
- C55: renamed from C903; footprint Capacitor_SMD:C_0805_2012Metric_Pad1.15x1.40mm_HandSolder -> Capacitor_SMD:C_0805_2012Metric_Pad1.18x1.45mm_HandSolder
- C56: renamed from C907; footprint Capacitor_SMD:C_0805_2012Metric_Pad1.15x1.40mm_HandSolder -> Capacitor_SMD:C_0805_2012Metric_Pad1.18x1.45mm_HandSolder
- C57: renamed from C911; footprint Capacitor_SMD:C_0805_2012Metric_Pad1.15x1.40mm_HandSolder -> Capacitor_SMD:C_0805_2012Metric_Pad1.18x1.45mm_HandSolder
- C58: renamed from C908; footprint Capacitor_SMD:C_0805_2012Metric_Pad1.15x1.40mm_HandSolder -> Capacitor_SMD:C_0805_2012Metric_Pad1.18x1.45mm_HandSolder
- C59: renamed from C912; footprint Capacitor_SMD:C_0805_2012Metric_Pad1.15x1.40mm_HandSolder -> Capacitor_SMD:C_0805_2012Metric_Pad1.18x1.45mm_HandSolder
- C60: renamed from C909; footprint Capacitor_SMD:C_0805_2012Metric_Pad1.15x1.40mm_HandSolder -> Capacitor_SMD:C_0805_2012Metric_Pad1.18x1.45mm_HandSolder
- C61: renamed from C904; footprint Capacitor_SMD:C_0805_2012Metric_Pad1.15x1.40mm_HandSolder -> Capacitor_SMD:C_0805_2012Metric_Pad1.18x1.45mm_HandSolder
- C62: renamed from C910; footprint Capacitor_SMD:C_0805_2012Metric_Pad1.15x1.40mm_HandSolder -> Capacitor_SMD:C_0805_2012Metric_Pad1.18x1.45mm_HandSolder
- C63: renamed from C905; footprint Capacitor_SMD:C_0805_2012Metric_Pad1.15x1.40mm_HandSolder -> Capacitor_SMD:C_0805_2012Metric_Pad1.18x1.45mm_HandSolder
- R66: renamed from R901; footprint Resistor_SMD:R_0805_2012Metric_Pad1.15x1.40mm_HandSolder -> Resistor_SMD:R_0805_2012Metric_Pad1.20x1.40mm_HandSolder
- R67: renamed from R908; footprint Resistor_SMD:R_0805_2012Metric_Pad1.15x1.40mm_HandSolder -> Resistor_SMD:R_0805_2012Metric_Pad1.20x1.40mm_HandSolder
- R68: renamed from R909; footprint Resistor_SMD:R_0805_2012Metric_Pad1.15x1.40mm_HandSolder -> Resistor_SMD:R_0805_2012Metric_Pad1.20x1.40mm_HandSolder
- R69: renamed from R904; footprint Resistor_SMD:R_0805_2012Metric_Pad1.15x1.40mm_HandSolder -> Resistor_SMD:R_0805_2012Metric_Pad1.20x1.40mm_HandSolder
- R70: renamed from R906; footprint Resistor_SMD:R_0805_2012Metric_Pad1.15x1.40mm_HandSolder -> Resistor_SMD:R_0805_2012Metric_Pad1.20x1.40mm_HandSolder
- R71: renamed from R902; footprint Resistor_SMD:R_0805_2012Metric_Pad1.15x1.40mm_HandSolder -> Resistor_SMD:R_0805_2012Metric_Pad1.20x1.40mm_HandSolder
- R72: renamed from R903; footprint Resistor_SMD:R_0805_2012Metric_Pad1.15x1.40mm_HandSolder -> Resistor_SMD:R_0805_2012Metric_Pad1.20x1.40mm_HandSolder
- R73: renamed from R905; footprint Resistor_SMD:R_0805_2012Metric_Pad1.15x1.40mm_HandSolder -> Resistor_SMD:R_0805_2012Metric_Pad1.20x1.40mm_HandSolder
- R74: renamed from R907; footprint Resistor_SMD:R_0805_2012Metric_Pad1.15x1.40mm_HandSolder -> Resistor_SMD:R_0805_2012Metric_Pad1.20x1.40mm_HandSolder
- R75: renamed from R910; footprint Resistor_SMD:R_0805_2012Metric_Pad1.15x1.40mm_HandSolder -> Resistor_SMD:R_0805_2012Metric_Pad1.20x1.40mm_HandSolder
- renumbered C901 to C52, C902 to C53, D901 to D1, F901 to F1, J901 to J12, J905 to J13, J902 to J14, J904 to J15, J903 to J16, JP901 to JP1, L901 to L1, Q901 to Q1, RN901 to RN2, SW901 to SW1, SW902 to SW2, TP901 to TP1, TP902 to TP2, TP904 to TP3, TP905 to TP4, TP906 to TP5, TP903 to TP6, U904 to U10, U901 to U7, U903 to U8, U902 to U9

Commit message: Add 4-bit Video DAC, and re-wire BMC.
Now the BMC is an SPI device, and has a four-wire UART.
Parts:
- removed R70: 10k, Resistor_SMD:R_0805_2012Metric_Pad1.20x1.40mm_HandSolder, symbol Device:R
- removed TP1, TP2, TP3, TP4, TP5, TP6: TestPoint_Small, Connector_PinHeader_2.54mm:PinHeader_1x01_P2.54mm_Vertical, symbol Connector:TestPoint_Small
- added D902: LED, LED_THT:LED_D3.0mm, symbol Device:LED
- added J905: Header, Connector_PinHeader_2.54mm:PinHeader_1x02_P2.54mm_Vertical, symbol Connector:Conn_01x02_Male
- added R901: 100k, Resistor_SMD:R_0805_2012Metric_Pad1.20x1.40mm_HandSolder, symbol Device:R
- added R905, R906: 1k, Resistor_SMD:R_0805_2012Metric_Pad1.20x1.40mm_HandSolder, symbol Device:R
- J906: renamed from J16; value Conn_01x03 -> Conn_01x06; footprint Connector_PinHeader_2.54mm:PinHeader_1x03_P2.54mm_Vertical -> Connector_PinHeader_2.54mm:PinHeader_1x06_P2.54mm_Vertical; symbol Connector_Generic:Conn_01x03 -> Connector_Generic:Conn_01x06
- renumbered C52 to C901, C53 to C902, C54 to C903, C55 to C904, C56 to C905, C58 to C906, C60 to C907, C61 to C908, C62 to C909, C63 to C910, C57 to C911, C59 to C912, D1 to D901, F1 to F901, J12 to J901, J13 to J902, J14 to J903, J15 to J904, JP1 to JP901, L1 to L901, Q1 to Q901, R66 to R902, R67 to R903, R68 to R904, R69 to R907, R74 to R908, R75 to R909, R71 to R910, R72 to R911, R73 to R912, RN2 to RN901, SW1 to SW901, SW2 to SW902, U7 to U901, U8 to U902, U10 to U903, U9 to U904
Connections:
- net labels added: BOOT_MODE_SEL, KB_CLK, KB_DAT, LED0, LED1, MS_CLK, MS_DAT, SPI_CIPO, SPI_CLK, SPI_COPI, SWCLK, UART_CTS, UART_RTS, ~SPI_CS, ~SYS_RESET
- net labels removed: BOOT_RX, SWCLK_BOOT_TX, ~STATUS_LED
- wire segments 177 -> 222
- no-connect marks 5 -> 6
Other:
- note added: "BMC SWD Header"
- note added: "BMC UART Console\nFit FTDI TTL-FT232R-3V3"
- note added: "Black"
- note added: "Brown"
- note added: "FTDI puts 5V here!"
- note added: "Green"
- note added: "Most of our board runs on 3.3V. We expect\nto draw around 100 mA from this 1A linear\nregulator.\n\nNorm. power wasted: (5V - 3.3V) * 0.1A = 0.17W\nMax power wasted: (5V - 3.3V) * 1A = 1.7W\n\nAt 50 °C/W that's 85 °C over ambient at the\njunction at max power. Best to use a\nheatsink if you want to pull over 250 mA.\nOr replace with a 3-terminal switching\nPSU module."
- note added: "Orange"
- note added: "Place near Ux03 VDD"
- note added: "Place near Ux03 VDDA"
- note added: "Red"
- note added: "Yellow"
- note removed: "If JPx01 fitted, UART on Jx02.2 / Jx02.3\nIf JPx01 removed, SWD on Jx02.3 / Jx02.4"
- note removed: "Most of our board runs on 3.3V. We expect\nto draw around 100 mA from this 1A linear\nregulator.\n\nMax power wasted: (5V - 3.3V) * 1A = 1.7W\n\nAt 50 °C/W that's 85 °C over ambient at the\njunction - so use a heatsink if you want to\npull over 250 mA. Or replace with a\n3-terminal switching PSU module."
- note removed: "Place near Ux04 VDD"
- note removed: "Place near Ux04 VDDA"
- note removed: "UART Console"
- moved on the sheet: C906, C907, C908, C909, C910, C911, C912, D901, J902, J903, J904, JP901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

Commit message: Tidy up part nos and swapped I2C/UART on BMC.
Mark all resistors as 1% if not specified.
Added some Mouser part numbers.
BMC can now be programmed over UART.
Parts:
- C901, C902: Mouser (none) -> 647-UVR1H101MPD1TD
- C906, C907, C908: Mouser (none) -> 594-K104K15X7RF5TL2
- D901, D902: Mouser (none) -> 151031SS06000
- F901: Mouser (none) -> 530-0ZRS0200FF1E
- J901: Mouser (none) -> 490-PJ-063AH
- J902: Mouser (none) -> 806-KMDGX-6S/6S-S4N
- J903: value Conn_01x06 -> Conn_01x05; footprint Connector_PinHeader_2.54mm:PinHeader_1x06_P2.54mm_Vertical -> Connector_PinHeader_2.54mm:PinHeader_1x05_P2.54mm_Vertical; symbol Connector_Generic:Conn_01x06 -> Connector_Generic:Conn_01x05
- L901: Mouser (none) -> 815-AIAP03220K
- Q901: Mouser (none) -> 512-BC548BU
- R901: value 100k -> 100k 1%
- R902: value 2k -> 1k 1%; Digikey RMCF0805FT100K-ND -> RMCF0805FT1K00-ND; MPN RMCF0805FT100K -> RMCF0805FT1K00
- R903, R904, R905, R906: value 1k -> 1k 1%
- R907, R908, R909, R910, R911, R912: value 10k -> 10k 1%
- RN901: Mouser (none) -> 652-4605X-1LF-2.7K
- U902: Mouser (none) -> 700-MAX1615EUKT
- U903: Mouser (none) -> 511-STM32F031K6T6
- U904: Mouser (none) -> 595-TLV1117LV33DCYR
Connections:
- net labels removed: BOOT_MODE_SEL
- wire segments 222 -> 215
Other:
- note added: "1.65V nominal"
- note added: "Board Management\nController"
- note added: "Dual mini-DIN 6 connectors for PS/2 Keyboard and PS/2 Mouse.\nSignalling is 5V open-collector, with pull-up required."
- note added: "Fit Jx01 to enable UART\nbootloader on PA9/PA10"
- note added: "Serial Wire Debug"
- note removed: "BMC SWD Header"
- note removed: "Board Management Controller"
- note removed: "Dual mini-DIN 6 connectors for PS/2 Keyboard and PS/2 Mouse.\nSignalling is 5V open-collector, with pull-up required.\n\nKeyboard max current is 275 mA so cannot be run from\nstandby regulator."
- moved on the sheet: C906, C907, C909, C911, C912, D901, D902, J904, J905, R903, R904, R905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
