File: Kicad/ethernet.sch (KiCad schematic (older format))
At the start: 27 parts, among them J1101 RJ45 MagJack, U1101 ENC424J600, Y1101 25M

Commit message: Switch some of the radial THT Electrolytic caps for SMD MLCCs.
Also changed the STM32 for an LQFP-32 as it has a bigger pitch on the
pins.

The LQFP is easier to solder than the TSSOP, and the MLCC takes are
cheaper and take up less space.
Parts:
- C1105: footprint Capacitor_THT:CP_Radial_D6.3mm_P2.50mm -> Capacitor_SMD:C_0805_2012Metric_Pad1.15x1.40mm_HandSolder; symbol Device:CP -> Device:C; Digikey 493-11317-1-ND -> 1276-6455-1-ND; MPN UPS1C100MDD1TD -> CL21A106KOQNNNG; Manufacturer Nichicon -> Samsung
- R1102, R1106: value 10 -> 10R
- R1108, R1109: value 180 -> 180R
Other:
- moved on the sheet: C1112
Changed lines of the file:
@@
 $Descr A4 11693 8268
 encoding utf-8
-Sheet 9 12
+Sheet 11 12
 Title "Neotron Common Hardware - Ethernet MAC/PHY"
 Date "2021-01-01"
@@
 $EndComp
 $Comp
-L Device:CP C1105
+L Device:C C1105
 U 1 1 6084ED3D
 P 5250 5750
 F 0 "C1105" H 5368 5796 50  0000 L CNN
 F 1 "10u Low ESR" H 5368 5705 50  0000 L CNN
-F 2 "Capacitor_THT:CP_Radial_D6.3mm_P2.50mm" H 5288 5600 50  0001 C CNN
+F 2 "Capacitor_SMD:C_0805_2012Metric_Pad1.15x1.40mm_HandSolder" H 5288 5600 50  0001 C CNN
 F 3 "~" H 5250 5750 50  0001 C CNN
 F 4 "0" H 5250 5750 50  0001 C CNN "DNP"
-F 5 "493-11317-1-ND" H 5250 5750 50  0001 C CNN "Digikey"
-F 6 "UPS1C100MDD1TD" H 5250 5750 50  0001 C CNN "MPN"
-F 7 "Nichicon" H 5250 5750 50  0001 C CNN "Manufacturer"
+F 5 "1276-6455-1-ND" H 5250 5750 50  0001 C CNN "Digikey"
+F 6 "CL21A106KOQNNNG" H 5250 5750 50  0001 C CNN "MPN"
+F 7 "Samsung" H 5250 5750 50  0001 C CNN "Manufacturer"
 	1    5250 5750
 	1    0    0    -1
@@
 L Device:C C1112
 U 1 1 608563EB
-P 3750 7250
-F 0 "C1112" H 3865 7296 50  0000 L CNN
-F 1 "1n" H 3865 7205 50  0000 L CNN
-F 2 "Capacitor_SMD:C_0805_2012Metric_Pad1.15x1.40mm_HandSolder" H 3788 7100 50  0001 C CNN
-F 3 "~" H 3750 7250 50  0001 C CNN
-F 4 "0" H 3750 7250 50  0001 C CNN "DNP"
-F 5 "1276-2424-1-ND" H 3750 7250 50  0001 C CNN "Digikey"
-F 6 "CL21B102KBANFNC" H 3750 7250 50  0001 C CNN "MPN"
-F 7 "Samsung" H 3750 7250 50  0001 C CNN "Manufacturer"
-	1    3750 7250
+P 3800 7250
+F 0 "C1112" H 3915 7296 50  0000 L CNN
+F 1 "1n" H 3915 7205 50  0000 L CNN
+F 2 "Capacitor_SMD:C_0805_2012Metric_Pad1.15x1.40mm_HandSolder" H 3838 7100 50  0001 C CNN
+F 3 "~" H 3800 7250 50  0001 C CNN
+F 4 "0" H 3800 7250 50  0001 C CNN "DNP"
+F 5 "1276-2424-1-ND" H 3800 7250 50  0001 C CNN "Digikey"
+F 6 "CL21B102KBANFNC" H 3800 7250 50  0001 C CNN "MPN"
+F 7 "Samsung" H 3800 7250 50  0001 C CNN "Manufacturer"
+	1    3800 7250
 	1    0    0    -1
 $EndComp
@@
 	1    0    0    -1
 $EndComp
-Text Notes 3750 7000 1    50   ~ 0
+Text Notes 3825 7000 1    50   ~ 0
 For VDDTX
-Text Notes 3350 7000 1    50   ~ 0
+Text Notes 3375 7000 1    50   ~ 0
 For VDDPLL
-Text Notes 2450 7000 1    50   ~ 0
+Text Notes 2475 7000 1    50   ~ 0
 For VDDTX
-Text Notes 2900 7000 1    50   ~ 0
+Text Notes 2925 7000 1    50   ~ 0
 For VDD
-Text Notes 2000 7000 1    50   ~ 0
+Text Notes 2025 7000 1    50   ~ 0
 For VDDRX
-Text Notes 1550 7000 1    50   ~ 0
+Text Notes 1575 7000 1    50   ~ 0
 For VDDPLL
-Text Notes 1100 7000 1    50   ~ 0
+Text Notes 1125 7000 1    50   ~ 0
 For VDDOSC
 $Comp
@@
 P 8000 3900
 F 0 "R1108" V 8100 3900 50  0000 C CNN
-F 1 "180" V 7900 3900 50  0000 C CNN
+F 1 "180R" V 7900 3900 50  0000 C CNN
 F 2 "Resistor_SMD:R_0805_2012Metric_Pad1.15x1.40mm_HandSolder" V 7930 3900 50  0001 C CNN
 F 3 "~" H 8000 3900 50  0001 C CNN
@@
 P 7750 4100
 F 0 "R1109" V 7850 4100 50  0000 C CNN
-F 1 "180" V 7650 4100 50  0000 C CNN
+F 1 "180R" V 7650 4100 50  0000 C CNN
 F 2 "Resistor_SMD:R_0805_2012Metric_Pad1.15x1.40mm_HandSolder" V 7680 4100 50  0001 C CNN
 F 3 "~" H 7750 4100 50  0001 C CNN
@@
 P 6950 3050
 F 0 "R1106" V 7050 3050 50  0000 C CNN
-F 1 "10" V 6850 3050 50  0000 C CNN
+F 1 "10R" V 6850 3050 50  0000 C CNN
 F 2 "Resistor_SMD:R_0805_2012Metric_Pad1.15x1.40mm_HandSolder" V 6880 3050 50  0001 C CNN
 F 3 "~" H 6950 3050 50  0001 C CNN
@@
 P 6950 1900
 F 0 "R1102" V 7050 1900 50  0000 C CNN
-F 1 "10" V 6850 1900 50  0000 C CNN
+F 1 "10R" V 6850 1900 50  0000 C CNN
 F 2 "Resistor_SMD:R_0805_2012Metric_Pad1.15x1.40mm_HandSolder" V 6880 1900 50  0001 C CNN
 F 3 "~" H 6950 1900 50  0001 C CNN
@@
 L power:GND #PWR01116
 U 1 1 60A2DE94
-P 3750 7550
-F 0 "#PWR01116" H 3750 7300 50  0001 C CNN
-F 1 "GND" H 3755 7377 50  0000 C CNN
-F 2 "" H 3750 7550 50  0001 C CNN
-F 3 "" H 3750 7550 50  0001 C CNN
-	1    3750 7550
-	1    0    0    -1
-$EndComp
-Wire Wire Line
-	3750 7050 3750 7100
-Wire Wire Line
-	3750 7400 3750 7450
-Wire Wire Line
-	3750 7450 3350 7450
-Connection ~ 3750 7450
-Wire Wire Line
-	3750 7450 3750 7550
+P 3800 7550
+F 0 "#PWR01116" H 3800 7300 50  0001 C CNN
+F 1 "GND" H 3805 7377 50  0000 C CNN
+F 2 "" H 3800 7550 50  0001 C CNN
+F 3 "" H 3800 7550 50  0001 C CNN
+	1    3800 7550
+	1    0    0    -1
+$EndComp
+Wire Wire Line
+	3800 7050 3800 7100
+Wire Wire Line
+	3800 7400 3800 7450
+Wire Wire Line
+	3800 7450 3350 7450
+Connection ~ 3800 7450
+Wire Wire Line
+	3800 7450 3800 7550
 Wire Wire Line
 	3350 7050 3350 7100
@@
 Connection ~ 3350 7050
 Wire Wire Line
-	3350 7050 3750 7050
+	3350 7050 3800 7050
 Wire Wire Line
 	3350 7450 2900 7450

Commit message: Added 12-bit video DAC.
Also had to change footprints to suit Kicad 5.1.9
Parts:
- C75: renamed from C1106; footprint Capacitor_SMD:C_0805_2012Metric_Pad1.15x1.40mm_HandSolder -> Capacitor_SMD:C_0805_2012Metric_Pad1.18x1.45mm_HandSolder
- C76: renamed from C1107; footprint Capacitor_SMD:C_0805_2012Metric_Pad1.15x1.40mm_HandSolder -> Capacitor_SMD:C_0805_2012Metric_Pad1.18x1.45mm_HandSolder
- C77: renamed from C1108; footprint Capacitor_SMD:C_0805_2012Metric_Pad1.15x1.40mm_HandSolder -> Capacitor_SMD:C_0805_2012Metric_Pad1.18x1.45mm_HandSolder
- C78: renamed from C1109; footprint Capacitor_SMD:C_0805_2012Metric_Pad1.15x1.40mm_HandSolder -> Capacitor_SMD:C_0805_2012Metric_Pad1.18x1.45mm_HandSolder
- C79: renamed from C1110; footprint Capacitor_SMD:C_0805_2012Metric_Pad1.15x1.40mm_HandSolder -> Capacitor_SMD:C_0805_2012Metric_Pad1.18x1.45mm_HandSolder
- C80: renamed from C1111; footprint Capacitor_SMD:C_0805_2012Metric_Pad1.15x1.40mm_HandSolder -> Capacitor_SMD:C_0805_2012Metric_Pad1.18x1.45mm_HandSolder
- C81: renamed from C1112; footprint Capacitor_SMD:C_0805_2012Metric_Pad1.15x1.40mm_HandSolder -> Capacitor_SMD:C_0805_2012Metric_Pad1.18x1.45mm_HandSolder
- C82: renamed from C1105; footprint Capacitor_SMD:C_0805_2012Metric_Pad1.15x1.40mm_HandSolder -> Capacitor_SMD:C_0805_2012Metric_Pad1.18x1.45mm_HandSolder
- C83: renamed from C1103; footprint Capacitor_SMD:C_0805_2012Metric_Pad1.15x1.40mm_HandSolder -> Capacitor_SMD:C_0805_2012Metric_Pad1.18x1.45mm_HandSolder
- C84: renamed from C1104; footprint Capacitor_SMD:C_0805_2012Metric_Pad1.15x1.40mm_HandSolder -> Capacitor_SMD:C_0805_2012Metric_Pad1.18x1.45mm_HandSolder
- C85: renamed from C1101; footprint Capacitor_SMD:C_0805_2012Metric_Pad1.15x1.40mm_HandSolder -> Capacitor_SMD:C_0805_2012Metric_Pad1.18x1.45mm_HandSolder
- C86: renamed from C1102; footprint Capacitor_SMD:C_0805_2012Metric_Pad1.15x1.40mm_HandSolder -> Capacitor_SMD:C_0805_2012Metric_Pad1.18x1.45mm_HandSolder
- R84: renamed from R1105; footprint Resistor_SMD:R_0805_2012Metric_Pad1.15x1.40mm_HandSolder -> Resistor_SMD:R_0805_2012Metric_Pad1.20x1.40mm_HandSolder
- R85: renamed from R1112; footprint Resistor_SMD:R_0805_2012Metric_Pad1.15x1.40mm_HandSolder -> Resistor_SMD:R_0805_2012Metric_Pad1.20x1.40mm_HandSolder
- R86: renamed from R1111; footprint Resistor_SMD:R_0805_2012Metric_Pad1.15x1.40mm_HandSolder -> Resistor_SMD:R_0805_2012Metric_Pad1.20x1.40mm_HandSolder
- R87: renamed from R1101; footprint Resistor_SMD:R_0805_2012Metric_Pad1.15x1.40mm_HandSolder -> Resistor_SMD:R_0805_2012Metric_Pad1.20x1.40mm_HandSolder
- R88: renamed from R1103; footprint Resistor_SMD:R_0805_2012Metric_Pad1.15x1.40mm_HandSolder -> Resistor_SMD:R_0805_2012Metric_Pad1.20x1.40mm_HandSolder
- R89: renamed from R1104; footprint Resistor_SMD:R_0805_2012Metric_Pad1.15x1.40mm_HandSolder -> Resistor_SMD:R_0805_2012Metric_Pad1.20x1.40mm_HandSolder
- R90: renamed from R1107; footprint Resistor_SMD:R_0805_2012Metric_Pad1.15x1.40mm_HandSolder -> Resistor_SMD:R_0805_2012Metric_Pad1.20x1.40mm_HandSolder
- R91: renamed from R1102; footprint Resistor_SMD:R_0805_2012Metric_Pad1.15x1.40mm_HandSolder -> Resistor_SMD:R_0805_2012Metric_Pad1.20x1.40mm_HandSolder
- R92: renamed from R1106; footprint Resistor_SMD:R_0805_2012Metric_Pad1.15x1.40mm_HandSolder -> Resistor_SMD:R_0805_2012Metric_Pad1.20x1.40mm_HandSolder
- R93: renamed from R1109; footprint Resistor_SMD:R_0805_2012Metric_Pad1.15x1.40mm_HandSolder -> Resistor_SMD:R_0805_2012Metric_Pad1.20x1.40mm_HandSolder
- R94: renamed from R1108; footprint Resistor_SMD:R_0805_2012Metric_Pad1.15x1.40mm_HandSolder -> Resistor_SMD:R_0805_2012Metric_Pad1.20x1.40mm_HandSolder
- R95: renamed from R1110; footprint Resistor_SMD:R_0805_2012Metric_Pad1.15x1.40mm_HandSolder -> Resistor_SMD:R_0805_2012Metric_Pad1.20x1.40mm_HandSolder
- renumbered J1101 to J19, U1101 to U17, Y1101 to Y3

Commit message: Add 4-bit Video DAC, and re-wire BMC.
Now the BMC is an SPI device, and has a four-wire UART.
Parts:
- renumbered C75 to C1101, C76 to C1102, C77 to C1103, C78 to C1104, C79 to C1105, C80 to C1106, C81 to C1107, C82 to C1108, C83 to C1109, C84 to C1110, C85 to C1111, C86 to C1112, J19 to J1101, R84 to R1101, R85 to R1102, R86 to R1103, R87 to R1104, R88 to R1105, R89 to R1106, R90 to R1107, R91 to R1108, R92 to R1109, R93 to R1110, R94 to R1111, R95 to R1112, U17 to U1101, Y3 to Y1101

Commit message: Tidy up part nos and swapped I2C/UART on BMC.
Mark all resistors as 1% if not specified.
Added some Mouser part numbers.
BMC can now be programmed over UART.
Parts:
- C1101, C1102, C1103, C1104, C1105: Mouser (none) -> 594-K104K15X7RF5TL2
- J1101: Mouser (none) -> 523-RJMG1BD3B8K1ANR
- R1101: value 100k -> 100k 1%
- R1102: Digikey MCF0805FT12K4CT-ND -> RMCF0805FT12K4CT-ND
- R1103: value 1M -> 1M 1%; Digikey RMCF0805FG1M00-ND -> RMCF0805FT1M00CT-ND; MPN RMCF0805FG1M00 -> RMCF0805FT1M00
- R1108, R1109: value 10R -> 10R 1%
- R1110, R1111: value 180R -> 180R 1%
- U1101: Mouser (none) -> 579-ENC424J600-I/PT
- Y1101: Mouser (none) -> 815-ABL-25-B2F
Other:
- moved on the sheet: R1101, R1110, R1111
Changed lines of the file:
@@
 P 9250 3700
 F 0 "J1101" H 9150 4450 50  0000 L CNN
-F 1 "RJ45 MagJack" H 8600 4350 50  0000 L CNN
+F 1 "RJ45 MagJack" H 9000 4350 50  0000 L CNN
 F 2 "Connector_RJ:RJ45_Amphenol_RJMG1BD3B8K1ANR" H 9250 4400 50  0001 C CNN
 F 3 "https://www.amphenolcanada.com/ProductSearch/Drawings/AC/RJMG1BD3B8K1ANR.PDF" H 9250 4500 50  0001 C CNN
@@
 F 6 "RJMG1BD3B8K1ANR" H 9250 3700 50  0001 C CNN "MPN"
 F 7 "Amphenol" H 9250 3700 50  0001 C CNN "Manufacturer"
+F 8 "523-RJMG1BD3B8K1ANR" H 9250 3700 50  0001 C CNN "Mouser"
 	1    9250 3700
 	1    0    0    -1
 $EndComp
-Text Notes 1300 2850 0    50   ~ 0
+Text Notes 1150 2850 0    50   ~ 0
 Ethernet Jack with integrated magnetics.\nGreen LED is Activity.\nYellow LED is 100base-T mode active.
 Text HLabel 2850 3700 0    50   Input ~ 0
@@
 F 6 "ENC424J600-I/PT" H 4200 4400 50  0001 C CNN "MPN"
 F 7 "Microchip" H 4200 4400 50  0001 C CNN "Manufacturer"
+F 8 "579-ENC424J600-I/PT" H 4200 4400 50  0001 C CNN "Mouser"
 	1    4200 4400
 	1    0    0    -1
 $EndComp
-Text HLabel 2850 3300 0    50   Output ~ 0
+Text HLabel 2700 3300 0    50   Output ~ 0
 ~IRQ
 $Comp
@@
 F 6 "ABL-25.000MHZ-B2F" H 6700 5050 50  0001 C CNN "MPN"
 F 7 "Abracon" H 6700 5050 50  0001 C CNN "Manufacturer"
+F 8 "815-ABL-25-B2F" H 6700 5050 50  0001 C CNN "Mouser"
 	1    6700 5050
 	1    0    0    -1
@@
 $EndComp
 Wire Wire Line
-	7550 4000 7550 3900
-Wire Wire Line
-	7550 3900 7850 3900
+	7500 4000 7500 3900
+Wire Wire Line
+	7500 3900 7900 3900
 $Comp
 L Device:R R1101
 U 1 1 6082A933
-P 3050 3000
-F 0 "R1101" H 3120 3046 50  0000 L CNN
-F 1 "100k" H 3120 2955 50  0000 L CNN
-F 2 "Resistor_SMD:R_0805_2012Metric_Pad1.20x1.40mm_HandSolder" V 2980 3000 50  0001 C CNN
-F 3 "~" H 3050 3000 50  0001 C CNN
-F 4 "0" H 3050 3000 50  0001 C CNN "DNP"
-F 5 "RMCF0805FT100K-ND" H 3050 3000 50  0001 C CNN "Digikey"
-F 6 "RMCF0805FT100K" H 3050 3000 50  0001 C CNN "MPN"
-F 7 "Stackpole" H 3050 3000 50  0001 C CNN "Manufacturer"
-	1    3050 3000
-	1    0    0    -1
-$EndComp
-Wire Wire Line
-	2850 3300 3050 3300
-Wire Wire Line
-	3050 3300 3050 3150
-Wire Wire Line
-	3050 3300 3300 3300
-Connection ~ 3050 3300
+P 2900 3000
+F 0 "R1101" H 2970 3046 50  0000 L CNN
+F 1 "100k 1%" H 2970 2955 50  0000 L CNN
+F 2 "Resistor_SMD:R_0805_2012Metric_Pad1.20x1.40mm_HandSolder" V 2830 3000 50  0001 C CNN
+F 3 "~" H 2900 3000 50  0001 C CNN
+F 4 "0" H 2900 3000 50  0001 C CNN "DNP"
+F 5 "RMCF0805FT100K-ND" H 2900 3000 50  0001 C CNN "Digikey"
+F 6 "RMCF0805FT100K" H 2900 3000 50  0001 C CNN "MPN"
+F 7 "Stackpole" H 2900 3000 50  0001 C CNN "Manufacturer"
+	1    2900 3000
+	1    0    0    -1
+$EndComp
+Wire Wire Line
+	2700 3300 2900 3300
+Wire Wire Line
+	2900 3300 2900 3150
+Connection ~ 2900 3300
 $Comp
 L power:+3V3 #PWR01102
 U 1 1 6082BF84
-P 3050 2750
-F 0 "#PWR01102" H 3050 2600 50  0001 C CNN
-F 1 "+3V3" H 3065 2923 50  0000 C CNN
-F 2 "" H 3050 2750 50  0001 C CNN
-F 3 "" H 3050 2750 50  0001 C CNN
-	1    3050 2750
-	1    0    0    -1
-$EndComp
-Wire Wire Line
-	3050 2750 3050 2850
+P 2900 2750
+F 0 "#PWR01102" H 2900 2600 50  0001 C CNN
+F 1 "+3V3" H 2915 2923 50  0000 C CNN
+F 2 "" H 2900 2750 50  0001 C CNN
+F 3 "" H 2900 2750 50  0001 C CNN
+	1    2900 2750
+	1    0    0    -1
+$EndComp
+Wire Wire Line
+	2900 2750 2900 2850
 $Comp
 L power:+3V3 #PWR01104
@@
 P 5700 4900
 F 0 "R1103" V 5800 4900 50  0000 C CNN
-F 1 "1M" V 5600 4900 50  0000 C CNN
+F 1 "1M 1%" V 5600 4900 50  0000 C CNN
 F 2 "Resistor_SMD:R_0805_2012Metric_Pad1.20x1.40mm_HandSolder" V 5630 4900 50  0001 C CNN
 F 3 "~" H 5700 4900 50  0001 C CNN
 F 4 "0" H 5700 4900 50  0001 C CNN "DNP"
-F 5 "RMCF0805FG1M00-ND" H 5700 4900 50  0001 C CNN "Digikey"
-F 6 "RMCF0805FG1M00" H 5700 4900 50  0001 C CNN "MPN"
+F 5 "RMCF0805FT1M00CT-ND" H 5700 4900 50  0001 C CNN "Digikey"
+F 6 "RMCF0805FT1M00" H 5700 4900 50  0001 C CNN "MPN"
 F 7 "Stackpole" H 5700 4900 50  0001 C CNN "Manufacturer"
 	1    5700 4900
@@
 F 6 "K104K15X7RF5TL2" H 2900 7250 50  0001 C CNN "MPN"
 F 7 "Vishay" H 2900 7250 50  0001 C CNN "Manufacturer"
+F 8 "594-K104K15X7RF5TL2" H 2900 7250 50  0001 C CNN "Mouser"
 	1    2900 7250
 	1    0    0    -1
@@
 F 6 "K104K15X7RF5TL2" H 2450 7250 50  0001 C CNN "MPN"
 F 7 "Vishay" H 2450 7250 50  0001 C CNN "Manufacturer"
+F 8 "594-K104K15X7RF5TL2" H 2450 7250 50  0001 C CNN "Mouser"
 	1    2450 7250
 	1    0    0    -1
@@
 F 6 "K104K15X7RF5TL2" H 2000 7250 50  0001 C CNN "MPN"
 F 7 "Vishay" H 2000 7250 50  0001 C CNN "Manufacturer"
+F 8 "594-K104K15X7RF5TL2" H 2000 7250 50  0001 C CNN "Mouser"
 	1    2000 7250
 	1    0    0    -1
@@
 F 6 "K104K15X7RF5TL2" H 1550 7250 50  0001 C CNN "MPN"
 F 7 "Vishay" H 1550 7250 50  0001 C CNN "Manufacturer"
+F 8 "594-K104K15X7RF5TL2" H 1550 7250 50  0001 C CNN "Mouser"
 	1    1550 7250
 	1    0    0    -1
@@
 F 6 "K104K15X7RF5TL2" H 1100 7250 50  0001 C CNN "MPN"
 F 7 "Vishay" H 1100 7250 50  0001 C CNN "Manufacturer"
+F 8 "594-K104K15X7RF5TL2" H 1100 7250 50  0001 C CNN "Mouser"
 	1    1100 7250
 	1    0    0    -1
@@
 F 3 "~" H 5400 5200 50  0001 C CNN
 F 4 "0" H 5400 5200 50  0001 C CNN "DNP"
-F 5 "MCF0805FT12K4CT-ND" H 5400 5200 50  0001 C CNN "Digikey"
+F 5 "RMCF0805FT12K4CT-ND" H 5400 5200 50  0001 C CNN "Digikey"
 F 6 "RMCF0805FT12K4" H 5400 5200 50  0001 C CNN "MPN"
 F 7 "Stackpole" H 5400 5200 50  0001 C CNN "Manufacturer"
@@
 L Device:R R1111
 U 1 1 6085F410
-P 8000 3900
-F 0 "R1111" V 8100 3900 50  0000 C CNN
-F 1 "180R" V 7900 3900 50  0000 C CNN
-F 2 "Resistor_SMD:R_0805_2012Metric_Pad1.20x1.40mm_HandSolder" V 7930 3900 50  0001 C CNN
-F 3 "~" H 8000 3900 50  0001 C CNN
-F 4 "0" H 8000 3900 50  0001 C CNN "DNP"
-F 5 "RMCF0805FT180R-ND" H 8000 3900 50  0001 C CNN "Digikey"
-F 6 "RMCF0805FT180R" H 8000 3900 50  0001 C CNN "MPN"
-F 7 "Stackpole" H 8000 3900 50  0001 C CNN "Manufacturer"
-	1    8000 3900
+P 8050 3900
+F 0 "R1111" V 8150 3900 50  0000 C CNN
+F 1 "180R 1%" V 7950 3900 50  0000 C CNN
+F 2 "Resistor_SMD:R_0805_2012Metric_Pad1.20x1.40mm_HandSolder" V 7980 3900 50  0001 C CNN
+F 3 "~" H 8050 3900 50  0001 C CNN
+F 4 "0" H 8050 3900 50  0001 C CNN "DNP"
+F 5 "RMCF0805FT180R-ND" H 8050 3900 50  0001 C CNN "Digikey"
+F 6 "RMCF0805FT180R" H 8050 3900 50  0001 C CNN "MPN"
+F 7 "Stackpole" H 8050 3900 50  0001 C CNN "Manufacturer"
+	1    8050 3900
 	0    -1   -1   0
 $EndComp
 Wire Wire Line
-	8150 3900 8350 3900
+	8200 3900 8350 3900
 $Comp
 L Device:R R1110
 U 1 1 6085F9CE
-P 7750 4100
-F 0 "R1110" V 7850 4100 50  0000 C CNN
-F 1 "180R" V 7650 4100 50  0000 C CNN
-F 2 "Resistor_SMD:R_0805_2012Metric_Pad1.20x1.40mm_HandSolder" V 7680 4100 50  0001 C CNN
-F 3 "~" H 7750 4100 50  0001 C CNN
-F 4 "0" H 7750 4100 50  0001 C CNN "DNP"
-F 5 "RMCF0805FT180R-ND" H 7750 4100 50  0001 C CNN "Digikey"
-F 6 "RMCF0805FT180R" H 7750 4100 50  0001 C CNN "MPN"
-F 7 "Stackpole" H 7750 4100 50  0001 C CNN "Manufacturer"
-	1    7750 4100
+P 7700 4100
+F 0 "R1110" V 7800 4100 50  0000 C CNN
+F 1 "180R 1%" V 7600 4100 50  0000 C CNN
+F 2 "Resistor_SMD:R_0805_2012Metric_Pad1.20x1.40mm_HandSolder" V 7630 4100 50  0001 C CNN
+F 3 "~" H 7700 4100 50  0001 C CNN
+F 4 "0" H 7700 4100 50  0001 C CNN "DNP"
+F 5 "RMCF0805FT180R-ND" H 7700 4100 50  0001 C CNN "Digikey"
+F 6 "RMCF0805FT180R" H 7700 4100 50  0001 C CNN "MPN"
+F 7 "Stackpole" H 7700 4100 50  0001 C CNN "Manufacturer"
+	1    7700 4100
 	0    -1   -1   0
 $EndComp
 Wire Wire Line
-	7900 4100 8350 4100
+	7850 4100 8350 4100
 $Comp
 L power:GND #PWR01114
@@
 P 6950 3050
 F 0 "R1109" V 7050 3050 50  0000 C CNN
-F 1 "10R" V 6850 3050 50  0000 C CNN
+F 1 "10R 1%" V 6850 3050 50  0000 C CNN
 F 2 "Resistor_SMD:R_0805_2012Metric_Pad1.20x1.40mm_HandSolder" V 6880 3050 50  0001 C CNN
 F 3 "~" H 6950 3050 50  0001 C CNN
@@
 P 6950 1900
 F 0 "R1108" V 7050 1900 50  0000 C CNN
-F 1 "10R" V 6850 1900 50  0000 C CNN
+F 1 "10R 1%" V 6850 1900 50  0000 C CNN
 F 2 "Resistor_SMD:R_0805_2012Metric_Pad1.20x1.40mm_HandSolder" V 6880 1900 50  0001 C CNN
 F 3 "~" H 6950 1900 50  0001 C CNN
@@
 	7200 2250 7200 2300
 Wire Wire Line
-	5100 4100 7600 4100
-Wire Wire Line
-	5100 4000 7550 4000
+	5100 4100 7550 4100
+Wire Wire Line
+	5100 4000 7500 4000
 Wire Wire Line
 	5100 3700 6100 3700
@@
 Wire Wire Line
 	8250 4200 8250 4500
+Wire Wire Line
+	2900 3300 3300 3300
 $EndSCHEMATC

Commit message: Changes to BMC
* Swapped BUTTON_PWR and SYS_RESET to avoid DRC issue
* Split PSU and BMC into two separate sheets
* Swapped some pins on the STM32 to make it compatible with more
alternatives
Parts:
- renumbered C1101 to C1001, C1102 to C1002, C1103 to C1003, C1104 to C1004, C1105 to C1005, C1106 to C1006, C1107 to C1007, C1108 to C1008, C1109 to C1009, C1110 to C1010, C1111 to C1011, C1112 to C1012, J1101 to J1001, R1101 to R1001, R1102 to R1002, R1103 to R1003, R1104 to R1004, R1105 to R1005, R1106 to R1006, R1107 to R1007, R1108 to R1008, R1109 to R1009, R1110 to R1010, R1111 to R1011, R1112 to R1012, U1101 to U1001, Y1101 to Y1001

Commit message: Merge in more changes.
Mostly lowering voltage tolerances to minimum required.
Parts:
- C1001, C1002, C1003, C1004, C1005: value 100n -> 100nF; MPN K104K15X7RF5TL2 -> CPL-CAP-X7R-0805-100NF-50V; Tolerance (none) -> X5R; Voltage (none) -> 10V
- C1006, C1007: value 1n -> 1nF; Tolerance (none) -> X5R; Voltage (none) -> 10V
- C1008: value 10u Low ESR -> 10uF; MPN CL21A106KOQNNNG -> CPL-CAP-X5R-0805-10UF-16V; Tolerance (none) -> X5R; Voltage (none) -> 6.3V
- C1009, C1010: Tolerance (none) -> C0G; Voltage (none) -> 10V
- C1011, C1012: value 10n -> 10nF; Tolerance (none) -> X5R; Voltage (none) -> 50V
- R1001: value 100k 1% -> 100k; Tolerance (none) -> 1%
- R1002: value 12k4 1% -> 12k4; Tolerance (none) -> 1%
- R1003: value 1M 1% -> 1M; Tolerance (none) -> 1%
- R1004, R1005, R1006, R1007: value 49R9 1% -> 49R9; Tolerance (none) -> 1%
- R1008, R1009: value 10R 1% -> 10R; Tolerance (none) -> 1%
- R1010, R1011: value 180R 1% -> 180R; Tolerance (none) -> 1%
Other:
- note added: "VCAP must be low-ESP, e.g.\ntantalum or ceramic"
