File: Kicad/sdcard.sch (KiCad schematic (older format))
At the start: 4 parts, among them J701 SD_Card

Commit message: Merge in more changes.
Mostly lowering voltage tolerances to minimum required.
Parts:
- C701, C702: Tolerance (none) -> X5R; Voltage (none) -> 10V
- RN701: value 8x10k -> 10k; Tolerance (none) -> 2%
Changed lines of the file:
@@
 $Descr A4 11693 8268
 encoding utf-8
-Sheet 7 18
-Title "Neotron Common Hardware"
-Date "2021-06-18"
+Sheet 3 18
+Title "Neotron Common Hardware - SD Card Slot"
+Date "2021-06-10"
 Rev "[Uncontrolled]"
 Comp "https://neotron-compute.github.io/"
@@
 F 8 "581-145638009211859+" H 5950 3750 50  0001 C CNN "Mouser"
 F 9 "~" H 5950 3750 50  0001 C CNN "LCSC Part#"
+F 10 "~" H 5950 3750 50  0001 C CNN "Tolerance"
+F 11 "~" H 5950 3750 50  0001 C CNN "Voltage"
 	1    5950 3750
 	1    0    0    -1
@@
 F 3 "~" H 8250 3750 50  0001 C CNN
 F 4 "0" H 8250 3750 50  0001 C CNN "DNP"
-F 5 "" H 8250 3750 50  0001 C CNN "Digikey"
+F 5 "~" H 8250 3750 50  0001 C CNN "Digikey"
 F 6 "CPL-CAP-X5R-0805-10UF-16V" H 8250 3750 50  0001 C CNN "MPN"
 F 7 "CPL" H 8250 3750 50  0001 C CNN "Manufacturer"
 F 8 "C15850" H 8250 3750 50  0001 C CNN "LCSC Part#"
+F 9 "X5R" H 8250 3750 50  0001 C CNN "Tolerance"
+F 10 "10V" H 8250 3750 50  0001 C CNN "Voltage"
+F 11 "~" H 8250 3750 50  0001 C CNN "Mouser"
 	1    8250 3750
 	1    0    0    -1
@@
 F 3 "~" H 8800 3750 50  0001 C CNN
 F 4 "0" H 8800 3750 50  0001 C CNN "DNP"
-F 5 "" H 8800 3750 50  0001 C CNN "Digikey"
+F 5 "~" H 8800 3750 50  0001 C CNN "Digikey"
 F 6 "CPL-CAP-X7R-0805-100NF-50V" H 8800 3750 50  0001 C CNN "MPN"
 F 7 "CPL" H 8800 3750 50  0001 C CNN "Manufacturer"
-F 8 "" H 8800 3750 50  0001 C CNN "Mouser"
+F 8 "~" H 8800 3750 50  0001 C CNN "Mouser"
 F 9 "C49678" H 8800 3750 50  0001 C CNN "LCSC Part#"
+F 10 "X5R" H 8800 3750 50  0001 C CNN "Tolerance"
+F 11 "10V" H 8800 3750 50  0001 C CNN "Voltage"
 	1    8800 3750
 	1    0    0    -1
@@
 P 4300 2500
 F 0 "RN701" H 4300 2800 50  0000 C CNN
-F 1 "8x10k" H 4300 2700 50  0000 C CNN
+F 1 "10k" H 4300 2700 50  0000 C CNN
 F 2 "Resistor_THT:R_Array_SIP9" V 4675 2500 50  0001 C CNN
 F 3 "http://www.vishay.com/docs/31509/csc.pdf" H 4300 2500 50  0001 C CNN
@@
 F 8 "652-4609X-1LF-10K" H 4300 2500 50  0001 C CNN "Mouser"
 F 9 "~" H 4300 2500 50  0001 C CNN "LCSC Part#"
+F 10 "2%" H 4300 2500 50  0001 C CNN "Tolerance"
+F 11 "~" H 4300 2500 50  0001 C CNN "Voltage"
 	1    4300 2500
 	1    0    0    -1
