File: Kicad/io_exp.sch (KiCad schematic (older format))
At the start: 4 parts, among them U1801 MCP23S17_SO, U1802 74HC245

Commit message: Merge in more changes.
Mostly lowering voltage tolerances to minimum required.
Parts:
- C1801, C1802: Tolerance (none) -> X5R; Voltage (none) -> 10V
- U1801: symbol Interface_Expansion:MCP23S17_SO -> neotron-pico:MCP23S17_SO
- U1802: Mouser (none) -> 595-SN74HC245NSR
Changed lines of the file:
@@
 $Descr A4 11693 8268
 encoding utf-8
-Sheet 18 18
+Sheet 10 18
 Title ""
 Date "2021-06-10"
@@
 $EndDescr
 $Comp
-L Interface_Expansion:MCP23S17_SO U1801
+L neotron-pico:MCP23S17_SO U1801
 U 1 1 60EED5B0
 P 4425 3050
@@
 F 7 "Microchip" H 4425 3050 50  0001 C CNN "Manufacturer"
 F 8 "C145413" H 4425 3050 50  0001 C CNN "LCSC Part#"
+F 9 "~" H 4425 3050 50  0001 C CNN "Mouser"
+F 10 "~" H 4425 3050 50  0001 C CNN "Tolerance"
+F 11 "~" H 4425 3050 50  0001 C CNN "Voltage"
 	1    4425 3050
 	1    0    0    -1
@@
 F 7 "Texas Instruments" H 6050 3650 50  0001 C CNN "Manufacturer"
 F 8 "C5625" H 6050 3650 50  0001 C CNN "LCSC Part#"
+F 9 "595-SN74HC245NSR" H 6050 3650 50  0001 C CNN "Mouser"
+F 10 "~" H 6050 3650 50  0001 C CNN "Tolerance"
+F 11 "~" H 6050 3650 50  0001 C CNN "Voltage"
 	1    6050 3650
 	1    0    0    -1
@@
 F 3 "~" H 7900 2500 50  0001 C CNN
 F 4 "0" H 7900 2500 50  0001 C CNN "DNP"
-F 5 "" H 7900 2500 50  0001 C CNN "Digikey"
+F 5 "~" H 7900 2500 50  0001 C CNN "Digikey"
 F 6 "CPL-CAP-X7R-0805-100NF-50V" H 7900 2500 50  0001 C CNN "MPN"
 F 7 "CPL" H 7900 2500 50  0001 C CNN "Manufacturer"
-F 8 "" H 7900 2500 50  0001 C CNN "Mouser"
+F 8 "~" H 7900 2500 50  0001 C CNN "Mouser"
 F 9 "C49678" H 7900 2500 50  0001 C CNN "LCSC Part#"
+F 10 "X5R" H 7900 2500 50  0001 C CNN "Tolerance"
+F 11 "10V" H 7900 2500 50  0001 C CNN "Voltage"
 	1    7900 2500
 	1    0    0    -1
@@
 F 3 "~" H 8375 2500 50  0001 C CNN
 F 4 "0" H 8375 2500 50  0001 C CNN "DNP"
-F 5 "" H 8375 2500 50  0001 C CNN "Digikey"
+F 5 "~" H 8375 2500 50  0001 C CNN "Digikey"
 F 6 "CPL-CAP-X7R-0805-100NF-50V" H 8375 2500 50  0001 C CNN "MPN"
 F 7 "CPL" H 8375 2500 50  0001 C CNN "Manufacturer"
-F 8 "" H 8375 2500 50  0001 C CNN "Mouser"
+F 8 "~" H 8375 2500 50  0001 C CNN "Mouser"
 F 9 "C49678" H 8375 2500 50  0001 C CNN "LCSC Part#"
+F 10 "X5R" H 8375 2500 50  0001 C CNN "Tolerance"
+F 11 "10V" H 8375 2500 50  0001 C CNN "Voltage"
 	1    8375 2500
 	1    0    0    -1

Commit message: Fixups after last copy-over.
Parts:
- U1801: symbol neotron-pico:MCP23S17_SO -> Neotron-Common-Hardware:MCP23S17_SO
Changed lines of the file:
@@
 $EndDescr
 $Comp
-L neotron-pico:MCP23S17_SO U1801
+L Neotron-Common-Hardware:MCP23S17_SO U1801
 U 1 1 60EED5B0
 P 4425 3050
