File: Kicad/Neotron-Common-Hardware.kicad_pcb (KiCad board)
At the start: 4 copper layers, 243.8 x 243.8 mm, 264 parts, among them J1001 USB Ports External, J1002 USB Ports Internal, J101 Neotron-Expansion-Slot, J102 Neotron-Expansion-Slot, J103 Neotron-Expansion-Slot, J104 Neotron-Expansion-Slot, J1101 RJ45 MagJack, J201 DE15HD, J601 Line Out, J602 AC'97 Audio Header, J603 CD Audio In, J701 SD_Card, J801 Conn_02x05, J802 DB9_Male_MountingHoles, J901 Jack-DC, J902 Conn_01x06, J903 Conn_01x03, J904 Header, J905 Double-mini-DIN-6, Q901 BC548, SW901 SW_DIP_x01, SW902 SW_DIP_x01, U1001 AP2501, U1002 MIC2005A-2YM5, U1003 MIC2005A-2YM5, U1004 XR22404CG28, U1005 MIC2005A-2YM5, U1006 MIC2005A-2YM5, U101 Neotron-CPU, U1101 ENC424J600, U1201 MCP7940, U201 THS7316, U202 TPD7S019, U601 TLV320AIC23BPW, U602 STX-4335-5BGP-S1, U801 ST3232CDR, U901 5V DC-DC Module, U902 TLV1117 3.3V 1A, U903 MAX1615, U904 STM32F031K6T6, Y1001 12M, Y1101 25M, Y1201 32,768 Hz, Y601 12M

Commit message: Added 12-bit video DAC.
Also had to change footprints to suit Kicad 5.1.9
Parts:
- added C2: 100n, Capacitor_SMD:C_0805_2012Metric_Pad1.18x1.45mm_HandSolder, F.Cu at (176.0, 250.9)
- added C4: 100n, Capacitor_SMD:C_0805_2012Metric_Pad1.18x1.45mm_HandSolder, F.Cu at (180.8, 251.1)
- added C5: 10u 10V, Capacitor_SMD:C_0805_2012Metric_Pad1.18x1.45mm_HandSolder, F.Cu at (176.0, 253.9)
- added C90: 100n, Capacitor_SMD:C_0805_2012Metric_Pad1.18x1.45mm_HandSolder, F.Cu at (189.3, 237.3)
- added C91: 100n, Capacitor_SMD:C_0805_2012Metric_Pad1.18x1.45mm_HandSolder, F.Cu at (194.1, 234.2)
- added C92: 100n, Capacitor_SMD:C_0805_2012Metric_Pad1.18x1.45mm_HandSolder, F.Cu at (184.4, 237.3)
- added C93: 100n, Capacitor_SMD:C_0805_2012Metric_Pad1.18x1.45mm_HandSolder, F.Cu at (189.3, 234.2)
- added C94: 10u 10V, Capacitor_SMD:C_0805_2012Metric_Pad1.18x1.45mm_HandSolder, F.Cu at (208.9, 223.4)
- added C95: 220n, Capacitor_SMD:C_0805_2012Metric_Pad1.18x1.45mm_HandSolder, F.Cu at (184.4, 234.2)
- added J20: DE15HD, Connector_Dsub:DSUB-15-HD_Female_Horizontal_P2.29x1.98mm_EdgePinOffset3.03mm_Housed_MountingHolesOffset4.94mm, F.Cu at (40.8, 246.5)
- added R10: 24k 0.5%, Resistor_SMD:R_0805_2012Metric_Pad1.20x1.40mm_HandSolder, F.Cu at (222.9, 216.7)
- added R100: 75R, Resistor_SMD:R_0805_2012Metric_Pad1.20x1.40mm_HandSolder, F.Cu at (198.8, 237.2)
- added R101: 75R, Resistor_SMD:R_0805_2012Metric_Pad1.20x1.40mm_HandSolder, F.Cu at (213.7, 223.4)
- added R102: DNF, Resistor_SMD:R_0805_2012Metric_Pad1.20x1.40mm_HandSolder, F.Cu at (208.9, 226.4)
- added R103: 1k5, Resistor_SMD:R_0805_2012Metric_Pad1.20x1.40mm_HandSolder, F.Cu at (194.0, 237.2)
- added R104: 1k5, Resistor_SMD:R_0805_2012Metric_Pad1.20x1.40mm_HandSolder, F.Cu at (198.8, 234.2)
- added R105: 24k 0.5%, Resistor_SMD:R_0805_2012Metric_Pad1.20x1.40mm_HandSolder, F.Cu at (262.0, 216.7)
- added R106: 24k 0.5%, Resistor_SMD:R_0805_2012Metric_Pad1.20x1.40mm_HandSolder, F.Cu at (257.2, 219.6)
- added R107: 12k 0.5%, Resistor_SMD:R_0805_2012Metric_Pad1.20x1.40mm_HandSolder, F.Cu at (252.5, 222.6)
- added R108: 24k 0.5%, Resistor_SMD:R_0805_2012Metric_Pad1.20x1.40mm_HandSolder, F.Cu at (247.7, 219.6)
- added R109: 12k 0.5%, Resistor_SMD:R_0805_2012Metric_Pad1.20x1.40mm_HandSolder, F.Cu at (247.7, 216.7)
- added R11: 24k 0.5%, Resistor_SMD:R_0805_2012Metric_Pad1.20x1.40mm_HandSolder, F.Cu at (227.7, 225.5)
- added R110: 24k 0.5%, Resistor_SMD:R_0805_2012Metric_Pad1.20x1.40mm_HandSolder, F.Cu at (257.2, 222.6)
- added R111: 12k 0.5%, Resistor_SMD:R_0805_2012Metric_Pad1.20x1.40mm_HandSolder, F.Cu at (252.5, 216.7)
- added R112: 24k 0.5%, Resistor_SMD:R_0805_2012Metric_Pad1.20x1.40mm_HandSolder, F.Cu at (247.7, 222.6)
- added R113: 12k 0.5%, Resistor_SMD:R_0805_2012Metric_Pad1.20x1.40mm_HandSolder, F.Cu at (252.5, 219.6)
- added R114: 3480 0.5%, Resistor_SMD:R_0805_2012Metric_Pad1.20x1.40mm_HandSolder, F.Cu at (257.2, 216.7)
- added R115: 24k 0.5%, Resistor_SMD:R_0805_2012Metric_Pad1.20x1.40mm_HandSolder, F.Cu at (226.2, 245.7)
- added R116: 24k 0.5%, Resistor_SMD:R_0805_2012Metric_Pad1.20x1.40mm_HandSolder, F.Cu at (226.2, 248.6)
- added R117: 12k 0.5%, Resistor_SMD:R_0805_2012Metric_Pad1.20x1.40mm_HandSolder, F.Cu at (230.9, 245.7)
- added R118: 24k 0.5%, Resistor_SMD:R_0805_2012Metric_Pad1.20x1.40mm_HandSolder, F.Cu at (226.2, 251.6)
- added R119: 12k 0.5%, Resistor_SMD:R_0805_2012Metric_Pad1.20x1.40mm_HandSolder, F.Cu at (230.9, 248.6)
- added R12: 12k 0.5%, Resistor_SMD:R_0805_2012Metric_Pad1.20x1.40mm_HandSolder, F.Cu at (232.4, 222.6)
- added R120: 24k 0.5%, Resistor_SMD:R_0805_2012Metric_Pad1.20x1.40mm_HandSolder, F.Cu at (235.7, 245.7)
- added R121: 12k 0.5%, Resistor_SMD:R_0805_2012Metric_Pad1.20x1.40mm_HandSolder, F.Cu at (230.9, 251.6)
- added R122: 24k 0.5%, Resistor_SMD:R_0805_2012Metric_Pad1.20x1.40mm_HandSolder, F.Cu at (235.7, 248.6)
- added R123: 12k 0.5%, Resistor_SMD:R_0805_2012Metric_Pad1.20x1.40mm_HandSolder, F.Cu at (240.4, 245.7)
- added R124: 3480 0.5%, Resistor_SMD:R_0805_2012Metric_Pad1.20x1.40mm_HandSolder, F.Cu at (235.7, 251.6)
- added R125: 24k 0.5%, Resistor_SMD:R_0805_2012Metric_Pad1.20x1.40mm_HandSolder, F.Cu at (226.2, 231.9)
- added R126: 24k 0.5%, Resistor_SMD:R_0805_2012Metric_Pad1.20x1.40mm_HandSolder, F.Cu at (226.2, 234.9)
- added R127: 12k 0.5%, Resistor_SMD:R_0805_2012Metric_Pad1.20x1.40mm_HandSolder, F.Cu at (230.9, 231.9)
- added R128: 24k 0.5%, Resistor_SMD:R_0805_2012Metric_Pad1.20x1.40mm_HandSolder, F.Cu at (226.2, 237.8)
- added R129: 12k 0.5%, Resistor_SMD:R_0805_2012Metric_Pad1.20x1.40mm_HandSolder, F.Cu at (230.9, 234.9)
- added R13: 24k 0.5%, Resistor_SMD:R_0805_2012Metric_Pad1.20x1.40mm_HandSolder, F.Cu at (237.2, 219.6)
- added R130: 24k 0.5%, Resistor_SMD:R_0805_2012Metric_Pad1.20x1.40mm_HandSolder, F.Cu at (235.7, 231.9)
- added R131: 12k 0.5%, Resistor_SMD:R_0805_2012Metric_Pad1.20x1.40mm_HandSolder, F.Cu at (230.9, 237.8)
- added R132: 24k 0.5%, Resistor_SMD:R_0805_2012Metric_Pad1.20x1.40mm_HandSolder, F.Cu at (235.7, 234.9)
- added R133: 12k 0.5%, Resistor_SMD:R_0805_2012Metric_Pad1.20x1.40mm_HandSolder, F.Cu at (240.4, 231.9)
- added R134: 3480 0.5%, Resistor_SMD:R_0805_2012Metric_Pad1.20x1.40mm_HandSolder, F.Cu at (235.7, 237.8)
- added R14: 12k 0.5%, Resistor_SMD:R_0805_2012Metric_Pad1.20x1.40mm_HandSolder, F.Cu at (237.2, 216.7)
- added R15: 24k 0.5%, Resistor_SMD:R_0805_2012Metric_Pad1.20x1.40mm_HandSolder, F.Cu at (232.4, 219.6)
- added R16: 12k 0.5%, Resistor_SMD:R_0805_2012Metric_Pad1.20x1.40mm_HandSolder, F.Cu at (227.7, 222.6)
- added R17: 24k 0.5%, Resistor_SMD:R_0805_2012Metric_Pad1.20x1.40mm_HandSolder, F.Cu at (222.9, 225.5)
- added R18: 12k 0.5%, Resistor_SMD:R_0805_2012Metric_Pad1.20x1.40mm_HandSolder, F.Cu at (232.4, 216.7)
- added R19: 24k 0.5%, Resistor_SMD:R_0805_2012Metric_Pad1.20x1.40mm_HandSolder, F.Cu at (227.7, 219.6)
- added R2: 10k, Resistor_SMD:R_0805_2012Metric_Pad1.20x1.40mm_HandSolder, F.Cu at (192.4, 247.4)
- added R20: 12k 0.5%, Resistor_SMD:R_0805_2012Metric_Pad1.20x1.40mm_HandSolder, F.Cu at (222.9, 222.6)
- added R21: 24k 0.5%, Resistor_SMD:R_0805_2012Metric_Pad1.20x1.40mm_HandSolder, F.Cu at (227.7, 216.7)
- added R22: 4990 0.5%, Resistor_SMD:R_0805_2012Metric_Pad1.20x1.40mm_HandSolder, F.Cu at (222.9, 219.6)
- added R23: 24k 0.5%, Resistor_SMD:R_0805_2012Metric_Pad1.20x1.40mm_HandSolder, F.Cu at (176.0, 260.0)
- added R3: 10k, Resistor_SMD:R_0805_2012Metric_Pad1.20x1.40mm_HandSolder, F.Cu at (185.6, 251.1)
- added R30: 24k 0.5%, Resistor_SMD:R_0805_2012Metric_Pad1.20x1.40mm_HandSolder, F.Cu at (180.7, 260.0)
- added R36: 24k 0.5%, Resistor_SMD:R_0805_2012Metric_Pad1.20x1.40mm_HandSolder, F.Cu at (215.7, 247.4)
- added R37: 24k 0.5%, Resistor_SMD:R_0805_2012Metric_Pad1.20x1.40mm_HandSolder, F.Cu at (201.4, 244.4)
- added R38: 12k 0.5%, Resistor_SMD:R_0805_2012Metric_Pad1.20x1.40mm_HandSolder, F.Cu at (201.4, 247.4)
- added R39: 24k 0.5%, Resistor_SMD:R_0805_2012Metric_Pad1.20x1.40mm_HandSolder, F.Cu at (206.2, 244.4)
- added R40: 12k 0.5%, Resistor_SMD:R_0805_2012Metric_Pad1.20x1.40mm_HandSolder, F.Cu at (201.4, 250.3)
- added R41: 24k 0.5%, Resistor_SMD:R_0805_2012Metric_Pad1.20x1.40mm_HandSolder, F.Cu at (206.2, 247.4)
- added R42: 12k 0.5%, Resistor_SMD:R_0805_2012Metric_Pad1.20x1.40mm_HandSolder, F.Cu at (210.9, 244.4)
- added R43: 24k 0.5%, Resistor_SMD:R_0805_2012Metric_Pad1.20x1.40mm_HandSolder, F.Cu at (201.4, 253.3)
- added R44: 12k 0.5%, Resistor_SMD:R_0805_2012Metric_Pad1.20x1.40mm_HandSolder, F.Cu at (206.2, 250.3)
- added R45: 24k 0.5%, Resistor_SMD:R_0805_2012Metric_Pad1.20x1.40mm_HandSolder, F.Cu at (210.9, 247.4)
- added R46: 12k 0.5%, Resistor_SMD:R_0805_2012Metric_Pad1.20x1.40mm_HandSolder, F.Cu at (215.7, 244.4)
- added R47: 24k 0.5%, Resistor_SMD:R_0805_2012Metric_Pad1.20x1.40mm_HandSolder, F.Cu at (206.2, 253.3)
- added R48: 4990 0.5%, Resistor_SMD:R_0805_2012Metric_Pad1.20x1.40mm_HandSolder, F.Cu at (210.9, 250.3)
- added R7: DNF, Resistor_SMD:R_0805_2012Metric_Pad1.20x1.40mm_HandSolder, F.Cu at (192.4, 244.4)
- added R96: 10k, Resistor_SMD:R_0805_2012Metric_Pad1.20x1.40mm_HandSolder, F.Cu at (208.9, 232.3)
- added R97: 10k, Resistor_SMD:R_0805_2012Metric_Pad1.20x1.40mm_HandSolder, F.Cu at (213.7, 226.4)
- added R98: 10k, Resistor_SMD:R_0805_2012Metric_Pad1.20x1.40mm_HandSolder, F.Cu at (208.9, 229.3)
- added R99: 75R, Resistor_SMD:R_0805_2012Metric_Pad1.20x1.40mm_HandSolder, F.Cu at (203.6, 234.2)
- added U19: THS7316, Package_SO:SOIC-8_3.9x4.9mm_P1.27mm, F.Cu at (177.8, 236.0)
- added U2: THS7316, Package_SO:SOIC-8_3.9x4.9mm_P1.27mm, F.Cu at (177.8, 246.2)
- added U20: TPD7S019, Package_SO:SSOP-16_3.9x4.9mm_P0.635mm, F.Cu at (210.5, 218.6)
- added U3: TPD7S019, Package_SO:SSOP-16_3.9x4.9mm_P0.635mm, F.Cu at (186.0, 246.3)
- C70: renamed from C1005; value 4u7 10V -> 4u7 16V
- R35: renamed from R413; value 3300 -> 4990 0.5%
- renumbered BT1201 to BT1, C202 to C1, C637 to C10, C629 to C11, C603 to C12, C612 to C13, C634 to C14, C638 to C15, C604 to C16, C613 to C17, C602 to C18, C601 to C19, C635 to C20, C627 to C21, C626 to C22, C636 to C23, C605 to C24, C606 to C25, C614 to C26, C615 to C27, C620 to C28, C621 to C29, C204 to C3, C630 to C30, C607 to C31, C616 to C32, C608 to C33, C617 to C34, C631 to C35, C622 to C36, C609 to C37, C618 to C38, C623 to C39, C632 to C40, C610 to C41, C624 to C42, C619 to C43, C625 to C44, C701 to C45, C702 to C46, C805 to C47, C801 to C48, C802 to C49, C803 to C50, C804 to C51, C901 to C52, C902 to C53, C906 to C54, C903 to C55, C907 to C56, C911 to C57, C908 to C58, C912 to C59, C201 to C6, C909 to C60, C904 to C61, C910 to C62, C905 to C63, C1008 to C64, C1001 to C65, C1009 to C66, C1002 to C67, C1003 to C68, C1004 to C69, C628 to C7, C1006 to C71, C1007 to C72, C1010 to C73, C1011 to C74, C1106 to C75, C1107 to C76, C1108 to C77, C1109 to C78, C1110 to C79, C611 to C8, C1111 to C80, C1112 to C81, C1105 to C82, C1103 to C83, C1104 to C84, C1101 to C85, C1102 to C86, C1202 to C87, C1203 to C88, C1201 to C89, C633 to C9, D901 to D1, F901 to F1, FB608 to FB1, FB604 to FB10, FB606 to FB11, FB610 to FB2, FB609 to FB3, FB611 to FB4, FB601 to FB5, FB603 to FB6, FB607 to FB7, FB605 to FB8, FB602 to FB9, H104 to H1, H101 to H2, H105 to H3, H102 to H4, H106 to H5, H108 to H6, H103 to H7, H107 to H8, H109 to H9, J101 to J1, J801 to J10, J802 to J11, J901 to J12, J905 to J13, J902 to J14, J904 to J15, J903 to J16, J1001 to J17, J1002 to J18, J1101 to J19, J102 to J2, J103 to J3, J104 to J4, J201 to J5, J603 to J6, J602 to J7, J601 to J8, J701 to J9, JP901 to JP1, L901 to L1, LOGO101 to LOGO1, LOGO102 to LOGO2, LOGO103 to LOGO3, Q901 to Q1, R204 to R1, R412 to R24, R407 to R25, R402 to R26, R408 to R27, R403 to R28, R409 to R29, R410 to R31, R405 to R32, R411 to R33, R406 to R34, R201 to R4, R614 to R49, R202 to R5, R616 to R50, R615 to R51, R601 to R52, R602 to R53, R603 to R54, R605 to R55, R609 to R56, R604 to R57, R606 to R58, R611 to R59, R203 to R6, R612 to R60, R610 to R61, R607 to R62, R608 to R63, R613 to R64, R801 to R65, R901 to R66, R908 to R67, R909 to R68, R904 to R69, R906 to R70, R902 to R71, R903 to R72, R905 to R73, R907 to R74, R910 to R75, R1001 to R76, R1004 to R77, R1005 to R78, R1006 to R79, R208 to R8, R1007 to R80, R1002 to R81, R1008 to R82, R1003 to R83, R1105 to R84, R1112 to R85, R1111 to R86, R1101 to R87, R1103 to R88, R1104 to R89, R209 to R9, R1107 to R90, R1102 to R91, R1106 to R92, R1109 to R93, R1108 to R94, R1110 to R95, RN701 to RN1, RN901 to RN2, SW901 to SW1, SW902 to SW2, TP901 to TP1, TP902 to TP2, TP904 to TP3, TP905 to TP4, TP906 to TP5, TP903 to TP6, U101 to U1, U904 to U10, U1001 to U11, U1004 to U12, U1002 to U13, U1003 to U14, U1005 to U15, U1006 to U16, U1101 to U17, U1201 to U18, U601 to U4, U602 to U5, U801 to U6, U901 to U7, U903 to U8, U902 to U9, Y601 to Y1, Y1001 to Y2, Y1101 to Y3, Y1201 to Y4
Connections:
- C6 pad 2: Net-(C201-Pad2) -> Net-(C6-Pad2)
- J1 pad 1: (no net) -> Net-(J1-Pad1)
- J1 pad 10: (no net) -> Net-(J1-Pad10)
- J1 pad 14: (no net) -> Net-(J1-Pad14)
- J1 pad 3: (no net) -> Net-(J1-Pad3)
- J1 pad 5: (no net) -> Net-(J1-Pad5)
- J1 pad 7: (no net) -> Net-(J1-Pad7)
- J1 pad 8: (no net) -> Net-(J1-Pad8)
- J1 pad 9: (no net) -> Net-(J1-Pad9)
- J10 pad 1: (no net) -> Net-(J10-Pad1)
- J10 pad 10: (no net) -> Net-(J10-Pad10)
- J10 pad 4: (no net) -> Net-(J10-Pad4)
- J10 pad 6: (no net) -> Net-(J10-Pad6)
- J10 pad 9: (no net) -> Net-(J10-Pad9)
- J11 pad 1: (no net) -> Net-(J11-Pad1)
- J11 pad 4: (no net) -> Net-(J11-Pad4)
- J11 pad 6: (no net) -> Net-(J11-Pad6)
- J11 pad 9: (no net) -> Net-(J11-Pad9)
- J13 pad 12: (no net) -> Net-(J13-Pad12)
- J13 pad 2: (no net) -> Net-(J13-Pad2)
- J13 pad 6: (no net) -> Net-(J13-Pad6)
- J13 pad 8: (no net) -> Net-(J13-Pad8)
- J19 pad R7: (no net) -> Net-(J19-PadR7)
- J2 pad 1: (no net) -> Net-(J2-Pad1)
- J2 pad 10: (no net) -> Net-(J2-Pad10)
- J2 pad 14: (no net) -> Net-(J2-Pad14)
- J2 pad 3: (no net) -> Net-(J2-Pad3)
- J2 pad 5: (no net) -> Net-(J2-Pad5)
- J2 pad 7: (no net) -> Net-(J2-Pad7)
- J2 pad 8: (no net) -> Net-(J2-Pad8)
- J2 pad 9: (no net) -> Net-(J2-Pad9)
- J3 pad 1: (no net) -> Net-(J3-Pad1)
- J3 pad 10: (no net) -> Net-(J3-Pad10)
- J3 pad 14: (no net) -> Net-(J3-Pad14)
- J3 pad 3: (no net) -> Net-(J3-Pad3)
- J3 pad 5: (no net) -> Net-(J3-Pad5)
- J3 pad 7: (no net) -> Net-(J3-Pad7)
- J3 pad 8: (no net) -> Net-(J3-Pad8)
- J3 pad 9: (no net) -> Net-(J3-Pad9)
- J4 pad 1: (no net) -> Net-(J4-Pad1)
- J4 pad 10: (no net) -> Net-(J4-Pad10)
- J4 pad 14: (no net) -> Net-(J4-Pad14)
- J4 pad 3: (no net) -> Net-(J4-Pad3)
- J4 pad 5: (no net) -> Net-(J4-Pad5)
- J4 pad 7: (no net) -> Net-(J4-Pad7)
- J4 pad 8: (no net) -> Net-(J4-Pad8)
- J4 pad 9: (no net) -> Net-(J4-Pad9)
- J5 pad 0: Net-(J201-Pad0) -> Net-(J5-Pad0)
- J5 pad 1: /Video/VGA_RED -> /18-bit Video/VGA_RED
- J5 pad 11: (no net) -> Net-(J5-Pad11)
- J5 pad 12: /Video/VGA_DDC_SDA -> /18-bit Video/VGA_DDC_SDA
- J5 pad 13: /Video/VGA_HSYNC -> /18-bit Video/VGA_HSYNC
- J5 pad 14: /Video/VGA_VSYNC -> /18-bit Video/VGA_VSYNC
- J5 pad 15: /Video/VGA_DDC_SCL -> /18-bit Video/VGA_DDC_SCL
- J5 pad 2: /Video/VGA_GRN -> /18-bit Video/VGA_GRN
- J5 pad 3: /Video/VGA_BLU -> /18-bit Video/VGA_BLU
- J5 pad 4: (no net) -> Net-(J5-Pad4)
- J7 pad 8: (no net) -> Net-(J7-Pad8)
- R1 pad 2: /Video/RED_ANA -> /18-bit Video/RED_ANA
- R24 pad 1: Net-(R401-Pad2) -> Net-(R23-Pad2)
- R25 pad 2: Net-(R401-Pad2) -> Net-(R23-Pad2)
- R26 pad 1: /Video/Blue DAC/DIGITAL_IN1 -> /12-bit Video/Blue DAC/DIGITAL_IN1
- R28 pad 1: /Video/Blue DAC/DIGITAL_IN2 -> /12-bit Video/Blue DAC/DIGITAL_IN2
- R29 pad 1: Net-(R404-Pad2) -> Net-(R29-Pad1)
- R31 pad 2: Net-(R404-Pad2) -> Net-(R29-Pad1)
- R32 pad 1: /Video/Blue DAC/DIGITAL_IN4 -> /18-bit Video/Blue DAC/DIGITAL_IN4
- R33 pad 1: /Video/GREEN_ANA -> /18-bit Video/GREEN_ANA
- R34 pad 1: /Video/Blue DAC/DIGITAL_IN5 -> /18-bit Video/Blue DAC/DIGITAL_IN5
- R34 pad 2: /Video/GREEN_ANA -> /18-bit Video/GREEN_ANA
- R35 pad 1: /Video/GREEN_ANA -> /18-bit Video/GREEN_ANA
- R4 pad 1: /Video/VGA_RED -> /18-bit Video/VGA_RED
- R4 pad 2: Net-(R201-Pad2) -> Net-(R4-Pad2)
- R5 pad 1: /Video/VGA_GRN -> /18-bit Video/VGA_GRN
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
Commit message: Changes to BMC
* Swapped BUTTON_PWR and SYS_RESET to avoid DRC issue
* Split PSU and BMC into two separate sheets
* Swapped some pins on the STM32 to make it compatible with more
alternatives
Parts:
- removed the C203 at (253.7, 79.6)
- removed the C205 at (245.7, 85.5)
- removed the C206 at (236.6, 79.1)
- removed C55: 22u 16V, Capacitor_SMD:C_0805_2012Metric_Pad1.15x1.40mm_HandSolder
- removed C57: 10n, Capacitor_SMD:C_0805_2012Metric_Pad1.15x1.40mm_HandSolder
- removed C58, C60, C61: 100n, Capacitor_SMD:C_0805_2012Metric_Pad1.15x1.40mm_HandSolder
- removed C59, C63: 1u 10V, Capacitor_SMD:C_0805_2012Metric_Pad1.15x1.40mm_HandSolder
- removed C62: 4u7 10V, Capacitor_SMD:C_0805_2012Metric_Pad1.15x1.40mm_HandSolder
- removed D1: LED, LED_THT:LED_D3.0mm
- removed F1: 32V 2A PTC, Fuse:Fuse_BelFuse_0ZRE0016FF_L9.9mm_W3.8mm
- removed J12: Jack-DC, Connector_BarrelJack:BarrelJack_CUI_PJ-063AH_Horizontal
- removed J13: Double-mini-DIN-6, Neotron-Common-Hardware:Double_mini-DIN_6
- removed J14: Conn_01x06, Connector_PinHeader_2.54mm:PinHeader_1x06_P2.54mm_Vertical
- removed J15: Header, Connector_PinHeader_2.54mm:PinHeader_1x02_P2.54mm_Vertical
- removed J16: Conn_01x03, Connector_PinHeader_2.54mm:PinHeader_1x03_P2.54mm_Vertical
- removed JP1: Jumper, Connector_PinHeader_2.54mm:PinHeader_1x02_P2.54mm_Vertical
- removed L1: 22uH 6A, Inductor_THT:L_Axial_L26.7mm_D12.1mm_P35.00mm_Horizontal_Vishay_IHA-103
- removed the R205 at (248.9, 76.7)
- removed the R206 at (244.2, 79.6)
- removed the R207 at (244.2, 76.7)
- removed the R301 at (54.7, 116.4)
- removed the R302 at (68.9, 116.4)
- removed the R303 at (64.2, 119.3)
- removed the R304 at (59.4, 122.3)
- removed the R305 at (68.9, 113.4)
- removed the R306 at (64.2, 116.4)
- removed the R307 at (59.4, 119.3)
- removed the R308 at (54.7, 122.3)
- removed the R309 at (64.2, 113.4)
- removed the R310 at (59.4, 116.4)
- removed the R311 at (54.7, 113.4)
- removed the R312 at (54.7, 119.3)
- removed the R313 at (59.4, 113.4)
- removed the R401 at (64.2, 134.6)
- removed the R404 at (64.2, 131.6)
- removed the R501 at (93.7, 116.4)
- removed the R502 at (89.0, 119.3)
- removed the R503 at (84.2, 122.3)
- removed the R504 at (93.7, 113.4)
- removed the R505 at (89.0, 116.4)
- removed the R506 at (84.2, 119.3)
- removed the R507 at (79.5, 122.3)
- removed the R508 at (89.0, 113.4)
- removed the R509 at (84.2, 116.4)
- removed the R510 at (79.5, 119.3)
- removed the R511 at (84.2, 113.4)
- removed the R512 at (79.5, 116.4)
- removed the R513 at (79.5, 113.4)
- removed R67, R68: 1k, Resistor_SMD:R_0805_2012Metric_Pad1.15x1.40mm_HandSolder
- removed R69, R70, R71, R72, R73, R74, R75: 10k, Resistor_SMD:R_0805_2012Metric_Pad1.15x1.40mm_HandSolder
- removed RN2: 2k7 x 4, Resistor_THT:R_Array_SIP5
- removed SW1, SW2: SW_DIP_x01, Connector_PinHeader_2.54mm:PinHeader_1x02_P2.54mm_Vertical
- removed TP1, TP2, TP3, TP4, TP5, TP6: TestPoint_Small, Connector_PinHeader_2.54mm:PinHeader_1x01_P2.54mm_Vertical
- removed U10: STM32F031K6T6, Package_QFP:LQFP-32_7x7mm_P0.8mm
- removed the U201 at (232.9, 53.5)
- removed the U202 at (221.2, 53.3)
- removed U7: 5V DC-DC Module, Neotron-Common-Hardware:K78xx-3AR3
- removed U8: MAX1615, Package_TO_SOT_SMD:SOT-23-5
- added C1601: 100n, Capacitor_SMD:C_0805_2012Metric_Pad1.18x1.45mm_HandSolder, F.Cu at (154.4, 259.8)
- added C1602: 100n, Capacitor_SMD:C_0805_2012Metric_Pad1.18x1.45mm_HandSolder, F.Cu at (150.8, 264.4)
- added C1603: 4u7 10V, Capacitor_SMD:C_0805_2012Metric_Pad1.18x1.45mm_HandSolder, F.Cu at (161.0, 253.0)
- added C1604: 10n, Capacitor_SMD:C_0805_2012Metric_Pad1.18x1.45mm_HandSolder, F.Cu at (161.0, 250.0)
- added C1605: 1u 10V, Capacitor_SMD:C_0805_2012Metric_Pad1.18x1.45mm_HandSolder, F.Cu at (149.6, 261.4)
- added C1704: 22u 16V, Capacitor_SMD:C_0805_2012Metric_Pad1.18x1.45mm_HandSolder, F.Cu at (122.8, 235.5)
- added C1706: 100n, Capacitor_SMD:C_0805_2012Metric_Pad1.18x1.45mm_HandSolder, F.Cu at (127.6, 235.5)
- added C1707: 1u 10V, Capacitor_SMD:C_0805_2012Metric_Pad1.18x1.45mm_HandSolder, F.Cu at (132.4, 235.5)
- added D1601: LED, LED_THT:LED_D3.0mm, F.Cu at (153.5, 255.5)
- added D1602: LED, LED_THT:LED_D3.0mm, F.Cu at (144.2, 266.1)
- added F1701: 32V 2A PTC, Fuse:Fuse_BelFuse_0ZRE0016FF_L9.9mm_W3.8mm, F.Cu at (162.5, 211.0)
- added J1601: Header, Connector_PinHeader_2.54mm:PinHeader_1x02_P2.54mm_Vertical, F.Cu at (140.2, 261.0)
- added J1602: Header, Connector_PinHeader_2.54mm:PinHeader_1x02_P2.54mm_Vertical, F.Cu at (144.9, 258.4)
- added J1603: Conn_01x05, Connector_PinHeader_2.54mm:PinHeader_1x05_P2.54mm_Vertical, F.Cu at (144.9, 243.6)
- added J1604: Conn_01x06, Connector_PinHeader_2.54mm:PinHeader_1x06_P2.54mm_Vertical, F.Cu at (140.2, 243.6)
- added J1605: Double-mini-DIN-6, Neotron-Common-Hardware:Double_mini-DIN_6, F.Cu at (268.7, 42.6)
- added J1701: Jack-DC, Connector_BarrelJack:BarrelJack_CUI_PJ-063AH_Horizontal, F.Cu at (252.2, 32.5)
- added JP1601: Jumper, Connector_PinHeader_2.54mm:PinHeader_1x02_P2.54mm_Vertical, F.Cu at (149.5, 255.1)
- added L1701: 22uH 6A, Inductor_THT:L_Axial_L26.7mm_D12.1mm_P35.00mm_Horizontal_Vishay_IHA-103, F.Cu at (122.4, 215.9)
- added R1601: 1k 1%, Resistor_SMD:R_0805_2012Metric_Pad1.20x1.40mm_HandSolder, F.Cu at (165.8, 250.0)
- added R1602: 1k 1%, Resistor_SMD:R_0805_2012Metric_Pad1.20x1.40mm_HandSolder, F.Cu at (160.1, 256.0)
- added R1603: 1k 1%, Resistor_SMD:R_0805_2012Metric_Pad1.20x1.40mm_HandSolder, F.Cu at (165.8, 252.9)
- added R1604: 1k 1%, Resistor_SMD:R_0805_2012Metric_Pad1.20x1.40mm_HandSolder, F.Cu at (150.8, 267.4)
- added R1605: 10k 1%, Resistor_SMD:R_0805_2012Metric_Pad1.20x1.40mm_HandSolder, F.Cu at (155.6, 262.8)
- added R1606: 10k 1%, Resistor_SMD:R_0805_2012Metric_Pad1.20x1.40mm_HandSolder, F.Cu at (160.1, 259.0)
- added R1607: 10k 1%, Resistor_SMD:R_0805_2012Metric_Pad1.20x1.40mm_HandSolder, F.Cu at (164.9, 256.0)
- added R1608: 10k 1%, Resistor_SMD:R_0805_2012Metric_Pad1.20x1.40mm_HandSolder, F.Cu at (155.6, 265.7)
- added R1609: 10k 1%, Resistor_SMD:R_0805_2012Metric_Pad1.20x1.40mm_HandSolder, F.Cu at (160.4, 261.9)
- added R1610: 10k 1%, Resistor_SMD:R_0805_2012Metric_Pad1.20x1.40mm_HandSolder, F.Cu at (164.9, 259.0)
- added R1701: 100k 1%, Resistor_SMD:R_0805_2012Metric_Pad1.20x1.40mm_HandSolder, F.Cu at (137.2, 235.5)
- added RN1601: 2k7 x 4, Resistor_THT:R_Array_SIP5, F.Cu at (122.6, 264.6)
- added SW1601: SW_DIP_x01, Connector_PinHeader_2.54mm:PinHeader_1x02_P2.54mm_Vertical, F.Cu at (160.9, 243.6)
- added SW1602: SW_DIP_x01, Connector_PinHeader_2.54mm:PinHeader_1x02_P2.54mm_Vertical, F.Cu at (165.6, 243.6)
- added U1601: STM32F031K6T6, Package_QFP:LQFP-32_7x7mm_P0.8mm, F.Cu at (152.9, 247.0)
- added U1701: 5V DC-DC Module, Neotron-Common-Hardware:K78xx-3AR3, F.Cu at (136.2, 225.8)
- added U1702: MAX1615, Package_TO_SOT_SMD:SOT-23-5, F.Cu at (161.8, 216.8)
- C1001: renamed from C75; footprint Capacitor_SMD:C_0805_2012Metric_Pad1.15x1.40mm_HandSolder -> Capacitor_SMD:C_0805_2012Metric_Pad1.18x1.45mm_HandSolder
- C1002: renamed from C76; footprint Capacitor_SMD:C_0805_2012Metric_Pad1.15x1.40mm_HandSolder -> Capacitor_SMD:C_0805_2012Metric_Pad1.18x1.45mm_HandSolder
- C1003: renamed from C77; footprint Capacitor_SMD:C_0805_2012Metric_Pad1.15x1.40mm_HandSolder -> Capacitor_SMD:C_0805_2012Metric_Pad1.18x1.45mm_HandSolder
- C1004: renamed from C78; footprint Capacitor_SMD:C_0805_2012Metric_Pad1.15x1.40mm_HandSolder -> Capacitor_SMD:C_0805_2012Metric_Pad1.18x1.45mm_HandSolder
- C1005: renamed from C79; footprint Capacitor_SMD:C_0805_2012Metric_Pad1.15x1.40mm_HandSolder -> Capacitor_SMD:C_0805_2012Metric_Pad1.18x1.45mm_HandSolder
- C1006: renamed from C80; footprint Capacitor_SMD:C_0805_2012Metric_Pad1.15x1.40mm_HandSolder -> Capacitor_SMD:C_0805_2012Metric_Pad1.18x1.45mm_HandSolder
- C1007: renamed from C81; footprint Capacitor_SMD:C_0805_2012Metric_Pad1.15x1.40mm_HandSolder -> Capacitor_SMD:C_0805_2012Metric_Pad1.18x1.45mm_HandSolder
- C1008: renamed from C82; footprint Capacitor_SMD:C_0805_2012Metric_Pad1.15x1.40mm_HandSolder -> Capacitor_SMD:C_0805_2012Metric_Pad1.18x1.45mm_HandSolder
- C1009: renamed from C83; footprint Capacitor_SMD:C_0805_2012Metric_Pad1.15x1.40mm_HandSolder -> Capacitor_SMD:C_0805_2012Metric_Pad1.18x1.45mm_HandSolder
- C1010: renamed from C84; footprint Capacitor_SMD:C_0805_2012Metric_Pad1.15x1.40mm_HandSolder -> Capacitor_SMD:C_0805_2012Metric_Pad1.18x1.45mm_HandSolder
- C1011: renamed from C85; footprint Capacitor_SMD:C_0805_2012Metric_Pad1.15x1.40mm_HandSolder -> Capacitor_SMD:C_0805_2012Metric_Pad1.18x1.45mm_HandSolder
- C1012: renamed from C86; footprint Capacitor_SMD:C_0805_2012Metric_Pad1.15x1.40mm_HandSolder -> Capacitor_SMD:C_0805_2012Metric_Pad1.18x1.45mm_HandSolder
- C1101: renamed from C87; footprint Capacitor_SMD:C_0805_2012Metric_Pad1.15x1.40mm_HandSolder -> Capacitor_SMD:C_0805_2012Metric_Pad1.18x1.45mm_HandSolder
- C1102: renamed from C88; footprint Capacitor_SMD:C_0805_2012Metric_Pad1.15x1.40mm_HandSolder -> Capacitor_SMD:C_0805_2012Metric_Pad1.18x1.45mm_HandSolder
- C1103: renamed from C89; footprint Capacitor_SMD:C_0805_2012Metric_Pad1.15x1.40mm_HandSolder -> Capacitor_SMD:C_0805_2012Metric_Pad1.18x1.45mm_HandSolder
- C1703: renamed from C54; footprint Capacitor_SMD:C_0805_2012Metric_Pad1.15x1.40mm_HandSolder -> Capacitor_SMD:C_0805_2012Metric_Pad1.18x1.45mm_HandSolder
- C1705: renamed from C56; footprint Capacitor_SMD:C_0805_2012Metric_Pad1.15x1.40mm_HandSolder -> Capacitor_SMD:C_0805_2012Metric_Pad1.18x1.45mm_HandSolder
- C201: renamed from C1; footprint Capacitor_SMD:C_0805_2012Metric_Pad1.15x1.40mm_HandSolder -> Capacitor_SMD:C_0805_2012Metric_Pad1.18x1.45mm_HandSolder
- C203: renamed from C3; footprint Capacitor_SMD:C_0805_2012Metric_Pad1.15x1.40mm_HandSolder -> Capacitor_SMD:C_0805_2012Metric_Pad1.18x1.45mm_HandSolder
- C206: renamed from C6; footprint Capacitor_SMD:C_0805_2012Metric_Pad1.15x1.40mm_HandSolder -> Capacitor_SMD:C_0805_2012Metric_Pad1.18x1.45mm_HandSolder
- C601: renamed from C7; footprint Capacitor_SMD:C_0805_2012Metric_Pad1.15x1.40mm_HandSolder -> Capacitor_SMD:C_0805_2012Metric_Pad1.18x1.45mm_HandSolder
- C602: renamed from C8; footprint Capacitor_SMD:C_0805_2012Metric_Pad1.15x1.40mm_HandSolder -> Capacitor_SMD:C_0805_2012Metric_Pad1.18x1.45mm_HandSolder
- renumbered BT1 to BT1101, C90 to C1201, C91 to C1202, C92 to C1203, C93 to C1204, C94 to C1205, C95 to C1206, C52 to C1701, C53 to C1702, C2 to C202, C4 to C204, C5 to C205, C26 to C620, C27 to C621, C71 to C908, C72 to C909, C73 to C910, C74 to C911, FB1 to FB601, FB2 to FB602, FB3 to FB603, FB4 to FB604, FB5 to FB605, FB6 to FB606, FB8 to FB607, FB7 to FB608, FB9 to FB609, FB10 to FB610, FB11 to FB611, H1 to H101, H2 to H102, H3 to H103, H4 to H104, H5 to H105, H6 to H106, H7 to H107, H8 to H108, H9 to H109, J19 to J1001, J1 to J101, J2 to J102, J3 to J103, J4 to J104, J20 to J1201, J5 to J201, J6 to J601, J7 to J602, J8 to J603, J9 to J701, J10 to J801, J11 to J802, J17 to J901, J18 to J902, LOGO1 to LOGO101, LOGO2 to LOGO102, LOGO3 to LOGO103, Q1 to Q1701, R102 to R1207, R105 to R1301, R106 to R1302, R107 to R1303, R108 to R1304, R109 to R1305, R110 to R1306, R111 to R1307, R112 to R1308, R113 to R1309, R114 to R1310, R115 to R1401, R116 to R1402, R117 to R1403, R118 to R1404, R119 to R1405, R120 to R1406, R121 to R1407, R122 to R1408, R123 to R1409, R124 to R1410, R125 to R1501, R126 to R1502, R127 to R1503, R128 to R1504, R129 to R1505, R130 to R1506, R131 to R1507, R132 to R1508, R133 to R1509, R134 to R1510, R7 to R207, R10 to R301, R11 to R302, R12 to R303, R13 to R304, R14 to R305, R15 to R306, R16 to R307, R17 to R308, R18 to R309, R19 to R310, R20 to R311, R21 to R312, R22 to R313, R23 to R401, R30 to R408, R36 to R501, R37 to R502, R38 to R503, R39 to R504, R40 to R505, R41 to R506, R42 to R507, R43 to R508, R44 to R509, R45 to R510, R46 to R511, R47 to R512, R48 to R513, RN1 to RN701, U17 to U1001, U1 to U101, U18 to U1101, U19 to U1201, U20 to U1202, U9 to U1703, U2 to U201, U3 to U202, U4 to U601, U5 to U602, U6 to U801, U11 to U901, U12 to U902, U13 to U903, U14 to U904, U15 to U905, U16 to U906, Y3 to Y1001, Y4 to Y1101, Y1 to Y601, Y2 to Y901
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Connections:
- J1001 pad R7: Net-(J19-PadR7) -> (no net)
- J101 pad 1: Net-(J1-Pad1) -> (no net)
- J101 pad 10: Net-(J1-Pad10) -> (no net)
- J101 pad 14: Net-(J1-Pad14) -> (no net)
- J101 pad 3: Net-(J1-Pad3) -> (no net)
- J101 pad 5: Net-(J1-Pad5) -> (no net)
- J101 pad 7: Net-(J1-Pad7) -> (no net)
- J101 pad 8: Net-(J1-Pad8) -> (no net)
- J101 pad 9: Net-(J1-Pad9) -> (no net)
- J102 pad 1: Net-(J2-Pad1) -> (no net)
- J102 pad 10: Net-(J2-Pad10) -> (no net)
- J102 pad 14: Net-(J2-Pad14) -> (no net)
- J102 pad 3: Net-(J2-Pad3) -> (no net)
- J102 pad 5: Net-(J2-Pad5) -> (no net)
- J102 pad 7: Net-(J2-Pad7) -> (no net)
- J102 pad 8: Net-(J2-Pad8) -> (no net)
- J102 pad 9: Net-(J2-Pad9) -> (no net)
- J103 pad 1: Net-(J3-Pad1) -> (no net)
- J103 pad 10: Net-(J3-Pad10) -> (no net)
- J103 pad 14: Net-(J3-Pad14) -> (no net)
- J103 pad 3: Net-(J3-Pad3) -> (no net)
- J103 pad 5: Net-(J3-Pad5) -> (no net)
- J103 pad 7: Net-(J3-Pad7) -> (no net)
- J103 pad 8: Net-(J3-Pad8) -> (no net)
- J103 pad 9: Net-(J3-Pad9) -> (no net)
- J104 pad 1: Net-(J4-Pad1) -> (no net)
- J104 pad 10: Net-(J4-Pad10) -> (no net)
- J104 pad 14: Net-(J4-Pad14) -> (no net)
- J104 pad 3: Net-(J4-Pad3) -> (no net)
- J104 pad 5: Net-(J4-Pad5) -> (no net)
- J104 pad 7: Net-(J4-Pad7) -> (no net)
- J104 pad 8: Net-(J4-Pad8) -> (no net)
- J104 pad 9: Net-(J4-Pad9) -> (no net)
- J1201 pad 11: Net-(J20-Pad11) -> (no net)
- J1201 pad 4: Net-(J20-Pad4) -> (no net)
- J201 pad 11: Net-(J5-Pad11) -> (no net)
- J201 pad 4: Net-(J5-Pad4) -> (no net)
- J602 pad 8: Net-(J7-Pad8) -> (no net)
- J801 pad 1: Net-(J10-Pad1) -> (no net)
- J801 pad 10: Net-(J10-Pad10) -> (no net)
- J801 pad 4: Net-(J10-Pad4) -> (no net)
- J801 pad 6: Net-(J10-Pad6) -> (no net)
- J801 pad 9: Net-(J10-Pad9) -> (no net)
- J802 pad 1: Net-(J11-Pad1) -> (no net)
- J802 pad 4: Net-(J11-Pad4) -> (no net)
- J802 pad 6: Net-(J11-Pad6) -> (no net)
- J802 pad 9: Net-(J11-Pad9) -> (no net)
- Q1701 pad 1: /Power Supply/~PSU_EN -> /Power Supply and BMC/~PSU_EN
- R1702 pad 2: /Power Supply/DC_ON -> /Power Supply and BMC/DC_ON
- U1001 pad 23: Net-(U17-Pad23) -> (no net)
- U1001 pad 25: Net-(U17-Pad25) -> (no net)
- U1001 pad 26: Net-(U17-Pad26) -> (no net)
- U1001 pad 27: Net-(U17-Pad27) -> (no net)
- U1001 pad 28: Net-(U17-Pad28) -> (no net)
- U1001 pad 29: Net-(U17-Pad29) -> (no net)
- U1001 pad 30: Net-(U17-Pad30) -> (no net)
- U1001 pad 31: Net-(U17-Pad31) -> (no net)
- U1001 pad 32: Net-(U17-Pad32) -> (no net)
- U1001 pad 34: /Ethernet/~SPI_CS -> (no net)
- U1001 pad 35: /Ethernet/SPI_CIPO -> (no net)
- U1001 pad 36: /Ethernet/SPI_COPI -> (no net)
- U1001 pad 37: /Ethernet/SPI_CLK -> (no net)
- U1001 pad 38: Net-(U17-Pad38) -> (no net)
- U1001 pad 39: Net-(U17-Pad39) -> (no net)
- U1001 pad 40: Net-(U17-Pad40) -> (no net)
- U1001 pad 41: Net-(U17-Pad41) -> (no net)
- U1001 pad 5: Net-(U17-Pad5) -> (no net)
- U1001 pad 6: Net-(U17-Pad6) -> (no net)
- U1001 pad 7: Net-(U17-Pad7) -> (no net)
- U1001 pad 8: Net-(U17-Pad8) -> (no net)
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
Commit message: Brought in sheets from Neotron Pico.
Also includes DB15HD and PSU 3D models.
Parts:
- removed the FB604 at (155.8, 62.0)
- removed the J1604 at (140.2, 243.6)
- removed RN1601: 2k7 x 4, Resistor_THT:R_Array_SIP5
- added C1706: 10uF, Capacitor_SMD:C_0805_2012Metric_Pad1.18x1.45mm_HandSolder, F.Cu at (68.5, 170.3)
- added Q1702: BC556, Package_TO_SOT_THT:TO-92_Inline, F.Cu at (74.6, 166.3)
- added R1606: 10k, Resistor_SMD:R_0805_2012Metric_Pad1.20x1.40mm_HandSolder, F.Cu at (96.9, 164.5)
- added R1612: 2k7, Resistor_SMD:R_0805_2012Metric_Pad1.20x1.40mm_HandSolder, F.Cu at (92.2, 167.5)
- added R1613: 2k7, Resistor_SMD:R_0805_2012Metric_Pad1.20x1.40mm_HandSolder, F.Cu at (92.2, 164.5)
- added R1614: 2k7, Resistor_SMD:R_0805_2012Metric_Pad1.20x1.40mm_HandSolder, F.Cu at (87.4, 167.5)
- added R1615: 2k7, Resistor_SMD:R_0805_2012Metric_Pad1.20x1.40mm_HandSolder, F.Cu at (87.4, 164.5)
- added R1701: 10k, Resistor_SMD:R_0805_2012Metric_Pad1.20x1.40mm_HandSolder, F.Cu at (78.0, 170.3)
- C1101, C1102: value 6p -> 6pF
- C1103, C1201, C1202, C1203, C1204, C1601, C1602, C607, C610, C611, C612, C615, C702: value 100n -> 100nF
- C1205, C602, C603, C604, C606, C608, C609, C613, C614, C616, C617, C701: value 10u 10V -> 10uF
- C1206: value 220n -> 220nF
- C1603, C1705: value 4u7 10V -> 4.7uF
- C1604: value 10n -> 10nF
- C1605, C624: value 1u 10V -> 1uF
- C1701, C1702: value 100u 50V -> 100uF; footprint Capacitor_THT:CP_Radial_D6.3mm_P2.50mm -> Capacitor_THT:CP_Radial_D8.0mm_P5.00mm
- C1703: value 1u 50V -> 100nF
- C1704: value 22u 16V -> 10uF
- C1707: renamed from C1706; value 100n -> 100nF
- C1708: renamed from C1707; value 1u 10V -> 1uF
- C601, C605: value 22p -> 22pF
- C618, C619, C622, C623: value 470n -> 470nF
- C620, C621: value 220u 16V -> 220uF; footprint Capacitor_THT:CP_Radial_D6.3mm_P2.50mm -> Capacitor_THT:CP_Radial_D8.0mm_P5.00mm
- C629: value 47p -> 47pF
- FB601, FB602, FB603: value 3k3 -> 330R@100MHz
- FB604: renamed from FB605; value 3k3 -> 330R@100MHz
- FB605: renamed from FB606; value 3k3 -> 330R@100MHz
- FB606: renamed from FB607; value 3k3 -> 330R@100MHz
- FB607: renamed from FB608; value 600R@100MHz -> 330R@100MHz
- FB608: renamed from FB609; value 3k3 -> 330R@100MHz
- FB609: renamed from FB610; value 3k3 -> 330R@100MHz
- FB610: renamed from FB611; value 3k3 -> 330R@100MHz
- J1201, J201: footprint Connector_Dsub:DSUB-15-HD_Female_Horizontal_P2.29x1.98mm_EdgePinOffset3.03mm_Housed_MountingHolesOffset4.94mm -> Neotron-Common-Hardware:Amphenol_ICD15S13E4GV00LF
- J1701: value Jack-DC -> Jack 2/6.3mm
- L1701: value 22uH 6A -> 22uH 2A; footprint Inductor_THT:L_Axial_L26.7mm_D12.1mm_P35.00mm_Horizontal_Vishay_IHA-103 -> Inductor_THT:L_Radial_D9.5mm_P5.00mm_Fastron_07HVP
- Q1701: value BC548 -> BC546; footprint Package_TO_SOT_THT:TO-92_HandSolder -> Package_TO_SOT_THT:TO-92_Inline
- R1201, R1202, R1203, R1605, R616: value 10k 1% -> 10k
- R1204, R1205, R1206: value 75R 1% -> 75R
- R1208, R1209: value 1k5 1% -> 1k5
- R1301, R1302, R1304, R1306, R1308, R1401, R1402, R1404, R1406, R1408, R1501, R1502, R1504, R1506, R1508, R301, R302, R304, R306, R308, R310, R312, R401, R402, R404, R406, R408, R410, R412, R501, R502, R504, R506, R508, R510, R512: value 24k 0.5% -> 24k
- R1303, R1305, R1307, R1309, R1403, R1405, R1407, R1409, R1503, R1505, R1507, R1509, R303, R305, R307, R309, R311, R403, R405, R407, R409, R411, R503, R505, R507, R509, R511: value 12k 0.5% -> 12k
- R1310, R1410, R1510: value 3480 0.5% -> 5490
- R1601, R1602, R1603, R1604: value 1k 1% -> 1k
- R1607: renamed from R1606; value 10k 1% -> 10k
- R1608: renamed from R1607; value 10k 1% -> 10k
- R1609: renamed from R1608; value 10k 1% -> 10k
- R1610: renamed from R1609; value 10k 1% -> 10k
- R1611: renamed from R1610; value 10k 1% -> 10k
- R1702: value 1k 1% -> 10k
- R1703: renamed from R1701; value 100k 1% -> 10k
- R313, R413, R513: value 4990 0.5% -> 4990
- R601, R602, R603: value 2R2 1% -> 2R2
- R604, R605: value 100R 1% -> 100R
- R606, R607, R611, R612: value 47k 1% -> 47k
- R608, R610, R613, R614, R615: value 4k7 1% -> 4k7
- R609: value 2k2 1% -> 2k2
- U1101: value MCP7940 -> MCP7940N; footprint Package_SO:SOIC-8_3.9x4.9mm_P1.27mm -> Package_DIP:DIP-8_W7.62mm
- U1701: value 5V DC-DC Module -> DC-DC Module
- Y601: value 12M -> 12M 20pF; footprint Crystal:Crystal_HC49-4H_Vertical -> Crystal:Crystal_SMD_5032-2Pin_5.0x3.2mm_HandSoldering
- moved R1702 203.6 mm to (73.3, 170.3)
- moved R304 198.6 mm to (46.4, 164.5)
- moved R305 197.0 mm to (46.4, 167.5)
- moved Q1701 192.2 mm to (68.1, 166.3)
- moved R306 189.5 mm to (51.1, 164.5)
- moved R307 188.7 mm to (46.4, 170.4)
- moved R309 184.1 mm to (55.9, 164.5)
- moved R310 183.3 mm to (51.1, 170.4)
- moved R308 181.3 mm to (51.1, 167.5)
- moved R312 177.9 mm to (55.9, 170.4)
- moved R302 177.8 mm to (60.6, 164.5)
- moved R311 175.9 mm to (55.9, 167.5)
- moved R507 170.4 mm to (68.5, 150.8)
- moved R510 168.8 mm to (68.5, 156.7)
- moved R511 168.8 mm to (73.2, 153.7)
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- renumbered J1605 to J1604
Connections:
- C1702 pad 1: Net-(C1702-Pad1) -> VDC
- C1703 pad 1: Net-(C1702-Pad1) -> VDC
- C604 pad 2: GNDA -> GND
- C606 pad 2: GNDA -> GND
- C609 pad 2: GNDA -> GND
- C610 pad 2: GNDA -> GND
- C612 pad 2: GNDA -> GND
- C613 pad 2: GNDA -> GND
- C615 pad 2: GNDA -> GND
- C616 pad 2: GNDA -> GND
- C625 pad 1: GNDA -> GND
- C626 pad 1: GNDA -> GND
- C627 pad 1: GNDA -> GND
- C628 pad 1: GNDA -> GND
- C629 pad 1: GNDA -> GND
- C630 pad 1: GNDA -> GND
- C631 pad 1: GNDA -> GND
- C632 pad 1: GNDA -> GND
- C633 pad 1: GNDA -> GND
- C634 pad 1: GNDA -> GND
- C635 pad 1: GNDA -> GND
- C636 pad 1: GNDA -> GND
- C637 pad 1: GNDA -> GND
- C638 pad 1: GNDA -> GND
- J601 pad 2: GNDA -> GND
- J601 pad 3: GNDA -> GND
- J602 pad 2: GNDA -> GND
- J602 pad 4: GNDA -> GND
- J603 pad 2: GNDA -> GND
- J603 pad 3: GNDA -> GND
- L1701 pad 2: Net-(C1702-Pad1) -> VDC
- Q1701 pad 1: /Power Supply and BMC/~PSU_EN -> Net-(Q1701-Pad1)
- R1702 pad 1: Net-(Q1701-Pad2) -> VDC
- R1702 pad 2: /Power Supply and BMC/DC_ON -> Net-(Q1701-Pad1)
- R1703 pad 1: /Power Supply and BMC/DC_ON -> /Power Supply and BMC/~SHDN
- R606 pad 2: GNDA -> GND
- R607 pad 2: GNDA -> GND
- R608 pad 2: GNDA -> GND
- R611 pad 1: GNDA -> GND
- R612 pad 1: GNDA -> GND
- R613 pad 1: GNDA -> GND
- R616 pad 1: GNDA -> GND
- U1202 pad 3: /12-bit Video/VGA_RED -> /12-bit Video/VGA_BLU
- U1202 pad 5: /12-bit Video/VGA_BLU -> /12-bit Video/VGA_RED
- U1601 pad 14: (no net) -> /Board Management Controller/LED0
- U1601 pad 15: (no net) -> /Board Management Controller/LED1
- U1601 pad 19: /Board Management Controller/UART_TX -> (no net)
- U1601 pad 20: /Board Management Controller/UART_RX -> (no net)
- U1601 pad 21: /Board Management Controller/UART_CTS -> (no net)
- U1601 pad 22: /Board Management Controller/UART_RTS -> (no net)
- U1601 pad 8: /Board Management Controller/LED0 -> /Board Management Controller/~RESET
- U1601 pad 9: /Board Management Controller/LED1 -> (no net)
- U1701 pad 1: /Power Supply and BMC/~PSU_EN -> /Power Supply and BMC/~SHDN
- U1701 pad 2: Net-(C1702-Pad1) -> VDC
- U1702 pad 1: Net-(C1702-Pad1) -> VDC
- U1702 pad 5: Net-(C1702-Pad1) -> VDC
- U601 pad 11: GNDA -> GND
- U601 pad 15: GNDA -> GND
- U602 pad 1: GNDA -> GND

Commit message: Fixups after last copy-over.
Parts:
- added C1801: 100nF, Capacitor_SMD:C_0805_2012Metric_Pad1.18x1.45mm_HandSolder, F.Cu at (246.3, 135.1)
- added C1802: 100nF, Capacitor_SMD:C_0805_2012Metric_Pad1.18x1.45mm_HandSolder, F.Cu at (258.7, 120.6)
- added U1801: MCP23S17_SO, Package_SO:SOIC-28W_7.5x17.9mm_P1.27mm, F.Cu at (237.4, 128.9)
- added U1802: 74HC245, Package_SO:SO-20_12.8x7.5mm_P1.27mm, F.Cu at (250.1, 126.4)
- C1001, C1002, C1003, C1004, C1005, C201, C202, C203, C204, C801, C802, C803, C804, C805, C902, C904, C906: value 100n -> 100nF
- C1006, C1007: value 1n -> 1nF
- C1008: value 10u Low ESR -> 10uF
- C1011, C1012: value 10n -> 10nF
- C205: value 10u 10V -> 10uF
- C206: value 220n -> 220nF
- C905: value 4u7 10V -> 4.7uF
- C907: value 4u7 16V -> 4.7uF
- C908, C909, C910, C911: value 120u 16V -> 120uF
- L1701: value 22uH 2A -> 22uH
- R1001: value 100k 1% -> 100k
- R1002: value 12k4 1% -> 12k4
- R1003: value 1M 1% -> 1M
- R1004, R1005, R1006, R1007: value 49R9 1% -> 49R9
- R1008, R1009: value 10R 1% -> 10R
- R1010, R1011: value 180R 1% -> 180R
- R1612, R1613, R1614, R1615: value 2k7 -> 1k
- R201, R202, R203, R901, R902, R903, R904, R905, R907, R908: value 10k 1% -> 10k
- R204, R205, R206: value 75R 1% -> 75R
- R208, R209: value 1k5 1% -> 1k5
- R906: value 2k7 1% -> 2k7
- RN701: value 8x10k -> 10k

Commit message: Update fileformats to Kicad 6.
Connections:
- net /Board Management Controller/~BMC_RST renamed /Board Management Controller/~{BMC_RST}
- net /Board Management Controller/~BUTTON_PWR renamed /Board Management Controller/~{BUTTON_PWR}
- net /Board Management Controller/~BUTTON_RST renamed /Board Management Controller/~{BUTTON_RST}
- net /Board Management Controller/~RESET renamed /Board Management Controller/~{RESET}
- net /Ethernet/~IRQ renamed /Ethernet/~{IRQ}
- net /IO Expander/~CS0 renamed /IO Expander/~{CS0}
- net /IO Expander/~CS1 renamed /IO Expander/~{CS1}
- net /IO Expander/~CS2 renamed /IO Expander/~{CS2}
- net /IO Expander/~CS3 renamed /IO Expander/~{CS3}
- net /IO Expander/~CS4 renamed /IO Expander/~{CS4}
- net /IO Expander/~CS5 renamed /IO Expander/~{CS5}
- net /IO Expander/~CS6 renamed /IO Expander/~{CS6}
- net /IO Expander/~CS7 renamed /IO Expander/~{CS7}
- net /Power Supply and BMC/~SHDN renamed /Power Supply and BMC/~{SHDN}
- net /SD Card/~CARD_DETECT renamed /SD Card/~{CARD_DETECT}
- net /SD Card/~WRITE_PROTECT renamed /SD Card/~{WRITE_PROTECT}
- net /USB/~ENABLE renamed /USB/~{ENABLE}
Other:
- net class Default removed
